File: pcb/asset tracker/asset tracker.kicad_sch (KiCad schematic)
At the start: 0 parts

Commit message: som board
som test board done
Other:
- added sheet beweging  (beweging.kicad_sch)
- added sheet gps (gps.kicad_sch)
- added sheet gsm (gsm.kicad_sch)
- added sheet io (io.kicad_sch)
- added sheet level shifter (level shifter.kicad_sch)
- added sheet mcu (mcu.kicad_sch)
- added sheet voeding (voeding.kicad_sch)
- note added: "MEMMORIE NOG UIT TE ZOEKEN"
- company: (none) -> eurocircutis
- title: (none) -> Asset tracker
