File: pcb/som asset tracker/som asset tracker/gps.kicad_sch (KiCad schematic)
At the start: 11 parts, among them U4 bga725l6

Commit message: clasificatie
op naar een betere clasificatie
Parts:
- removed C9: 120pF, vanalles:0603, symbol Device:C_Small
- removed R8: 10K, vanalles:0603, symbol Device:R_Small_US
- removed U4: bga725l6, halfgeleiders:INFINEON_BGA725L6E6327FTSA1, symbol Halfgelijders:bga725l6
- removed Z1: b4327, halfgeleiders:QUALCOMM_B39162B4327P810, symbol vanalles:b4327
Connections:
- net at mod2.11 (RF_IN): now also L1.1
- net ANT_OFF: no longer names the net of mod2.13 (ANT_OFF)
- net VCC: no longer names the net of mod2.14 (VCC_RF)
- no-connect marks 2 -> 4
Other:
- moved on the sheet: AE1, C10, L1
