File: pcb/som asset tracker/som asset tracker/io.kicad_sch (KiCad schematic)
At the start: 9 parts, among them J2 Screw_Terminal_01x02, Q1 BBS3002, U5 G3VM-61HR2(TR05), U6 DS28CM00R-A00+T

Commit message: key
pcb for the key
Parts:
- removed Q1: BBS3002, halfgeleiders:sot-23,, symbol Halfgelijders:BBS3002
- added Q?: BSS138, symbol Halfgelijders:BSS138
Connections:
- net +3V3: now also Q?.2
- net BUZZER: now also Q?.1
- net at PZ1.1: now also Q?.3
Changed lines of the file:
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@@
-(kicad_sch (version 20210126) (generator eeschema)
+(kicad_sch (version 20210406) (generator eeschema)
   (paper "A4")
   (junction (at 33.02 165.1) (diameter 0.9144) (color 0 0 0 0))
@@
     (stroke (width 0) (type solid) (color 0 0 0 0))
   )
-  (wire (pts (xy 54.61 154.94) (xy 54.61 160.02))
-    (stroke (width 0) (type solid) (color 0 0 0 0))
-  )
-  (wire (pts (xy 54.61 170.18) (xy 54.61 175.26))
+  (wire (pts (xy 54.61 153.67) (xy 54.61 156.21))
+    (stroke (width 0) (type solid) (color 0 0 0 0))
+  )
+  (wire (pts (xy 54.61 173.99) (xy 54.61 175.26))
     (stroke (width 0) (type solid) (color 0 0 0 0))
   )
@@
     (effects (font (size 1.27 1.27)) (justify right))
   )
-  (symbol (lib_id "power:+3V3") (at 54.61 154.94 0) (unit 1)
-    (in_bom yes) (on_board yes)
-    (property "Reference" "#PWR0132" (id 0) (at 54.61 158.75 0)
-      (effects (font (size 1.27 1.27)) hide)
-    )
-    (property "Value" "+3V3" (id 1) (at 54.61 151.13 0))
-    (property "Footprint" "" (id 2) (at 54.61 154.94 0)
-      (effects (font (size 1.27 1.27)) hide)
-    )
-    (property "Datasheet" "" (id 3) (at 54.61 154.94 0)
+  (symbol (lib_id "power:+3V3") (at 54.61 153.67 0) (unit 1)
+    (in_bom yes) (on_board yes)
+    (property "Reference" "#PWR0132" (id 0) (at 54.61 157.48 0)
+      (effects (font (size 1.27 1.27)) hide)
+    )
+    (property "Value" "+3V3" (id 1) (at 54.61 149.86 0))
+    (property "Footprint" "" (id 2) (at 54.61 153.67 0)
+      (effects (font (size 1.27 1.27)) hide)
+    )
+    (property "Datasheet" "" (id 3) (at 54.61 153.67 0)
       (effects (font (size 1.27 1.27)) hide)
     )
@@
     (pin "2")
   )
-  (symbol (lib_id "Halfgelijders:BBS3002") (at 53.34 165.1 0) (unit 1)
-    (in_bom yes) (on_board yes) (fields_autoplaced)
-    (property "Reference" "Q1" (id 0) (at 58.42 164.4649 0)
-      (effects (font (size 1.27 1.27)) (justify left))
-    )
-    (property "Value" "BBS3002" (id 1) (at 58.42 167.0049 0)
-      (effects (font (size 1.27 1.27)) (justify left))
-    )
-    (property "Footprint" "halfgeleiders:sot-23," (id 2) (at 52.07 160.02 0)
-      (effects (font (size 1.27 1.27)) hide)
-    )
-    (property "Datasheet" "" (id 3) (at 52.07 160.02 0)
+  (symbol (lib_id "Halfgelijders:BSS138") (at 53.34 165.1 0) (unit 1)
+    (in_bom yes) (on_board yes) (fields_autoplaced)
+    (property "Reference" "Q?" (id 0) (at 58.42 164.4649 0)
+      (effects (font (size 1.27 1.27)) (justify left))
+    )
+    (property "Value" "BSS138" (id 1) (at 58.42 167.0049 0)
+      (effects (font (size 1.27 1.27)) (justify left))
+    )
+    (property "Footprint" "" (id 2) (at 53.34 165.1 0)
+      (effects (font (size 1.27 1.27)) hide)
+    )
+    (property "Datasheet" "" (id 3) (at 53.34 165.1 0)
       (effects (font (size 1.27 1.27)) hide)
     )
@@
   )
   (symbol (lib_id "Halfgelijders:DS28CM00R-A00+T") (at 96.52 101.6 0) (unit 1)
-    (in_bom yes) (on_board yes) (fields_autoplaced)
+    (in_bom yes) (on_board yes)
     (property "Reference" "U6" (id 0) (at 106.68 100.3299 0)
       (effects (font (size 1.27 1.27)) (justify left))
