File: pcb/som asset tracker/som asset tracker/som asset tracker.kicad_pcb (KiCad board)
At the start: 2 copper layers, 100 x 100 mm, 48 parts, among them CON1 jtag, J1 Screw_Terminal_01x02, J2 Screw_Terminal_01x02, J3 Conn_01x05_Male, J4 Conn_01x05_Male, J5 Conn_01x05_Male, J6 Conn_01x02_Male, J7 Conn_01x02_Male, Q1 BBS3002, U1 INA219BxDCN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

Commit message: clasificatie
op naar een betere clasificatie
Parts:
- removed C9: 120pF, vanalles:0603
- removed R8: 10K, vanalles:0603
- removed U4: bga725l6, halfgeleiders:INFINEON_BGA725L6E6327FTSA1
- removed Z1: b4327, halfgeleiders:QUALCOMM_B39162B4327P810
- added REF**: MountingHole_2.2mm_M2_ISO7380, vanalles:MountingHole_2.2mm_M2_ISO7380, F.Cu at (100.3, 42.0)
- added REF**: MountingHole_2.2mm_M2_ISO7380, vanalles:MountingHole_2.2mm_M2_ISO7380, F.Cu at (196.1, 42.2)
- added REF**: MountingHole_2.2mm_M2_ISO7380, vanalles:MountingHole_2.2mm_M2_ISO7380, F.Cu at (100.2, 137.8)
- moved D3 277.6 mm to (-79.5, 122.8), turned to 0 degrees
- moved Q1 273.6 mm to (-79.2, 158.7), turned to 0 degrees
- moved R3 273.5 mm to (-79.9, 125.1)
- moved D2 272.3 mm to (-75.0, 120.1), turned to 0 degrees
- moved R2 268.2 mm to (-75.4, 122.6)
- moved PZ1 267.2 mm to (-74.4, 138.1)
- moved R9 266.5 mm to (-70.7, 147.3)
- moved U5 255.9 mm to (-77.1, 154.6), turned to 0 degrees
- moved J2 237.4 mm to (-62.5, 131.8), turned to 0 degrees
- moved R10 229.9 mm to (-61.4, 134.8), turned to 0 degrees
- moved J3 215.1 mm to (-16.7, 38.5), turned to 0 degrees
- moved R11 193.2 mm to (-65.1, 137.2), turned to 0 degrees
- moved J5 190.6 mm to (-16.7, 32.3)
- moved R12 188.8 mm to (-65.1, 134.8)
- moved J4 183.8 mm to (-16.7, 26.6), turned to 0 degrees
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Connections:
- R10 pad 2: /SSR -> Net-(R10-Pad2)
- U5 pad 1: /SSR -> Net-(R10-Pad2)
- mod2 pad 11: Net-(C9-Pad1) -> Net-(L1-Pad1)
- mod2 pad 13: /gps/ANT_OFF -> unconnected-(mod2-Pad13)
- mod2 pad 14: VCC -> unconnected-(mod2-Pad14)
Routing:
- net /SDA: track 153.1 -> 0.00 mm, vias 6 -> 0
- net /SCL: track 144.3 -> 0.00 mm, vias 4 -> 0
- net GND: track 191.5 -> 73.0 mm, vias 26 -> 19
- net /SOM/GREEN: track 74.0 -> 0.00 mm, vias 2 -> 0
- net /SOM/BLUE: track 69.4 -> 0.00 mm, vias 2 -> 0
- net /INT1: track 68.4 -> 0.00 mm, vias 2 -> 0
- net VDC: track 68.1 -> 0.00 mm
- net /SOM/RED: track 66.6 -> 0.00 mm, vias 2 -> 0
- net /INT2: track 60.4 -> 0.00 mm, vias 5 -> 0
- net /BUZZER: track 43.7 -> 0.00 mm, vias 2 -> 0
- net /SSR: track 38.9 -> 0.00 mm, vias 1 -> 0
- net Net-(BT1-Pad1): track 81.6 -> 109.4 mm
- net /WAKE: track 81.7 -> 56.1 mm
- net /PPS: track 75.3 -> 50.8 mm, vias 0 -> 2
- net /LED1: track 22.5 -> 0.00 mm, vias 3 -> 0
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Other:
- board text removed: "GNDS"
- board text removed: "I,U,P sensor"
- board text removed: "JTAG"
- board text removed: "SCL"
- board text removed: "SDA"
- board text removed: "TP 1"
- board text removed: "TP 2"
- board text removed: "TP 3"
- board text removed: "VIN+"
- board text removed: "VIN-"
- board text removed: "big noise maker +"
- board text removed: "big noise maker -"
- board text removed: "buzzer"
- board text removed: "int1"
- board text removed: "int2"
- board text removed: "movment sensor"
- board text removed: "pps"
- board text removed: "reset"
- board text removed: "rx"
- board text removed: "ssr"
- board text removed: "tx"
- board text removed: "unique ID"
- board text removed: "wake"

Commit message: key
pcb for the key
Parts:
- moved D3 279.7 mm to (196.1, 75.2), turned to 180 degrees
- moved R3 276.5 mm to (192.0, 75.2)
- moved D2 274.9 mm to (195.6, 71.7), turned to 180 degrees
- moved R2 272.2 mm to (192.0, 71.7)
- moved Q1 270.7 mm to (173.4, 61.5), turned to 90 degrees
- moved PZ1 264.2 mm to (174.4, 49.3)
- moved R9 261.3 mm to (176.9, 64.0), turned to -90 degrees
- moved U5 249.8 mm to (152.1, 55.3), turned to 180 degrees
- moved J2 230.9 mm to (153.3, 49.8), turned to 180 degrees
- moved R10 219.3 mm to (144.9, 60.7)
- moved J3 212.1 mm to (194.8, 54.1), turned to 90 degrees
- moved R11 199.0 mm to (121.3, 67.7), turned to 180 degrees
- moved R12 193.8 mm to (116.5, 67.1)
- moved C2 188.9 mm to (128.2, 59.7)
- moved J5 188.1 mm to (163.4, 86.4)
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Routing:
- net /SDA: track 0.00 -> 159.7 mm, vias 0 -> 5
- net /SCL: track 0.00 -> 158.6 mm, vias 0 -> 5
- net GND: track 73.0 -> 150.3 mm, vias 19 -> 27
- net /SOM/GREEN: track 0.00 -> 75.8 mm, vias 0 -> 4
- net /SOM/RED: track 0.00 -> 72.2 mm, vias 0 -> 4
- net /SOM/BLUE: track 0.00 -> 68.9 mm, vias 0 -> 4
- net /INT2: track 0.00 -> 52.6 mm
- net /INT1: track 0.00 -> 51.9 mm, vias 0 -> 2
- net VDC: track 0.00 -> 51.1 mm
- net /BUZZER: track 0.00 -> 50.3 mm, vias 0 -> 2
- net /SSR: track 0.00 -> 49.6 mm, vias 0 -> 3
- net +3V3: track 0.00 -> 37.2 mm, vias 0 -> 2
- net /TX: track 61.7 -> 93.7 mm, vias 2 -> 4
- net /RX: track 63.0 -> 92.3 mm
- net Net-(J1-Pad2): track 0.00 -> 17.6 mm, vias 0 -> 2
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Other:
- board text added: "+"
- board text added: "-"
- board text added: "BIG NOISEMAKER +"
- board text added: "BIG NOISEMAKER -"
- board text added: "BUZZER"
- board text added: "GNDS"
- board text added: "INT1"
- board text added: "INT2"
- board text added: "P,U,I meter"
- board text added: "PPS"
- board text added: "RESET"
- board text added: "RX"
- board text added: "SCL"
- board text added: "SDA"
- board text added: "SMALL NOISEMAKER"
- board text added: "SOM"
- board text added: "SSR"
- board text added: "TP1"
- board text added: "TP2"
- board text added: "TP3"
- board text added: "TX"
- board text added: "WAKE"
- board text added: "gps"
- board text added: "jtag"
- board text added: "movment sensor"
- board text added: "unique id number"
