File: pcb/asset tracker LoRa/LoRa tracker/LoRa tracker.kicad_pcb (KiCad board)
At the start: 0 parts

Commit message: 34t
34t
Parts:
- added AE1: sma, connectors_user:sma_right angeld, F.Cu at (85.9, 133.2)
- added AE2: Antenna, vanalles:Texas_SWRA117D_2.4GHz_Right, F.Cu at (117.1, 131.6)
- added AE3: Antenna_Shield, connectors_user:sma_right angeld, F.Cu at (136.6, 133.4)
- added BT1: Battery_Cell, vanalles:3012TR, F.Cu at (70.9, 90.1)
- added C1: 100nF, vanalles:0603, F.Cu at (98.9, 62.1)
- added C10: 4.7uF, vanalles:0603, F.Cu at (111.1, 114.5)
- added C11: 100nF, vanalles:0603, F.Cu at (111.2, 108.2)
- added C12: 100nF, vanalles:0603, F.Cu at (111.2, 111.5)
- added C13: 1uF, vanalles:0603, F.Cu at (121.6, 115.4)
- added C14: 100pF, vanalles:0603, F.Cu at (120.4, 124.9)
- added C15: 100nF, vanalles:0603, F.Cu at (119.5, 112.6)
- added C16: NM, vanalles:0603, F.Cu at (113.0, 125.3)
- added C17: 12pF, vanalles:0603, F.Cu at (122.5, 119.4)
- added C18: 12pF, vanalles:0603, F.Cu at (127.0, 120.1)
- added C19: NM, vanalles:0603, F.Cu at (113.0, 127.2)
- added C2: 10uF, vanalles:0603, F.Cu at (98.8, 60.1)
- added C20: 10uF, vanalles:0603, F.Cu at (118.3, 80.2)
- added C21: 10uF, vanalles:0603, F.Cu at (123.0, 83.4)
- added C22: 100nF, vanalles:0603, F.Cu at (123.0, 80.8)
- added C23: NM, vanalles:0603, F.Cu at (140.7, 124.9)
- added C24: NM, vanalles:0603, F.Cu at (132.6, 126.3)
- added C3: 100nF, vanalles:0603, F.Cu at (80.2, 57.5)
- added C4: 10uF, vanalles:0603, F.Cu at (80.2, 59.9)
- added C5: 10uF, vanalles:0603, F.Cu at (108.3, 67.5)
- added C6: 100nF, vanalles:0603, F.Cu at (108.3, 65.6)
- added C7: 10uF, vanalles:0603, F.Cu at (80.0, 107.8)
- added C8: 100nF, vanalles:0603, F.Cu at (80.0, 105.5)
- added C9: 120nF, vanalles:0603, F.Cu at (86.0, 123.8)
- added CON1: jtag, connectors_user:Tag-Connect_TC2050-IDC-FP_2x05_P1.27mm_Vertical, F.Cu at (104.2, 117.8)
- added CON2: jtag, connectors_user:Tag-Connect_TC2050-IDC-FP_2x05_P1.27mm_Vertical, F.Cu at (108.4, 82.1)
- added J1: Screw_Terminal_01x02, connectors_user:2pin_screw, F.Cu at (72.1, 54.0)
- added J2: Screw_Terminal_01x02, connectors_user:2pin_screw, F.Cu at (121.4, 48.0)
- added L1: 5n6, vanalles:0603, F.Cu at (85.9, 119.5)
- added MOD1: rfm95, Module:RFM69HW, F.Cu at (142.8, 113.0)
- added MOD2: teseo-LIV, Module:SON_STM_TESEO-LIV3R, F.Cu at (89.2, 110.6)
- added PZ1: buzzer, vanalles:PROSIGNAL_ABI-017-RC, F.Cu at (142.2, 46.6)
- added Q1: BSS138, halfgeleiders:sot-23,, F.Cu at (153.4, 46.7)
- added R1: 100m Ohm, vanalles:R_2512_6332Metric_Pad1.40x3.35mm_HandSolder, F.Cu at (84.8, 51.5)
- added R2: 10K, vanalles:0603, F.Cu at (155.5, 50.8)
- added R3: 220, vanalles:0603, F.Cu at (118.9, 67.4)
- added R4: 10K, vanalles:0603, F.Cu at (128.2, 79.3)
- added R5: 10K, vanalles:0603, F.Cu at (128.5, 73.3)
- added R6: 0, vanalles:0603RL, F.Cu at (117.2, 126.6)
- added R7: 10K, vanalles:0603, F.Cu at (132.8, 103.9)
- added R8: 0, vanalles:0603RL, F.Cu at (135.8, 125.5)
- added REF**: MountingHole_2.2mm_M2_Pad_Via, vanalles:MountingHole_2.2mm_M2_Pad_Via, F.Cu at (159.7, 40.4)
- added REF**: MountingHole_2.2mm_M2_Pad_Via, vanalles:MountingHole_2.2mm_M2_Pad_Via, F.Cu at (64.7, 135.3)
- added REF**: MountingHole_2.2mm_M2_Pad_Via, vanalles:MountingHole_2.2mm_M2_Pad_Via, F.Cu at (64.7, 40.4)
- added REF**: MountingHole_2.2mm_M2_Pad_Via, vanalles:MountingHole_2.2mm_M2_Pad_Via, F.Cu at (159.7, 135.1)
- added U1: INA219BxDCN, halfgeleiders:SOIC127P599X175-8N, F.Cu at (85.2, 60.3)
- added U2: R-783.3-1.0, vanalles:recom psu, F.Cu at (100.4, 55.3)
- added U3: LIS3DH, halfgeleiders:QFN-16_0.5MM, F.Cu at (110.1, 70.8)
- added U4: G3VM-61HR2(TR05), halfgeleiders:sop4 P=2.54, F.Cu at (121.5, 56.1)
- added U5: DS28CM00R-A00+T, halfgeleiders:SOT-25, F.Cu at (128.9, 76.3)
- added U6: nRF52810-QFxx, halfgeleiders:nrf, F.Cu at (116.6, 118.2)
- added U7: ATSAMD21, halfgeleiders:QFN49P40_600X600X90L40X20T460N, F.Cu at (118.9, 87.5)
- added Y1: 326MhZ, vanalles:OSCCC320X250X90L80X100N, B.Cu at (125.0, 123.7)
Routing:
- net GND: track 0.00 -> 176.7 mm, vias 0 -> 31
- net /SDA: track 0.00 -> 126.2 mm, vias 0 -> 6
- net /SCL: track 0.00 -> 122.8 mm, vias 0 -> 4
- net /INT2: track 0.00 -> 72.4 mm, vias 0 -> 2
- net /PPS: track 0.00 -> 71.0 mm, vias 0 -> 7
- net /BUZZER: track 0.00 -> 61.5 mm
- net VDC: track 0.00 -> 61.4 mm
- net /RESET_GPS: track 0.00 -> 61.0 mm, vias 0 -> 2
- net /WAKE: track 0.00 -> 59.5 mm, vias 0 -> 2
- net Net-(BT1-Pad1): track 0.00 -> 58.3 mm, vias 0 -> 1
- net /CS: track 0.00 -> 52.2 mm, vias 0 -> 3
- net /INT1: track 0.00 -> 50.2 mm, vias 0 -> 4
- net /IRQ: track 0.00 -> 48.6 mm, vias 0 -> 2
- net /SSR: track 0.00 -> 47.9 mm
- net /MISO: track 0.00 -> 38.6 mm
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- added copper zone on F.Cu, net +3V3
- added copper zone on B.Cu, net GND
Other:
- board outline added: 100 x 100 mm
- copper layers 0 -> 2
