File: pcb/asset tracker LoRa/LoRa tracker/LoRa tracker.kicad_pcb (KiCad board)
At the start: 2 copper layers, 100 x 100 mm, 57 parts, among them CON1 jtag, CON2 jtag, J1 Screw_Terminal_01x02, J2 Screw_Terminal_01x02, Q1 BSS138, U1 INA219BxDCN, U2 R-783.3-1.0, U3 LIS3DH, U4 G3VM-61HR2(TR05), U5 DS28CM00R-A00+T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

Commit message: pcb kastje
pcb in kastje getekend
Parts:
- removed C20: 10uF, vanalles:0603
- removed MOD1: rfm95, Module:RFM69HW
- removed REF** (x4): MountingHole_2.2mm_M2_Pad_Via, vanalles:MountingHole_2.2mm_M2_Pad_Via
- added C25: 10uF, vanalles:0603, F.Cu at (130.2, 64.6)
- added C26: 1uF, vanalles:0603, F.Cu at (130.1, 66.5)
- added C27: 0.1uF, vanalles:0603, F.Cu at (130.2, 62.5)
- added C28: 100nF, vanalles:0603, F.Cu at (160.2, 89.8)
- added C29: 10uF, vanalles:0603, F.Cu at (154.1, 116.5)
- added C30: 100nF, vanalles:0603, F.Cu at (158.0, 89.9)
- added C31: 10uF, vanalles:0603, F.Cu at (154.0, 113.6)
- added C32: 100nF, vanalles:0603, F.Cu at (115.0, 44.1)
- added C33: 20pF, vanalles:0603, F.Cu at (125.0, 120.1)
- added C34: 20pF, vanalles:0603, F.Cu at (115.1, 120.1)
- added CON3: jtag, connectors_user:Tag-Connect_TC2050-IDC-FP_2x05_P1.27mm_Vertical, F.Cu at (116.5, 54.5)
- added R9: 10K, vanalles:0603RL, F.Cu at (113.8, 47.8)
- added U8: murattaLora, Module:XCVR_CMWX1ZZABZ-078, F.Cu at (132.3, 53.6)
- added U9: ATECC608B, halfgeleiders:soic p1.27 lengt 5.40, F.Cu at (158.8, 110.0)
- added Y2: Crystal, vanalles:crystal tht, F.Cu at (119.2, 120.1)
- AE1, AE3: footprint connectors_user:sma_right angeld -> connectors_user:sma juist
- AE2: value Antenna -> Antenna_Shield; footprint vanalles:Texas_SWRA117D_2.4GHz_Right -> connectors_user:sma juist
- C10, C11, C12, C14: moved to B.Cu
- R7: footprint vanalles:0603 -> vanalles:0603RL
- U7: value ATSAMD21 -> ATSAMD21G18A-M; footprint halfgeleiders:QFN49P40_600X600X90L40X20T460N -> halfgeleiders:QFN50P700X700X90-49N
- Y1: moved to F.Cu
- moved J1 141.0 mm to (153.0, 169.5), turned to 0 degrees
- moved R1 131.5 mm to (155.7, 162.2), turned to 90 degrees
- moved J2 121.5 mm to (121.0, 169.6), turned to 180 degrees
- moved U1 116.7 mm to (146.7, 159.5), turned to 180 degrees
- moved C3 108.5 mm to (146.7, 143.3), turned to -90 degrees
- moved U4 108.1 mm to (120.5, 164.2), turned to 0 degrees
- moved U2 105.7 mm to (155.6, 145.5), turned to 90 degrees
- moved AE2 105.6 mm to (94.2, 28.5)
- moved AE3 105.4 mm to (134.3, 28.0), turned to 180 degrees
- moved C4 105.1 mm to (144.2, 143.3), turned to -90 degrees
- moved C2 101.0 mm to (146.7, 149.0), turned to -90 degrees
- moved C1 98.1 mm to (144.2, 149.1), turned to -90 degrees
- moved C19 89.9 mm to (93.5, 39.4)
- moved C24 87.9 mm to (135.0, 38.4), turned to 0 degrees
- moved R6 86.9 mm to (94.2, 42.8), turned to 90 degrees
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Connections:
- net /LoRa_RFM/ANT_RFM renamed /LoRa_RFM/ANT
- AE2 pad 1: Net-(AE2-Pad1) -> (no net)
- AE2 pad 2: (no net) -> GND
- AE3 pad 1: unconnected-(AE3-Pad1) -> Net-(AE3-Pad1)
- C19 pad 1: Net-(AE2-Pad1) -> (no net)
- C24 pad 1: Net-(C24-Pad1) -> Net-(AE3-Pad1)
- R6 pad 2: Net-(AE2-Pad1) -> (no net)
- R7 pad 1: +3V3 -> GND
- R7 pad 2: /CS -> Net-(R7-Pad2)
- R8 pad 2: Net-(C24-Pad1) -> Net-(AE3-Pad1)
- U7 pad 1: unconnected-(U7-Pad1) -> Net-(C33-Pad2)
- U7 pad 10: /TX -> /RX
- U7 pad 11: /CS -> /TX
- U7 pad 13: /RESET -> unconnected-(U7-Pad13)
- U7 pad 14: /IRQ -> unconnected-(U7-Pad14)
- U7 pad 19: /MOSI -> unconnected-(U7-Pad19)
- U7 pad 2: unconnected-(U7-Pad2) -> Net-(C34-Pad2)
- U7 pad 20: /SCK -> unconnected-(U7-Pad20)
- U7 pad 21: /MISO -> /MOSI
- U7 pad 22: unconnected-(U7-Pad22) -> /SCK
- U7 pad 23: unconnected-(U7-Pad23) -> /CS
- U7 pad 24: /INT1 -> /MISO
- U7 pad 25: /INT2 -> /INT1
- U7 pad 26: /BUZZER -> /INT2
- U7 pad 27: /SSR -> /BUZZER
- U7 pad 28: /PPS -> /SSR
- U7 pad 29: /WAKE -> /PPS
- U7 pad 30: /RESET_GPS -> /WAKE
- U7 pad 31: /SDA -> /RESET_GPS
- U7 pad 32: /SCL -> /SDA
- U7 pad 33: unconnected-(U7-Pad33) -> /SCL
- U7 pad 39: unconnected-(U7-Pad39) -> /RESET
- U7 pad 43: Net-(C20-Pad1) -> +3V3
- U7 pad 49: GND -> unconnected-(U7-Pad49)
- U7 pad 9: /RX -> unconnected-(U7-Pad9)
Routing:
- net /SCL: track 122.8 -> 212.7 mm, vias 4 -> 7
- net /SDA: track 126.2 -> 211.8 mm, vias 6 -> 5
- net /INT2: track 72.4 -> 0.00 mm, vias 2 -> 0
- net /PPS: track 71.0 -> 0.00 mm, vias 7 -> 0
- net /RESET_GPS: track 61.0 -> 0.00 mm, vias 2 -> 0
- net /WAKE: track 59.5 -> 0.00 mm, vias 2 -> 0
- net /CS: track 52.2 -> 0.00 mm, vias 3 -> 0
- net /INT1: track 50.2 -> 0.00 mm, vias 4 -> 0
- net /IRQ: track 48.6 -> 0.00 mm, vias 2 -> 0
- net /MISO: track 38.6 -> 0.00 mm
- net /MOSI: track 37.9 -> 0.00 mm
- net /RX: track 35.5 -> 0.00 mm
- net /SCK: track 35.1 -> 0.00 mm, vias 2 -> 0
- net /TX: track 34.3 -> 0.00 mm
- net +3V3: track 30.4 -> 6.17 mm, vias 4 -> 1
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Other:
- board size 100 x 100 mm -> 102.4 x 153.8 mm

Commit message: lora tracker
lora tracker afgemaakt
Parts:
- added TP1: RESET, vanalles:TestPoint_Pad_D3.0mm, F.Cu at (103.3, 168.6)
- added TP2: MOSI, vanalles:TestPoint_Pad_D3.0mm, F.Cu at (127.5, 146.7)
- added TP3: MISO, vanalles:TestPoint_Pad_D3.0mm, F.Cu at (134.0, 147.1)
- added TP4: CS, vanalles:TestPoint_Pad_D3.0mm, F.Cu at (121.2, 146.9)
- added TP5: SPICLK, vanalles:TestPoint_Pad_D3.0mm, F.Cu at (113.0, 146.9)
- AE1, AE2, AE3: footprint connectors_user:sma juist -> connectors_user:ufl connector
- C10, C11, C12: moved to F.Cu
- U7: footprint halfgeleiders:QFN50P700X700X90-49N -> halfgeleiders:ATSAMD21G18A-M
- moved U3 147.6 mm to (178.2, 190.9)
- moved C32 139.9 mm to (128.1, 183.4), turned to 0 degrees
- moved R9 136.8 mm to (124.7, 184.2), turned to 90 degrees
- moved AE3 134.4 mm to (98.0, 157.3), turned to 90 degrees
- moved C24 122.6 mm to (102.8, 156.7), turned to 90 degrees
- moved CON3 121.4 mm to (120.1, 175.9), turned to 180 degrees
- moved R8 119.1 mm to (106.1, 157.3), turned to 180 degrees
- moved PZ1 117.5 mm to (200.2, 174.8)
- moved Q1 117.0 mm to (198.9, 186.7), turned to -90 degrees
- moved R2 115.1 mm to (195.4, 185.1), turned to 90 degrees
- moved C23 115.0 mm to (109.6, 156.6), turned to 90 degrees
- moved C27 113.3 mm to (129.9, 175.8), turned to 90 degrees
- moved R7 112.5 mm to (125.9, 169.2), turned to 180 degrees
- moved C25 111.3 mm to (132.1, 175.8), turned to 90 degrees
- moved C26 109.3 mm to (127.7, 175.8), turned to 90 degrees
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Connections:
- AE2 pad 1: (no net) -> Net-(AE2-Pad1)
- C19 pad 1: (no net) -> Net-(AE2-Pad1)
- R6 pad 2: (no net) -> Net-(AE2-Pad1)
- U7 pad 49: unconnected-(U7-Pad49) -> GND
Routing:
- net GND: track 200.4 -> 308.1 mm, vias 35 -> 36
- net /RESET: track 36.5 -> 142.2 mm, vias 3 -> 5
- net /PPS: track 0.00 -> 93.1 mm, vias 0 -> 2
- net /RESET_GPS: track 0.00 -> 89.3 mm, vias 0 -> 2
- net /WAKE: track 0.00 -> 81.3 mm, vias 0 -> 2
- net /INT1: track 0.00 -> 72.6 mm, vias 0 -> 4
- net /INT2: track 0.00 -> 71.3 mm, vias 0 -> 2
- net /SCK: track 0.00 -> 69.5 mm, vias 0 -> 2
- net /CS: track 0.00 -> 55.6 mm
- net /RX: track 0.00 -> 51.6 mm, vias 0 -> 2
- net /MISO: track 0.00 -> 51.1 mm, vias 0 -> 2
- net /MOSI: track 0.00 -> 49.1 mm, vias 0 -> 2
- net /TX: track 0.00 -> 47.7 mm, vias 0 -> 2
- net VDC: track 71.8 -> 114.3 mm
- net /SDA: track 211.8 -> 190.5 mm, vias 5 -> 8
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Other:
- board size 102.4 x 153.8 mm -> 116.3 x 114.5 mm

Commit message: klaar
pcb klaar
Parts:
- U7: value ATSAMD21G18A-M -> QFN50P700X700X90-49N

Commit message: klaar
print hertekend naar stm32L5
Parts:
- removed C34: 20pF, vanalles:0603
- added BT2: Battery_Cell, vanalles:3012TR, F.Cu at (132.9, 190.5)
- added C20: 100nF, vanalles:0603, F.Cu at (146.6, 140.6)
- added R10: 10K, vanalles:0603RL, F.Cu at (98.6, 150.0)
- added R11: R_Small_US, vanalles:0603RL, F.Cu at (134.2, 125.9)
- added REF**: Fiducial_1mm_Mask3mm, vanalles:Fiducial_1mm_Mask3mm, F.Cu at (188.2, 86.8)
- added REF**: Fiducial_1mm_Mask3mm, vanalles:Fiducial_1mm_Mask3mm, F.Cu at (75.9, 197.3)
- added REF**: Fiducial_1mm_Mask3mm, vanalles:Fiducial_1mm_Mask3mm, F.Cu at (188.3, 197.3)
- added Y3: 16MHz, vanalles:MURATA_CSTCE16M0V53C-R0, B.Cu at (127.5, 133.7)
- C21: value 10uF -> 1uF
- C22: value 100nF -> 6.8pF
- C33: value 20pF -> 6.8pF
- U7: value QFN50P700X700X90-49N -> STM32L552CCT6; footprint halfgeleiders:ATSAMD21G18A-M -> halfgeleiders:STM32L552CCT6
- Y2: value Crystal -> 32khz
- moved C22 36.0 mm to (130.4, 124.9), turned to 90 degrees
- moved C21 21.2 mm to (146.5, 137.7)
- moved J2 20.0 mm to (178.9, 153.9)
- moved AE1 20.0 mm to (78.0, 101.0)
- moved AE2 20.0 mm to (78.2, 133.5)
- moved AE3 20.0 mm to (78.1, 156.6)
- moved BT1 20.0 mm to (120.6, 94.3)
- moved C1 20.0 mm to (156.5, 112.5)
- moved C10 20.0 mm to (87.8, 126.6)
- moved C11 20.0 mm to (87.8, 122.3)
- moved C12 20.0 mm to (87.9, 124.4)
- moved C13 20.0 mm to (98.4, 139.4)
- moved C14 20.0 mm to (89.0, 135.1)
- moved C15 20.0 mm to (104.3, 135.7)
- moved C16 20.0 mm to (89.4, 132.7)
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Connections:
- C22 pad 1: +3V3 -> /mcu/OSC_32_IN
- C33 pad 1: GND -> /mcu/OSC_32_OUT
- C33 pad 2: Net-(C33-Pad2) -> GND
- CON2 pad 6: unconnected-(CON2-Pad6) -> /mcu/SWO
- CON2 pad 8: unconnected-(CON2-Pad8) -> /mcu/TDI
- U7 pad 1: Net-(C33-Pad2) -> Net-(BT2-Pad1)
- U7 pad 10: /RX -> /TX
- U7 pad 11: /TX -> /RX
- U7 pad 14: unconnected-(U7-Pad14) -> /CS
- U7 pad 15: unconnected-(U7-Pad15) -> /SCK
- U7 pad 16: unconnected-(U7-Pad16) -> /MISO
- U7 pad 17: +3V3 -> /MOSI
- U7 pad 18: GND -> unconnected-(U7-Pad18)
- U7 pad 2: Net-(C34-Pad2) -> unconnected-(U7-Pad2)
- U7 pad 21: /MOSI -> unconnected-(U7-Pad21)
- U7 pad 22: /SCK -> unconnected-(U7-Pad22)
- U7 pad 23: /CS -> GND
- U7 pad 24: /MISO -> +3V3
- U7 pad 25: /INT1 -> unconnected-(U7-Pad25)
- U7 pad 26: /INT2 -> /PPS
- U7 pad 27: /BUZZER -> /WAKE
- U7 pad 28: /SSR -> /RESET_GPS
- U7 pad 29: /PPS -> /RESET
- U7 pad 3: unconnected-(U7-Pad3) -> /mcu/OSC_32_IN
- U7 pad 30: /WAKE -> /SSR
- U7 pad 31: /RESET_GPS -> /BUZZER
- U7 pad 32: /SDA -> /INT2
- U7 pad 33: /SCL -> /INT1
- U7 pad 34: unconnected-(U7-Pad34) -> /mcu/SWDIO
- U7 pad 37: unconnected-(U7-Pad37) -> /mcu/SWDCLK
- U7 pad 38: unconnected-(U7-Pad38) -> /mcu/TDI
- U7 pad 39: /RESET -> /mcu/SWO
- U7 pad 4: unconnected-(U7-Pad4) -> /mcu/OSC_32_OUT
- U7 pad 42: GND -> /SCL
- U7 pad 43: +3V3 -> /SDA
- U7 pad 44: +3V3 -> Net-(R11-Pad1)
- U7 pad 45: /mcu/SWDCLK -> unconnected-(U7-Pad45)
- U7 pad 46: /mcu/SWDIO -> unconnected-(U7-Pad46)
- U7 pad 47: unconnected-(U7-Pad47) -> GND
- U7 pad 48: unconnected-(U7-Pad48) -> +3V3
- U7 pad 5: GND -> /mcu/OSC_HS_IN
- U7 pad 6: +3V3 -> /mcu/OSC_HS_OUT
- U7 pad 7: unconnected-(U7-Pad7) -> +3V3
- U7 pad 8: unconnected-(U7-Pad8) -> GND
- U7 pad 9: unconnected-(U7-Pad9) -> +3V3
- Y2 pad 1: Net-(C34-Pad2) -> /mcu/OSC_32_OUT
- Y2 pad 2: Net-(C33-Pad2) -> /mcu/OSC_32_IN
Routing:
- net Net-(BT2-Pad1): track 0.00 -> 94.4 mm, vias 0 -> 4
- net /SDA: track 190.5 -> 229.8 mm, vias 8 -> 10
- net /mcu/TDI: track 0.00 -> 24.8 mm, vias 0 -> 2
- net /mcu/SWDIO: track 8.89 -> 27.6 mm, vias 0 -> 2
- net /mcu/SWO: track 0.00 -> 18.6 mm, vias 0 -> 2
- net Net-(C34-Pad2): track 14.6 -> 0.00 mm
- net Net-(C33-Pad2): track 13.4 -> 0.00 mm
- net /mcu/OSC_HS_OUT: track 0.00 -> 12.9 mm, vias 0 -> 1
- net /mcu/OSC_HS_IN: track 0.00 -> 10.6 mm, vias 0 -> 1
- net /mcu/OSC_32_OUT: track 0.00 -> 9.84 mm
- net /mcu/OSC_32_IN: track 0.00 -> 9.71 mm
- net /TX: track 47.7 -> 53.8 mm, vias 2 -> 0
- net /SCL: track 200.1 -> 205.9 mm
- net /mcu/RST: track 21.1 -> 15.8 mm
- net Net-(R11-Pad1): track 0.00 -> 5.19 mm
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
Commit message: code
code
Parts:
- C14: moved to F.Cu
- R11: value R_Small_US -> 10K
- Y3: footprint vanalles:MURATA_CSTCE16M0V53C-R0 -> vanalles:MURATA_CSTLS16M0X53-B0; moved to F.Cu
- moved C14 6.02 mm to (83.2, 136.8), turned to 90 degrees
- moved Y2 5.84 mm to (126.6, 126.0)
- moved C33 5.66 mm to (122.0, 126.1)
- moved Y3 1.85 mm to (127.8, 131.8)
Routing:
- net /SDA: track 229.8 -> 237.6 mm
- net Net-(C14-Pad2): track 4.98 -> 11.6 mm, vias 1 -> 0
- net /mcu/OSC_HS_OUT: track 12.9 -> 7.57 mm, vias 1 -> 0
- net /mcu/OSC_32_OUT: track 9.84 -> 15.1 mm
- net /mcu/OSC_32_IN: track 9.71 -> 12.4 mm
- net GND: track 312.7 -> 315.3 mm
- net /mcu/OSC_HS_IN: track 10.6 -> 8.39 mm, vias 1 -> 0
- net /RX: track 55.5 -> 56.1 mm
- net /TX: track 53.8 -> 54.3 mm

Commit message: schema
schema hergetekend
Parts:
- removed BT2: Battery_Cell, vanalles:3012TR
- removed R11: 10K, vanalles:0603RL
- removed Y3: 16MHz, vanalles:MURATA_CSTLS16M0X53-B0
- U7: value STM32L552CCT6 -> STM32L052K6Tx; footprint halfgeleiders:STM32L552CCT6 -> halfgeleiders:QFP32P80_900X900X160L60X37N
- moved C33 27.2 mm to (149.0, 129.1), turned to 0 degrees
- moved C22 21.2 mm to (148.7, 135.7), turned to 0 degrees
- moved Y2 21.0 mm to (146.8, 131.8), turned to -90 degrees
- moved CON2 8.41 mm to (139.3, 126.2), turned to 180 degrees
- moved C21 7.60 mm to (143.3, 144.6)
- moved U7 5.69 mm to (136.1, 138.2), turned to 180 degrees
- moved C20 3.16 mm to (143.6, 141.7)
- moved C4 0.17 mm to (151.5, 115.0)
- moved C2 0.08 mm to (156.5, 115.0)
Connections:
- CON2 pad 6: /mcu/SWO -> unconnected-(CON2-Pad6)
- CON2 pad 8: /mcu/TDI -> unconnected-(CON2-Pad8)
- U7 pad 1: Net-(BT2-Pad1) -> +3V3
- U7 pad 10: /TX -> /CS
- U7 pad 11: /RX -> /SCK
- U7 pad 12: unconnected-(U7-Pad12) -> /MISO
- U7 pad 13: unconnected-(U7-Pad13) -> /MOSI
- U7 pad 14: /CS -> unconnected-(U7-Pad14)
- U7 pad 15: /SCK -> unconnected-(U7-Pad15)
- U7 pad 16: /MISO -> GND
- U7 pad 17: /MOSI -> +3V3
- U7 pad 18: unconnected-(U7-Pad18) -> /RESET_GPS
- U7 pad 19: unconnected-(U7-Pad19) -> /TX
- U7 pad 2: unconnected-(U7-Pad2) -> /mcu/OSC_32_IN
- U7 pad 20: unconnected-(U7-Pad20) -> /RX
- U7 pad 21: unconnected-(U7-Pad21) -> /WAKE
- U7 pad 22: unconnected-(U7-Pad22) -> /PPS
- U7 pad 23: GND -> /mcu/SWDIO
- U7 pad 24: +3V3 -> /mcu/SWDCLK
- U7 pad 26: /PPS -> unconnected-(U7-Pad26)
- U7 pad 27: /WAKE -> /INT2
- U7 pad 28: /RESET_GPS -> /INT1
- U7 pad 29: /RESET -> /SCL
- U7 pad 3: /mcu/OSC_32_IN -> /mcu/OSC_32_OUT
- U7 pad 30: /SSR -> /SDA
- U7 pad 31: /BUZZER -> GND
- U7 pad 32: /INT2 -> GND
- U7 pad 4: /mcu/OSC_32_OUT -> /mcu/RST
- U7 pad 5: /mcu/OSC_HS_IN -> +3V3
- U7 pad 6: /mcu/OSC_HS_OUT -> /BUZZER
- U7 pad 7: +3V3 -> /SSR
- U7 pad 8: GND -> unconnected-(U7-Pad8)
- U7 pad 9: +3V3 -> /RESET
Routing:
- net Net-(BT2-Pad1): track 94.4 -> 0.00 mm, vias 4 -> 0
- net /SDA: track 237.6 -> 162.2 mm, vias 10 -> 9
- net /SCL: track 205.9 -> 159.4 mm, vias 7 -> 4
- net /SSR: track 31.7 -> 69.3 mm, vias 0 -> 2
- net /RESET: track 146.2 -> 112.3 mm
- net /mcu/TDI: track 24.8 -> 0.00 mm, vias 2 -> 0
- net /TX: track 54.3 -> 73.8 mm, vias 0 -> 4
- net /mcu/SWO: track 18.6 -> 0.00 mm, vias 2 -> 0
- net /RX: track 56.1 -> 69.1 mm
- net /PPS: track 91.3 -> 78.7 mm
- net /mcu/SWDCLK: track 11.4 -> 23.9 mm, vias 0 -> 2
- net /MISO: track 48.2 -> 38.1 mm, vias 4 -> 2
- net GND: track 315.3 -> 305.8 mm, vias 40 -> 37
- net /MOSI: track 46.9 -> 38.1 mm, vias 1 -> 2
- net /mcu/OSC_HS_IN: track 8.39 -> 0.00 mm
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
Commit message: remake
remake 2 van de print
Parts:
- removed C32: 100nF, vanalles:0603
- removed CON3: jtag, connectors_user:Tag-Connect_TC2050-IDC-FP_2x05_P1.27mm_Vertical
- removed R10: 10K, vanalles:0603RL
- removed R8: 0, vanalles:0603RL
- removed U8: murattaLora, Module:XCVR_CMWX1ZZABZ-078
- added MOD1: RFM98W-433S2, Module:XCVR_RFM98W-433S2, F.Cu at (99.6, 169.9)
- R9: value 10K -> 0
- moved R9 28.8 mm to (84.5, 162.9), turned to 180 degrees
- moved C25 27.3 mm to (86.3, 166.5), turned to 180 degrees
- moved C27 24.0 mm to (86.3, 171.0), turned to 180 degrees
- moved C26 22.3 mm to (86.3, 168.9), turned to 180 degrees
- moved TP1 21.0 mm to (85.1, 146.9)
- moved R7 19.8 mm to (98.6, 150.0), turned to 0 degrees
- moved C23 6.68 mm to (87.4, 162.2)
- moved AE3 6.47 mm to (78.2, 163.1)
- moved C24 3.49 mm to (84.0, 159.3)
Connections:
- R7 pad 1: GND -> +3V3
- R7 pad 2: Net-(R7-Pad2) -> /CS
- R9 pad 1: +3V3 -> /LoRa_RFM/ANT
- R9 pad 2: /RESET -> Net-(AE3-Pad1)
Routing:
- net GND: track 305.8 -> 258.6 mm, vias 37 -> 31
- net /MISO: track 38.1 -> 73.1 mm, vias 2 -> 1
- net /RESET: track 112.3 -> 85.2 mm, vias 3 -> 4
- net /MOSI: track 38.1 -> 62.6 mm, vias 2 -> 3
- net /SCK: track 59.8 -> 80.4 mm, vias 2 -> 0
- net /CS: track 47.7 -> 66.9 mm
- net /LoRa_RFM/SWDIO: track 11.5 -> 0.00 mm, vias 2 -> 0
- net /LoRa_RFM/SWCLK: track 9.62 -> 0.00 mm
- net Net-(R7-Pad2): track 7.23 -> 0.00 mm
- net Net-(AE3-Pad1): track 5.98 -> 7.29 mm
- net /LoRa_RFM/ANT: track 7.65 -> 6.47 mm

Commit message: versie2
aan versie 2 begonnen met tekenen en code beginnen schrijven voor quadkey
Parts:
- removed AE2: Antenna_Shield, connectors_user:ufl connector
- removed C10: 4.7uF, vanalles:0603
- removed C11, C12, C15: 100nF, vanalles:0603
- removed C13: 1uF, vanalles:0603
- removed C14: 100pF, vanalles:0603
- removed C16, C19: NM, vanalles:0603
- removed C17, C18: 12pF, vanalles:0603
- removed TP1: RESET, vanalles:TestPoint_Pad_D3.0mm
- removed TP2: MOSI, vanalles:TestPoint_Pad_D3.0mm
- removed TP3: MISO, vanalles:TestPoint_Pad_D3.0mm
- removed TP4: CS, vanalles:TestPoint_Pad_D3.0mm
- removed TP5: SPICLK, vanalles:TestPoint_Pad_D3.0mm
- removed Y1: 326MhZ, vanalles:OSCCC320X250X90L80X100N
- added R10: 10K, vanalles:0603RL, F.Cu at (106.8, 127.4)
- added R11: NM, vanalles:0603RL, F.Cu at (106.8, 123.8)
- CON1: value jtag -> TAGconnect_ESP; footprint connectors_user:Tag-Connect_TC2050-IDC-FP_2x05_P1.27mm_Vertical -> connectors_user:Tag-Connect_TC2030-IDC-NL_2x03_P1.27mm_Vertical
- R6: value 0 -> 10K
- U6: value nRF52810-QFxx -> ESP32-WROOM; footprint halfgeleiders:nrf -> Module:ESP32-WROOM-32
- moved R7 34.5 mm to (116.3, 179.6), turned to 180 degrees
- moved R6 22.1 mm to (89.7, 155.2), turned to 90 degrees
- moved AE3 10.9 mm to (78.2, 174.0)
- moved C24 10.8 mm to (84.2, 170.0)
- moved MOD1 10.8 mm to (99.8, 180.7)
- moved R9 10.8 mm to (84.8, 173.7)
- moved C23 10.8 mm to (87.6, 173.0)
- moved C25 10.8 mm to (86.5, 177.3)
- moved C26 10.8 mm to (86.5, 179.6)
- moved C27 10.8 mm to (86.5, 181.7)
- moved U6 6.20 mm to (95.2, 139.4), turned to 90 degrees
- moved CON1 1.87 mm to (96.5, 123.3)
- moved J2 1.67 mm to (180.6, 153.9)
Connections:
- CON1 pad 2: /nrf/SWDIO -> /esp32/GPIO0
- CON1 pad 3: GND -> /esp32/RESET
- CON1 pad 4: /nrf/SWDCLK -> /esp32/RX
- CON1 pad 5: GND -> /esp32/TX
- CON1 pad 6: unconnected-(CON1-Pad6) -> GND
- R6 pad 1: Net-(C16-Pad1) -> +3V3
- R6 pad 2: Net-(AE2-Pad1) -> /esp32/RESET
- U6 pad 1: Net-(C15-Pad2) -> GND
- U6 pad 10: /SDA -> unconnected-(U6-Pad10)
- U6 pad 13: +3V3 -> unconnected-(U6-Pad13)
- U6 pad 15: unconnected-(U6-Pad15) -> GND
- U6 pad 2: unconnected-(U6-Pad2) -> +3V3
- U6 pad 24: /nrf/RST -> unconnected-(U6-Pad24)
- U6 pad 25: /nrf/SWDCLK -> /esp32/GPIO0
- U6 pad 26: /nrf/SWDIO -> unconnected-(U6-Pad26)
- U6 pad 3: unconnected-(U6-Pad3) -> /esp32/RESET
- U6 pad 30: Net-(C16-Pad1) -> unconnected-(U6-Pad30)
- U6 pad 31: GND -> unconnected-(U6-Pad31)
- U6 pad 32: GND -> unconnected-(U6-Pad32)
- U6 pad 33: Net-(C14-Pad2) -> /SDA
- U6 pad 34: Net-(C17-Pad1) -> /esp32/RX
- U6 pad 35: Net-(C18-Pad1) -> /esp32/TX
- U6 pad 36: +3V3 -> /SCL
- U6 pad 38: unconnected-(U6-Pad38) -> GND
- U6 pad 39: unconnected-(U6-Pad39) -> GND
- U6 pad 9: /SCL -> unconnected-(U6-Pad9)
Routing:
- net /SCL: track 159.4 -> 246.6 mm
- net /SDA: track 162.2 -> 245.6 mm
- net /esp32/RESET: track 0.00 -> 41.4 mm, vias 0 -> 2
- net GND: track 258.6 -> 229.4 mm, vias 31 -> 24
- net /esp32/GPIO0: track 0.00 -> 27.0 mm
- net /RESET: track 85.2 -> 61.4 mm, vias 4 -> 0
- net /nrf/RST: track 18.0 -> 0.00 mm, vias 2 -> 0
- net /SCK: track 80.4 -> 65.7 mm
- net /nrf/SWDIO: track 13.4 -> 0.00 mm
- net /esp32/RX: track 0.00 -> 13.2 mm, vias 0 -> 2
- net /nrf/SWDCLK: track 12.9 -> 0.00 mm
- net /esp32/TX: track 0.00 -> 12.6 mm
- net Net-(C14-Pad2): track 11.6 -> 0.00 mm
- net Net-(C17-Pad1): track 10.4 -> 0.00 mm
- net Net-(C18-Pad1): track 8.35 -> 0.00 mm
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