File: pcb/asset tracker LoRa/LoRa tracker/LoRa tracker.kicad_sch (KiCad schematic)
At the start: 0 parts

Commit message: 34t
34t
Parts:
- added AE3: Antenna_Shield, connectors_user:sma_right angeld, symbol Device:Antenna_Shield
- added C23, C24: NM, vanalles:0603, symbol Device:C_Small
- added R8: 0, vanalles:0603RL, symbol Device:R_Small_US
Connections:
- new net: AE3.1 (A), C24.1, R8.2
- new net GND: AE3.2 (Shield), C23.2, C24.2
- new net LoRa_RFM/ANT_RFM: C23.1, R8.1
Other:
- added sheet IO (IO.kicad_sch)
- added sheet LoRa_RFM (LoRa_RFM.kicad_sch)
- added sheet beweging (beweging.kicad_sch)
- added sheet gps (gps.kicad_sch)
- added sheet mcu (mcu.kicad_sch)
- added sheet nrf (nrf.kicad_sch)
- added sheet voeding (voeding.kicad_sch)
