File: pcb/asset tracker LoRa/LoRa tracker/LoRa tracker.kicad_sch (KiCad schematic)
At the start: 4 parts

Commit message: pcb kastje
pcb in kastje getekend
Parts:
- AE3: footprint connectors_user:sma_right angeld -> connectors_user:sma juist
Connections:
- net LoRa_RFM/ANT_RFM renamed LoRa_RFM/ANT
Other:
- sheet IO ports: added SCL_CRYPTO, SDA_CRYPTO; removed none
- sheet LoRa_RFM ports: added ANT, CLK, CS, MISO, MOSI, RESET; removed ANT_RFM, CS_RFM, IRQ_RFM, MISO_RFM, MOSI_RFM, RESET_RFM, SCK_RFM
- sheet mcu ports: added MISO_MURATTA_MCU, MOSI_MURATTA_MCU, RESET_MURATTA_MCU, SCK_MURATTA_MCU; removed IRQ_RFM_MCU, MISO_RFM_MCU, MOSI_RFM_MCU, RESET_RFM_MCU, SCK_RFM_MCU

Commit message: lora tracker
lora tracker afgemaakt
Parts:
- added TP1: RESET, vanalles:TestPoint_Pad_D3.0mm, symbol Connector:Test_Point
- added TP2: MOSI, vanalles:TestPoint_Pad_D3.0mm, symbol Connector:Test_Point
- added TP3: MISO, vanalles:TestPoint_Pad_D3.0mm, symbol Connector:Test_Point
- added TP4: CS, vanalles:TestPoint_Pad_D3.0mm, symbol Connector:Test_Point
- added TP5: SPICLK, vanalles:TestPoint_Pad_D3.0mm, symbol Connector:Test_Point
- AE3: footprint connectors_user:sma juist -> connectors_user:ufl connector
Connections:
- net CS: now also TP4.1
- net MISO: now also TP3.1
- net MOSI: now also TP2.1
- net RESET: now also TP1.1
- net SCK: now also TP5.1
Changed lines of the file:
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@@
+    (stroke (width 0.1524) (type solid) (color 0 0 0 0))
+  )
+  (bus_entry (at 90.17 158.75) (size 2.54 -2.54)
+    (stroke (width 0.1524) (type solid) (color 0 0 0 0))
+  )
+  (bus_entry (at 104.14 158.75) (size 2.54 -2.54)
+    (stroke (width 0.1524) (type solid) (color 0 0 0 0))
+  )
+  (bus_entry (at 121.92 158.75) (size 2.54 -2.54)
+    (stroke (width 0.1524) (type solid) (color 0 0 0 0))
+  )
+  (bus_entry (at 134.62 158.75) (size 2.54 -2.54)
+    (stroke (width 0.1524) (type solid) (color 0 0 0 0))
+  )
+  (bus_entry (at 144.78 158.75) (size 2.54 -2.54)
     (stroke (width 0.1524) (type solid) (color 0 0 0 0))
   )
@@
     (stroke (width 0) (type solid) (color 0 0 0 0))
   )
+  (wire (pts (xy 90.17 158.75) (xy 90.17 165.1))
+    (stroke (width 0) (type solid) (color 0 0 0 0))
+  )
+  (wire (pts (xy 104.14 158.75) (xy 104.14 165.1))
+    (stroke (width 0) (type solid) (color 0 0 0 0))
+  )
+  (wire (pts (xy 121.92 158.75) (xy 121.92 165.1))
+    (stroke (width 0) (type solid) (color 0 0 0 0))
+  )
+  (wire (pts (xy 134.62 158.75) (xy 134.62 165.1))
+    (stroke (width 0) (type solid) (color 0 0 0 0))
+  )
+  (wire (pts (xy 144.78 158.75) (xy 144.78 165.1))
+    (stroke (width 0) (type solid) (color 0 0 0 0))
+  )
   (wire (pts (xy 154.94 57.15) (xy 179.07 57.15))
     (stroke (width 0) (type solid) (color 0 0 0 0))
@@
     (effects (font (size 1.27 1.27)) (justify right bottom))
   )
+  (label "RESET" (at 90.17 160.02 270)
+    (effects (font (size 1.27 1.27)) (justify right bottom))
+  )
   (label "INT1" (at 96.52 54.61 180)
     (effects (font (size 1.27 1.27)) (justify right bottom))
@@
   )
   (label "RESET" (at 99.06 36.83 180)
+    (effects (font (size 1.27 1.27)) (justify right bottom))
+  )
+  (label "MOSI" (at 104.14 160.02 270)
+    (effects (font (size 1.27 1.27)) (justify right bottom))
+  )
+  (label "MISO" (at 121.92 160.02 270)
+    (effects (font (size 1.27 1.27)) (justify right bottom))
+  )
+  (label "CS" (at 134.62 161.29 270)
+    (effects (font (size 1.27 1.27)) (justify right bottom))
+  )
+  (label "SCK" (at 144.78 160.02 270)
     (effects (font (size 1.27 1.27)) (justify right bottom))
   )
@@
   (label "RESET_GPS" (at 194.31 57.15 180)
     (effects (font (size 1.27 1.27)) (justify right bottom))
+  )
+  (symbol (lib_id "Connector:Test_Point") (at 90.17 165.1 180) (unit 1)
+    (in_bom yes) (on_board yes) (fields_autoplaced)
+    (property "Reference" "TP1" (id 0) (at 92.71 166.3064 0)
+      (effects (font (size 1.27 1.27)) (justify right))
+    )
+    (property "Value" "RESET" (id 1) (at 92.71 168.8464 0)
+      (effects (font (size 1.27 1.27)) (justify right))
+    )
+    (property "Footprint" "vanalles:TestPoint_Pad_D3.0mm" (id 2) (at 85.09 165.1 0)
+      (effects (font (size 1.27 1.27)) hide)
+    )
+    (property "Datasheet" "" (id 3) (at 85.09 165.1 0)
+      (effects (font (size 1.27 1.27)) hide)
+    )
+    (pin "1")
+  )
+  (symbol (lib_id "Connector:Test_Point") (at 104.14 165.1 180) (unit 1)
+    (in_bom yes) (on_board yes) (fields_autoplaced)
+    (property "Reference" "TP2" (id 0) (at 106.68 166.3064 0)
+      (effects (font (size 1.27 1.27)) (justify right))
+    )
+    (property "Value" "MOSI" (id 1) (at 106.68 168.8464 0)
+      (effects (font (size 1.27 1.27)) (justify right))
+    )
+    (property "Footprint" "vanalles:TestPoint_Pad_D3.0mm" (id 2) (at 99.06 165.1 0)
+      (effects (font (size 1.27 1.27)) hide)
+    )
+    (property "Datasheet" "" (id 3) (at 99.06 165.1 0)
+      (effects (font (size 1.27 1.27)) hide)
+    )
+    (pin "1")
+  )
+  (symbol (lib_id "Connector:Test_Point") (at 121.92 165.1 180) (unit 1)
+    (in_bom yes) (on_board yes) (fields_autoplaced)
+    (property "Reference" "TP3" (id 0) (at 124.46 166.3064 0)
+      (effects (font (size 1.27 1.27)) (justify right))
+    )
+    (property "Value" "MISO" (id 1) (at 124.46 168.8464 0)
+      (effects (font (size 1.27 1.27)) (justify right))
+    )
+    (property "Footprint" "vanalles:TestPoint_Pad_D3.0mm" (id 2) (at 116.84 165.1 0)
+      (effects (font (size 1.27 1.27)) hide)
+    )
+    (property "Datasheet" "" (id 3) (at 116.84 165.1 0)
+      (effects (font (size 1.27 1.27)) hide)
+    )
+    (pin "1")
+  )
+  (symbol (lib_id "Connector:Test_Point") (at 134.62 165.1 180) (unit 1)
+    (in_bom yes) (on_board yes) (fields_autoplaced)
+    (property "Reference" "TP4" (id 0) (at 137.16 166.3064 0)
+      (effects (font (size 1.27 1.27)) (justify right))
+    )
+    (property "Value" "CS" (id 1) (at 137.16 168.8464 0)
+      (effects (font (size 1.27 1.27)) (justify right))
+    )
+    (property "Footprint" "vanalles:TestPoint_Pad_D3.0mm" (id 2) (at 129.54 165.1 0)
+      (effects (font (size 1.27 1.27)) hide)
+    )
+    (property "Datasheet" "" (id 3) (at 129.54 165.1 0)
+      (effects (font (size 1.27 1.27)) hide)
+    )
+    (pin "1")
+  )
+  (symbol (lib_id "Connector:Test_Point") (at 144.78 165.1 180) (unit 1)
+    (in_bom yes) (on_board yes) (fields_autoplaced)
+    (property "Reference" "TP5" (id 0) (at 147.32 166.3064 0)
+      (effects (font (size 1.27 1.27)) (justify right))
+    )
+    (property "Value" "SPICLK" (id 1) (at 147.32 168.8464 0)
+      (effects (font (size 1.27 1.27)) (justify right))
+    )
+    (property "Footprint" "vanalles:TestPoint_Pad_D3.0mm" (id 2) (at 139.7 165.1 0)
+      (effects (font (size 1.27 1.27)) hide)
+    )
+    (property "Datasheet" "" (id 3) (at 139.7 165.1 0)
+      (effects (font (size 1.27 1.27)) hide)
+    )
+    (pin "1")
   )
   (symbol (lib_id "power:GND") (at 229.87 106.68 0) (unit 1)
@@
       (effects (font (size 1.27 1.27)) (justify left))
     )
-    (property "Footprint" "connectors_user:sma juist" (id 2) (at 274.32 101.6 0)
+    (property "Footprint" "connectors_user:ufl connector" (id 2) (at 274.32 101.6 0)
       (effects (font (size 1.27 1.27)) hide)
     )
@@
     )
     (path "/a54f423a-4358-497d-987f-745572e8f098/9e80dceb-6694-4b1a-af59-7381ae389295"
-      (reference "AE1") (unit 1) (value "sma") (footprint "connectors_user:sma juist")
+      (reference "AE1") (unit 1) (value "sma") (footprint "connectors_user:ufl connector")
     )
     (path "/5db711ae-0233-4ac0-a3c6-f143c625478c/b63a08fb-3ec1-4e6d-afcf-9ed6da4e9c91"
-      (reference "AE2") (unit 1) (value "Antenna_Shield") (footprint "connectors_user:sma juist")
+      (reference "AE2") (unit 1) (value "Antenna_Shield") (footprint "connectors_user:ufl connector")
     )
     (path "/91ce9766-a8a1-4c23-8f2b-fba906e4dbc2"
-      (reference "AE3") (unit 1) (value "Antenna_Shield") (footprint "connectors_user:sma juist")
+      (reference "AE3") (unit 1) (value "Antenna_Shield") (footprint "connectors_user:ufl connector")
     )
     (path "/a54f423a-4358-497d-987f-745572e8f098/0404f810-c943-49da-8783-0e33aefd54c5"
@@
       (reference "R9") (unit 1) (value "10K") (footprint "vanalles:0603RL")
     )
+    (path "/c700dc30-dbea-4934-a0d3-e9dc42835f75"
+      (reference "TP1") (unit 1) (value "RESET") (footprint "vanalles:TestPoint_Pad_D3.0mm")
+    )
+    (path "/d54192be-7abe-4eac-ac5b-4c02699c11a7"
+      (reference "TP2") (unit 1) (value "MOSI") (footprint "vanalles:TestPoint_Pad_D3.0mm")
+    )
+    (path "/8e4300a0-1cd7-4ca2-9bb0-94ecae19bbfb"
+      (reference "TP3") (unit 1) (value "MISO") (footprint "vanalles:TestPoint_Pad_D3.0mm")
+    )
+    (path "/cc919938-2c5c-4483-8a72-cbe1d3c0d2a1"
+      (reference "TP4") (unit 1) (value "CS") (footprint "vanalles:TestPoint_Pad_D3.0mm")
+    )
+    (path "/5a18b7db-664f-427d-8c1c-d045efcc0022"
+      (reference "TP5") (unit 1) (value "SPICLK") (footprint "vanalles:TestPoint_Pad_D3.0mm")
+    )
     (path "/6004ef5c-d3d2-40e4-b9e6-92f5cd630dc1/90b5f417-7acf-48d5-b5b2-d8a1cbc84cc1"
       (reference "U1") (unit 1) (value "INA219BxDCN") (footprint "halfgeleiders:SOIC127P599X175-8N")
@@
     )
     (path "/0e73f55d-2435-4bae-aa12-8b99ef7d3bab/24ff0685-6993-43a2-9027-c3ffa970ef01"
-      (reference "U7") (unit 1) (value "ATSAMD21G18A-M") (footprint "halfgeleiders:QFN50P700X700X90-49N")
+      (reference "U7") (unit 1) (value "ATSAMD21G18A-M") (footprint "halfgeleiders:ATSAMD21G18A-M")
     )
     (path "/4254a827-1935-476e-a2a2-5bc9aad7b66e/dfe86e24-0d47-490d-9999-e9ab36f17359"

Commit message: schema
schema hergetekend
Other:
- sheet mcu ports: added CS_MURATTA_MCU; removed CS_RFM
Changed lines of the file:
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@@
-      (effects (font (size 1.27 1.27)) (justify left))
-    )
-    (pin "CS_RFM" input (at 101.6 39.37 180)
       (effects (font (size 1.27 1.27)) (justify left))
     )
@@
     )
     (pin "MISO_MURATTA_MCU" input (at 101.6 41.91 180)
+      (effects (font (size 1.27 1.27)) (justify left))
+    )
+    (pin "CS_MURATTA_MCU" input (at 101.6 39.37 180)
       (effects (font (size 1.27 1.27)) (justify left))
     )
@@
       (reference "#PWR0141") (unit 1) (value "GND") (footprint "")
     )
-    (path "/0e73f55d-2435-4bae-aa12-8b99ef7d3bab/21aad396-c774-4f52-9d2c-6cd8c140641f"
-      (reference "#PWR0142") (unit 1) (value "GND") (footprint "")
+    (path "/0e73f55d-2435-4bae-aa12-8b99ef7d3bab/70c7d6d2-ab66-4b71-94c2-a64229f88028"
+      (reference "#PWR0142") (unit 1) (value "+3V3") (footprint "")
     )
     (path "/0e73f55d-2435-4bae-aa12-8b99ef7d3bab/1fe4dfd1-9523-4d33-a689-b41d6da1743a"
@@
       (reference "#PWR0149") (unit 1) (value "GND") (footprint "")
     )
-    (path "/0e73f55d-2435-4bae-aa12-8b99ef7d3bab/59c2d1fe-6723-4658-9507-e6af2d3e727f"
+    (path "/0e73f55d-2435-4bae-aa12-8b99ef7d3bab/5c715b41-4086-4c03-81fb-fad9f3e26686"
       (reference "#PWR0150") (unit 1) (value "GND") (footprint "")
     )
-    (path "/0e73f55d-2435-4bae-aa12-8b99ef7d3bab/4f73f405-b56a-4a4b-af61-11ac78d78a10"
+    (path "/0e73f55d-2435-4bae-aa12-8b99ef7d3bab/a80b3b84-7bcf-408c-aaa2-8676f5aeb766"
       (reference "#PWR0151") (unit 1) (value "GND") (footprint "")
     )
@@
       (reference "#PWR0161") (unit 1) (value "+3V3") (footprint "")
     )
-    (path "/0e73f55d-2435-4bae-aa12-8b99ef7d3bab/c57d6533-6b88-4466-bd3d-60b51a42d875"
-      (reference "#PWR0162") (unit 1) (value "GND") (footprint "")
-    )
-    (path "/0e73f55d-2435-4bae-aa12-8b99ef7d3bab/dc6fcd63-cbc4-49a3-a50b-73c1425bde64"
-      (reference "#PWR0163") (unit 1) (value "+3V3") (footprint "")
-    )
     (path "/0e73f55d-2435-4bae-aa12-8b99ef7d3bab/d2a6bcbb-8d4d-4a61-a7f7-09c4459a3fc4"
       (reference "#PWR0164") (unit 1) (value "+3V3") (footprint "")
@@
       (reference "BT1") (unit 1) (value "Battery_Cell") (footprint "vanalles:3012TR")
     )
-    (path "/0e73f55d-2435-4bae-aa12-8b99ef7d3bab/cdf00e59-de2a-482a-bc02-5c5a6fae4913"
-      (reference "BT2") (unit 1) (value "Battery_Cell") (footprint "vanalles:3012TR")
-    )
     (path "/6004ef5c-d3d2-40e4-b9e6-92f5cd630dc1/e7a1ddd4-8cd9-4658-b33f-bf697e63c769"
       (reference "C1") (unit 1) (value "100nF") (footprint "vanalles:0603")
@@
       (reference "R10") (unit 1) (value "10K") (footprint "vanalles:0603RL")
     )
-    (path "/0e73f55d-2435-4bae-aa12-8b99ef7d3bab/081080c3-a9b9-4cc6-8433-a9fae302bf2c"
-      (reference "R11") (unit 1) (value "10K") (footprint "vanalles:0603RL")
-    )
     (path "/c700dc30-dbea-4934-a0d3-e9dc42835f75"
       (reference "TP1") (unit 1) (value "RESET") (footprint "vanalles:TestPoint_Pad_D3.0mm")
@@
       (reference "U6") (unit 1) (value "nRF52810-QFxx") (footprint "halfgeleiders:nrf")
     )
-    (path "/0e73f55d-2435-4bae-aa12-8b99ef7d3bab/754059c8-d9e6-40fb-9d9e-f281aaf87bef"
-      (reference "U7") (unit 1) (value "STM32L552CCT6") (footprint "halfgeleiders:STM32L552CCT6")
-    )
-    (path "/0e73f55d-2435-4bae-aa12-8b99ef7d3bab/130cfecf-a3cb-4013-bd22-12c2267d4d7c"
-      (reference "U7") (unit 2) (value "STM32L552CCT6") (footprint "halfgeleiders:STM32L552CCT6")
+    (path "/0e73f55d-2435-4bae-aa12-8b99ef7d3bab/db47ca84-9ec8-4540-84e7-2b3da2184c1e"
+      (reference "U7") (unit 1) (value "STM32L052K6Tx") (footprint "halfgeleiders:QFP32P80_900X900X160L60X37N")
     )
     (path "/4254a827-1935-476e-a2a2-5bc9aad7b66e/dfe86e24-0d47-490d-9999-e9ab36f17359"
@@
       (reference "Y2") (unit 1) (value "32khz") (footprint "vanalles:crystal tht")
     )
-    (path "/0e73f55d-2435-4bae-aa12-8b99ef7d3bab/a419fcc8-3b3a-41c7-85c8-70a69bb868ce"
-      (reference "Y3") (unit 1) (value "16MHz") (footprint "vanalles:MURATA_CSTLS16M0X53-B0")
-    )
   )

Commit message: remake
remake 2 van de print
Parts:
- removed R8: 0, vanalles:0603RL, symbol Device:R_Small_US
- added R9: 0, vanalles:0603RL, symbol Device:R_Small_US
Connections:
- net LoRa_RFM/ANT: now also R9.1
- net at AE3.1 (A), C24.1: now also R9.2
Other:
- moved on the sheet: C23
Changed lines of the file:
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@@
 (kicad_sch (version 20210406) (generator eeschema)
   (paper "A4")
-  (junction (at 229.87 101.6) (diameter 0.9144) (color 0 0 0 0))
+  (junction (at 238.76 101.6) (diameter 0.9144) (color 0 0 0 0))
   (junction (at 257.81 101.6) (diameter 0.9144) (color 0 0 0 0))
   (bus_entry (at 78.74 44.45) (size 2.54 2.54)
@@
     (stroke (width 0) (type solid) (color 0 0 0 0))
   )
-  (wire (pts (xy 219.71 101.6) (xy 229.87 101.6))
-    (stroke (width 0) (type solid) (color 0 0 0 0))
-  )
-  (wire (pts (xy 229.87 101.6) (xy 242.57 101.6))
+  (wire (pts (xy 219.71 101.6) (xy 238.76 101.6))
+    (stroke (width 0) (type solid) (color 0 0 0 0))
+  )
+  (wire (pts (xy 238.76 101.6) (xy 242.57 101.6))
+    (stroke (width 0) (type solid) (color 0 0 0 0))
+  )
+  (wire (pts (xy 238.76 102.87) (xy 238.76 101.6))
     (stroke (width 0) (type solid) (color 0 0 0 0))
   )
@@
     (pin "1")
   )
-  (symbol (lib_id "power:GND") (at 229.87 106.68 0) (unit 1)
+  (symbol (lib_id "power:GND") (at 238.76 107.95 0) (unit 1)
     (in_bom yes) (on_board yes) (fields_autoplaced)
-    (property "Reference" "#PWR0147" (id 0) (at 229.87 113.03 0)
-      (effects (font (size 1.27 1.27)) hide)
-    )
-    (property "Value" "GND" (id 1) (at 229.87 111.76 0))
-    (property "Footprint" "" (id 2) (at 229.87 106.68 0)
-      (effects (font (size 1.27 1.27)) hide)
-    )
-    (property "Datasheet" "" (id 3) (at 229.87 106.68 0)
+    (property "Reference" "#PWR0147" (id 0) (at 238.76 114.3 0)
+      (effects (font (size 1.27 1.27)) hide)
+    )
+    (property "Value" "GND" (id 1) (at 238.76 113.03 0))
+    (property "Footprint" "" (id 2) (at 238.76 107.95 0)
+      (effects (font (size 1.27 1.27)) hide)
+    )
+    (property "Datasheet" "" (id 3) (at 238.76 107.95 0)
       (effects (font (size 1.27 1.27)) hide)
     )
@@
   (symbol (lib_id "Device:R_Small_US") (at 245.11 101.6 90) (unit 1)
     (in_bom yes) (on_board yes) (fields_autoplaced)
-    (property "Reference" "R8" (id 0) (at 245.11 96.52 90))
+    (property "Reference" "R9" (id 0) (at 245.11 96.52 90))
     (property "Value" "0" (id 1) (at 245.11 99.06 90))
     (property "Footprint" "vanalles:0603RL" (id 2) (at 245.11 101.6 0)
@@
     (pin "2")
   )
-  (symbol (lib_id "Device:C_Small") (at 229.87 104.14 0) (unit 1)
+  (symbol (lib_id "Device:C_Small") (at 238.76 105.41 0) (unit 1)
     (in_bom yes) (on_board yes) (fields_autoplaced)
-    (property "Reference" "C23" (id 0) (at 232.41 103.5049 0)
-      (effects (font (size 1.27 1.27)) (justify left))
-    )
-    (property "Value" "NM" (id 1) (at 232.41 106.0449 0)
-      (effects (font (size 1.27 1.27)) (justify left))
-    )
-    (property "Footprint" "vanalles:0603" (id 2) (at 229.87 104.14 0)
-      (effects (font (size 1.27 1.27)) hide)
-    )
-    (property "Datasheet" "~" (id 3) (at 229.87 104.14 0)
+    (property "Reference" "C23" (id 0) (at 241.3 104.7749 0)
+      (effects (font (size 1.27 1.27)) (justify left))
+    )
+    (property "Value" "NM" (id 1) (at 241.3 107.3149 0)
+      (effects (font (size 1.27 1.27)) (justify left))
+    )
+    (property "Footprint" "vanalles:0603" (id 2) (at 238.76 105.41 0)
+      (effects (font (size 1.27 1.27)) hide)
+    )
+    (property "Datasheet" "~" (id 3) (at 238.76 105.41 0)
       (effects (font (size 1.27 1.27)) hide)
     )
@@
       (reference "#PWR0143") (unit 1) (value "+3V3") (footprint "")
     )
-    (path "/4254a827-1935-476e-a2a2-5bc9aad7b66e/3428b2f6-724e-4c88-9882-e4487f329389"
-      (reference "#PWR0144") (unit 1) (value "GND") (footprint "")
-    )
-    (path "/4254a827-1935-476e-a2a2-5bc9aad7b66e/f27529a1-d88e-44bd-ac7b-91b720bd496f"
-      (reference "#PWR0145") (unit 1) (value "GND") (footprint "")
+    (path "/4254a827-1935-476e-a2a2-5bc9aad7b66e/7173777a-dd27-4b89-ae5d-6f69a21406c7"
+      (reference "#PWR0144") (unit 1) (value "+3V3") (footprint "")
     )
     (path "/4254a827-1935-476e-a2a2-5bc9aad7b66e/ea4b0a2f-2263-4ff3-b5e6-b8c309dda5a8"
@@
       (reference "#PWR0153") (unit 1) (value "GND") (footprint "")
     )
-    (path "/4254a827-1935-476e-a2a2-5bc9aad7b66e/3d6e69fd-edfb-4ecc-aca6-e37f723a8ddb"
-      (reference "#PWR0154") (unit 1) (value "+3V3") (footprint "")
-    )
     (path "/e23b1c3a-d6da-4307-9d87-0a5b67e1dee3/0dcab7b7-0cef-4818-9ef6-5275f720475e"
       (reference "#PWR0155") (unit 1) (value "GND") (footprint "")
@@
       (reference "#PWR0156") (unit 1) (value "+3V3") (footprint "")
     )
-    (path "/4254a827-1935-476e-a2a2-5bc9aad7b66e/dfbdc4c4-7866-4ffb-907e-5da1be3481ce"
-      (reference "#PWR0157") (unit 1) (value "+3V3") (footprint "")
-    )
-    (path "/4254a827-1935-476e-a2a2-5bc9aad7b66e/61649430-2b86-438f-9fe9-817644df44c4"
-      (reference "#PWR0158") (unit 1) (value "GND") (footprint "")
-    )
     (path "/0e73f55d-2435-4bae-aa12-8b99ef7d3bab/c9f4c330-92c4-4f99-8d89-78eead35cbce"
       (reference "#PWR0159") (unit 1) (value "GND") (footprint "")
@@
       (reference "#PWR0160") (unit 1) (value "GND") (footprint "")
     )
-    (path "/4254a827-1935-476e-a2a2-5bc9aad7b66e/908d0b81-bcb1-4e2a-8649-824b3329d4fe"
-      (reference "#PWR0161") (unit 1) (value "+3V3") (footprint "")
-    )
     (path "/0e73f55d-2435-4bae-aa12-8b99ef7d3bab/d2a6bcbb-8d4d-4a61-a7f7-09c4459a3fc4"
       (reference "#PWR0164") (unit 1) (value "+3V3") (footprint "")
@@
       (reference "C31") (unit 1) (value "10uF") (footprint "vanalles:0603")
     )
-    (path "/4254a827-1935-476e-a2a2-5bc9aad7b66e/fe587090-c20e-4c83-8356-fafe18fdaaf1"
-      (reference "C32") (unit 1) (value "100nF") (footprint "vanalles:0603")
-    )
     (path "/0e73f55d-2435-4bae-aa12-8b99ef7d3bab/d5bd3ff6-11cb-475f-9b94-b5a55d9b1db8"
       (reference "C33") (unit 1) (value "6.8pF") (footprint "vanalles:0603")
@@
       (reference "CON2") (unit 1) (value "jtag") (footprint "connectors_user:Tag-Connect_TC2050-IDC-FP_2x05_P1.27mm_Vertical")
     )
-    (path "/4254a827-1935-476e-a2a2-5bc9aad7b66e/9ea914a3-59b6-4d8b-a79b-a9c1170770bc"
-      (reference "CON3") (unit 1) (value "jtag") (footprint "connectors_user:Tag-Connect_TC2050-IDC-FP_2x05_P1.27mm_Vertical")
-    )
     (path "/6004ef5c-d3d2-40e4-b9e6-92f5cd630dc1/902dd638-c938-443d-9b44-9b478811d50f"
       (reference "J1") (unit 1) (value "Screw_Terminal_01x02") (footprint "connectors_user:2pin_screw")
@@
       (reference "L1") (unit 1) (value "5n6") (footprint "vanalles:0603")
     )
+    (path "/4254a827-1935-476e-a2a2-5bc9aad7b66e/ad49f2b8-9542-40ee-af29-5786fdcf34aa"
+      (reference "MOD1") (unit 1) (value "RFM98W-433S2") (footprint "Module:XCVR_RFM98W-433S2")
+    )
     (path "/a54f423a-4358-497d-987f-745572e8f098/09043f9f-c828-4bfb-b25a-116b174eefa1"
       (reference "MOD2") (unit 1) (value "teseo-LIV") (footprint "Module:SON_STM_TESEO-LIV3R")
@@
       (reference "R6") (unit 1) (value "0") (footprint "vanalles:0603RL")
     )
-    (path "/4254a827-1935-476e-a2a2-5bc9aad7b66e/3610d572-7658-46fb-a9d3-ffdf0013e981"
+    (path "/4254a827-1935-476e-a2a2-5bc9aad7b66e/8fc5ad05-a0bf-405e-95ac-4ebb219e2698"
       (reference "R7") (unit 1) (value "10K") (footprint "vanalles:0603RL")
     )
-    (path "/976b5c5f-a004-44fb-a8d1-0822100485a4"
-      (reference "R8") (unit 1) (value "0") (footprint "vanalles:0603RL")
-    )
-    (path "/4254a827-1935-476e-a2a2-5bc9aad7b66e/12c0e371-df36-4b59-ba57-12a83e977978"
-      (reference "R9") (unit 1) (value "10K") (footprint "vanalles:0603RL")
-    )
-    (path "/4254a827-1935-476e-a2a2-5bc9aad7b66e/3c42c2c2-d3ee-4d28-90c5-e041c4eec4f0"
-      (reference "R10") (unit 1) (value "10K") (footprint "vanalles:0603RL")
+    (path "/125c6828-29cc-4b48-9d1d-f055334d5a6f"
+      (reference "R9") (unit 1) (value "0") (footprint "vanalles:0603RL")
     )
     (path "/c700dc30-dbea-4934-a0d3-e9dc42835f75"
@@
       (reference "U7") (unit 1) (value "STM32L052K6Tx") (footprint "halfgeleiders:QFP32P80_900X900X160L60X37N")
     )
-    (path "/4254a827-1935-476e-a2a2-5bc9aad7b66e/dfe86e24-0d47-490d-9999-e9ab36f17359"
-      (reference "U8") (unit 1) (value "murattaLora") (footprint "Module:XCVR_CMWX1ZZABZ-078")
-    )
     (path "/e23b1c3a-d6da-4307-9d87-0a5b67e1dee3/55d07bbb-2ef2-4b66-bac7-29180ecc208d"
