File: pcb/asset tracker LoRa/LoRa tracker/nrf.kicad_sch (KiCad schematic)
At the start: 15 parts, among them CON1 jtag, U6 nRF52810-QFxx, Y1 326MhZ

Commit message: pcb kastje
pcb in kastje getekend
Parts:
- removed AE2: Antenna, vanalles:Texas_SWRA117D_2.4GHz_Right, symbol Device:Antenna
- added AE2: Antenna_Shield, connectors_user:sma juist, symbol Device:Antenna_Shield
Connections:
- net GND: now also AE2.2 (Shield)
- net at C19.1, R6.2: now also AE2.1 (A)
Changed lines of the file:
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@@
+    (stroke (width 0) (type solid) (color 0 0 0 0))
+  )
+  (wire (pts (xy 222.25 71.12) (xy 222.25 78.74))
     (stroke (width 0) (type solid) (color 0 0 0 0))
   )
@@
     )
     (property "Datasheet" "" (id 3) (at 198.12 73.66 0)
+      (effects (font (size 1.27 1.27)) hide)
+    )
+    (pin "1")
+  )
+  (symbol (lib_id "power:GND") (at 222.25 78.74 0) (unit 1)
+    (in_bom yes) (on_board yes) (fields_autoplaced)
+    (property "Reference" "#PWR0160" (id 0) (at 222.25 85.09 0)
+      (effects (font (size 1.27 1.27)) hide)
+    )
+    (property "Value" "GND" (id 1) (at 222.25 83.82 0))
+    (property "Footprint" "" (id 2) (at 222.25 78.74 0)
+      (effects (font (size 1.27 1.27)) hide)
+    )
+    (property "Datasheet" "" (id 3) (at 222.25 78.74 0)
       (effects (font (size 1.27 1.27)) hide)
     )
@@
     (pin "2")
   )
-  (symbol (lib_id "Device:Antenna") (at 227.33 68.58 270) (unit 1)
-    (in_bom yes) (on_board yes) (fields_autoplaced)
-    (property "Reference" "AE2" (id 0) (at 231.14 67.9449 90)
-      (effects (font (size 1.27 1.27)) (justify left))
-    )
-    (property "Value" "Antenna" (id 1) (at 231.14 70.4849 90)
-      (effects (font (size 1.27 1.27)) (justify left))
-    )
-    (property "Footprint" "vanalles:Texas_SWRA117D_2.4GHz_Right" (id 2) (at 227.33 68.58 0)
-      (effects (font (size 1.27 1.27)) hide)
-    )
-    (property "Datasheet" "~" (id 3) (at 227.33 68.58 0)
-      (effects (font (size 1.27 1.27)) hide)
-    )
-    (pin "1")
+  (symbol (lib_id "Device:Antenna_Shield") (at 227.33 68.58 270) (unit 1)
+    (in_bom yes) (on_board yes) (fields_autoplaced)
+    (property "Reference" "AE2" (id 0) (at 233.68 68.7069 90)
+      (effects (font (size 1.27 1.27)) (justify left))
+    )
+    (property "Value" "Antenna_Shield" (id 1) (at 233.68 71.2469 90)
+      (effects (font (size 1.27 1.27)) (justify left))
+    )
+    (property "Footprint" "connectors_user:sma juist" (id 2) (at 229.87 68.58 0)
+      (effects (font (size 1.27 1.27)) hide)
+    )
+    (property "Datasheet" "~" (id 3) (at 229.87 68.58 0)
+      (effects (font (size 1.27 1.27)) hide)
+    )
+    (pin "1")
+    (pin "2")
   )
   (symbol (lib_id "Device:Crystal_GND24") (at 161.29 92.71 90) (unit 1)

Commit message: lora tracker
lora tracker afgemaakt
Parts:
- AE2: footprint connectors_user:sma juist -> connectors_user:ufl connector
Changed lines of the file:
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@@
       (effects (font (size 1.27 1.27)) (justify left))
     )
-    (property "Footprint" "connectors_user:sma juist" (id 2) (at 229.87 68.58 0)
+    (property "Footprint" "connectors_user:ufl connector" (id 2) (at 229.87 68.58 0)
       (effects (font (size 1.27 1.27)) hide)
     )
