File: pcb/asset tracker LoRa/LoRa tracker/LoRa_RFM.kicad_sch (KiCad schematic)
At the start: 5 parts

Commit message: fgnhb
fgdh
Parts:
- U: renamed from C26; value 1uF -> (none); footprint vanalles:0603 -> (none)
- U: renamed from C25; value 10uF -> (none); footprint vanalles:0603 -> (none)
- U: renamed from R7; value 10K -> (none); footprint vanalles:0603RL -> (none)
- U: renamed from MOD1; value RFM98W-433S2 -> (none); footprint Module:XCVR_RFM98W-433S2 -> (none)
- U: renamed from C27; value 0.1uF -> (none); footprint vanalles:0603 -> (none)
