File: pcb/asset tracker LoRa/LoRa tracker/esp32.kicad_sch (KiCad schematic)
At the start: 5 parts, among them CON1 TAGconnect_ESP, U6 ESP32-WROOM

Commit message: fgnhb
fgdh
Parts:
- U: renamed from U6; value ESP32-WROOM -> (none); footprint Module:ESP32-WROOM-32 -> (none)
- U: renamed from R10; value 10K -> (none); footprint vanalles:0603RL -> (none)
- U: renamed from R11; value NM -> (none); footprint vanalles:0603RL -> (none)
- U: renamed from R6; value 10K -> (none); footprint vanalles:0603RL -> (none)
- U: renamed from CON1; value TAGconnect_ESP -> (none); footprint connectors_user:Tag-Connect_TC2030-IDC-NL_2x03_P1.27mm_Vertical -> (none)
