File: pcb/asset tracker LoRa/LoRa tracker/mcu.kicad_sch (KiCad schematic)
At the start: 7 parts, among them CON2 jtag, U7 STM32L052K6Tx, Y2 32khz

Commit message: fgnhb
fgdh
Parts:
- U: renamed from CON2; value jtag -> (none); footprint connectors_user:Tag-Connect_TC2050-IDC-FP_2x05_P1.27mm_Vertical -> (none)
- U: renamed from C21; value 1uF -> (none); footprint vanalles:0603 -> (none)
- U: renamed from C20; value 100nF -> (none); footprint vanalles:0603 -> (none)
- U: renamed from C22; value 6.8pF -> (none); footprint vanalles:0603 -> (none)
- U: renamed from C33; value 6.8pF -> (none); footprint vanalles:0603 -> (none)
- U: renamed from U7; value STM32L052K6Tx -> (none); footprint halfgeleiders:QFP32P80_900X900X160L60X37N -> (none)
- U: renamed from Y2; value 32khz -> (none); footprint vanalles:crystal tht -> (none)
