File: pcb/asset tracker LoRa/LoRa tracker/voeding.kicad_sch (KiCad schematic)
At the start: 8 parts, among them J1 Screw_Terminal_01x02, U1 INA219BxDCN, U2 R-78HB3.3-0.5L

Commit message: fgnhb
fgdh
Parts:
- U: renamed from R1; value 100m Ohm -> (none); footprint vanalles:R_2512_6332Metric_Pad1.40x3.35mm_HandSolder -> (none)
- U: renamed from C2; value 10uF -> (none); footprint vanalles:0603 -> (none)
- U: renamed from C4; value 10uF -> (none); footprint vanalles:0603 -> (none)
- U: renamed from C3; value 100nF -> (none); footprint vanalles:0603 -> (none)
- U: renamed from U2; value R-78HB3.3-0.5L -> (none); footprint vanalles:recom psu -> (none)
- U: renamed from J1; value Screw_Terminal_01x02 -> (none); footprint connectors_user:2pin_screw -> (none)
- U: renamed from U1; value INA219BxDCN -> (none); footprint halfgeleiders:SOIC127P599X175-8N -> (none)
- U: renamed from C1; value 100nF -> (none); footprint vanalles:0603 -> (none)
