File: pcb/asset tracker LoRa/quadkey/quadkey/quadkey.kicad_pcb (KiCad board)
At the start: 2 copper layers, 42.1 x 72.6 mm, 0 parts

Commit message: quadkey
quadkey print klaar
Parts:
- added AE1: Antenna, vanalles:Texas_SWRA117D_2.4GHz_Right, F.Cu at (100.3, 53.2)
- added BT1: Battery, connectors_user:jst 2 pin, B.Cu at (112.1, 113.3)
- added C1: 10uF, vanalles:0603, F.Cu at (95.1, 94.5)
- added C10: 100nF, vanalles:0603, F.Cu at (100.2, 72.4)
- added C11: NM, vanalles:0603, F.Cu at (99.6, 60.8)
- added C12: 12pF, vanalles:0603, F.Cu at (93.8, 59.7)
- added C13: 12pF, vanalles:0603, F.Cu at (92.5, 66.0)
- added C14: NM, vanalles:0603, F.Cu at (99.6, 55.0)
- added C2: 0.1uF, vanalles:0603, F.Cu at (104.4, 89.3)
- added C3: 10uF, vanalles:0603, F.Cu at (99.2, 85.3)
- added C4: 10uF, vanalles:0603, F.Cu at (97.3, 85.3)
- added C5: 4.7uF, vanalles:0603, F.Cu at (95.4, 74.3)
- added C6: 100nF, vanalles:0603, F.Cu at (93.5, 74.2)
- added C7: 100nF, vanalles:0603, F.Cu at (97.4, 74.3)
- added C8: 1uF, vanalles:0603, F.Cu at (93.7, 69.0)
- added C9: 100pF, vanalles:0603, B.Cu at (96.9, 60.2)
- added CON1: jtag, connectors_user:SAMTEC_FTSH-105-01-F-D-K, F.Cu at (114.0, 67.3)
- added D1: LED, halfgeleiders:led0603, F.Cu at (95.7, 96.6)
- added L1: L, vanalles:0603RL, F.Cu at (96.5, 105.0)
- added L2: 2.2uH, vanalles:INDM300X300X200L80X50, F.Cu at (94.7, 91.1)
- added R1: 100, vanalles:0603RL, F.Cu at (104.4, 93.1)
- added R2: 1K, vanalles:0603RL, F.Cu at (102.2, 96.6)
- added R3: 1k, vanalles:0603RL, F.Cu at (104.2, 101.6)
- added R4: 1k, vanalles:0603RL, F.Cu at (108.9, 101.6)
- added R5: 0, vanalles:0603RL, F.Cu at (100.3, 57.9)
- added U1: MCP73831, halfgeleiders:SOT-25, F.Cu at (99.7, 100.2)
- added U2: TPS63001, halfgeleiders:SON50P300X300X100-11N, F.Cu at (99.1, 91.2)
- added U3: nRF52810-QFxx, halfgeleiders:nrf, F.Cu at (100.0, 66.9)
- added Y1: 326MhZ, vanalles:OSCCC200X160X50L55X65, F.Cu at (93.2, 62.9)
- added con1: USB_micro, connectors_user:usb_connector, F.Cu at (98.1, 113.9)
Routing:
- net GND: track 0.00 -> 58.5 mm, vias 0 -> 15
- net VBAT: track 0.00 -> 44.1 mm, vias 0 -> 3
- net /mcu/SWDIO: track 0.00 -> 19.5 mm, vias 0 -> 1
- net /mcu/SWDCLK: track 0.00 -> 17.1 mm, vias 0 -> 1
- net Net-(C2-Pad1): track 0.00 -> 12.1 mm
- net Net-(C13-Pad1): track 0.00 -> 11.6 mm, vias 0 -> 2
- net VBUS: track 0.00 -> 10.7 mm
- net /mcu/RST: track 0.00 -> 10.4 mm
- net Net-(C12-Pad1): track 0.00 -> 8.20 mm
- net +3V3: track 0.00 -> 7.28 mm, vias 0 -> 2
- net Net-(C8-Pad2): track 0.00 -> 5.86 mm
- net Net-(C11-Pad1): track 0.00 -> 5.36 mm
- net Net-(D1-Pad1): track 0.00 -> 5.05 mm
- net Net-(R2-Pad1): track 0.00 -> 4.98 mm
- net Net-(L1-Pad1): track 0.00 -> 4.80 mm
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- added copper zone on B.Cu, net GND

Commit message: 34t
34t
Parts:
- removed con1: USB_micro, connectors_user:usb_connector
- added J1: USB_B_Mini, connectors_user:AMPHENOL_10118192-0001LF, F.Cu at (98.1, 116.0)
- CON1: footprint connectors_user:SAMTEC_FTSH-105-01-F-D-K -> connectors_user:Tag-Connect_TC2050-IDC-FP_2x05_P1.27mm_Vertical
- L2: footprint vanalles:INDM300X300X200L80X50 -> vanalles:WURTH_744025001
- Y1: footprint vanalles:OSCCC200X160X50L55X65 -> vanalles:OSCCC320X250X90L80X100N
- moved C13 1.03 mm to (91.5, 66.4), turned to 180 degrees
- moved CON1 0.75 mm to (114.0, 66.5), turned to -90 degrees
- moved L2 0.55 mm to (94.2, 91.0)
- moved Y1 0.17 mm to (93.1, 62.8)
Routing:
- net GND: track 58.5 -> 78.4 mm, vias 15 -> 19
- net /mcu/SWDIO: track 19.5 -> 14.4 mm, vias 1 -> 0
- net /mcu/SWDCLK: track 17.1 -> 12.7 mm, vias 1 -> 0
- net /mcu/RST: track 10.4 -> 14.7 mm, vias 0 -> 2
- net Net-(J1-Pad1): track 4.80 -> 7.70 mm
- net Net-(C13-Pad1): track 11.6 -> 13.4 mm
- net Net-(C8-Pad2): track 5.86 -> 4.77 mm
- net Net-(L2-Pad1): track 3.22 -> 3.91 mm

Commit message: klaar
pcb klaar
Parts:
- moved C12 1.28 mm to (93.9, 58.5)
Routing:
- net Net-(C12-Pad1): track 8.38 -> 9.99 mm
