File: pcb/asset tracker LoRa/LoRa_Tracker_V2/Lora_tracker_V2/Lora_tracker_V2.kicad_pcb (KiCad board)
At the start: 2 copper layers, 116.3 x 114.5 mm, 3 parts

Commit message: ferg
werg
Parts:
- added AE1: Antenna_Shield, connectors_user:ufl connector, F.Cu at (86.5, -73.2)
- added AE2: sma, connectors_user:ufl connector, F.Cu at (86.5, -81.9)
- added BT1: Battery_Cell, vanalles:3012TR, F.Cu at (96.8, -93.8)
- added C1: NM, vanalles:0603, F.Cu at (85.5, -69.2)
- added C10: 100nF, vanalles:0603, F.Cu at (162.4, -94.8)
- added C11: 100nF, vanalles:0603, F.Cu at (98.2, -43.2)
- added C12: 10uF, vanalles:0603, F.Cu at (110.0, -55.8)
- added C13: 100nF, vanalles:0603, F.Cu at (110.0, -53.4)
- added C14: 10uF, vanalles:0603, F.Cu at (106.0, -56.5)
- added C15: 10uF, vanalles:0603, F.Cu at (123.5, -101.7)
- added C16: 100nF, vanalles:0603, F.Cu at (91.1, -83.5)
- added C17: 120nF, vanalles:0603, F.Cu at (94.8, -83.5)
- added C18: 10uF, vanalles:0603, F.Cu at (151.8, -101.7)
- added C19: 1uF, vanalles:0603, F.Cu at (130.8, -84.1)
- added C2: NM, vanalles:0603, F.Cu at (91.1, -74.9)
- added C20: 0.1uF, vanalles:0603, F.Cu at (130.8, -81.7)
- added C21: 100nF, vanalles:0603, F.Cu at (93.3, -27.1)
- added C22: 1uF, vanalles:0603, F.Cu at (90.9, -24.8)
- added C23: 6.8pF, vanalles:0603, F.Cu at (87.2, -22.5)
- added C24: 6.8pF, vanalles:0603, F.Cu at (87.2, -24.9)
- added C25: 100nF, vanalles:0603, F.Cu at (135.1, -67.1)
- added C26: 10uF, vanalles:0603, F.Cu at (130.2, -62.1)
- added C3: 100nF, vanalles:0603, F.Cu at (61.9, -95.2)
- added C4: 10uF, vanalles:0603, F.Cu at (40.5, -70.0)
- added C5: 100nF, vanalles:0603, F.Cu at (65.6, -95.2)
- added C6: 10uF, vanalles:0603, F.Cu at (70.9, -101.7)
- added C7: 100nF, vanalles:0603, F.Cu at (61.9, -92.8)
- added C8: 10uF, vanalles:0603, F.Cu at (54.4, -81.3)
- added C9: 10uF, vanalles:0603, F.Cu at (162.4, -97.2)
- added CON1: TAGconnect_ESP, connectors_user:Tag-Connect_TC2030-IDC-NL_2x03_P1.27mm_Vertical, F.Cu at (30.0, -26.9)
- added CON2: jtag, connectors_user:Tag-Connect_TC2050-IDC-FP_2x05_P1.27mm_Vertical, F.Cu at (97.5, -33.1)
- added D1: PESD15VL2BT, halfgeleiders:sot-23,, F.Cu at (130.8, -65.8)
- added J1: Screw_Terminal_01x02, connectors_user:AMASS_XT60PW-F, F.Cu at (198.5, 53.8)
- added J2: Screw_Terminal_01x02, connectors_user:2pin_screw, F.Cu at (84.7, -44.1)
- added J3: Screw_Terminal_01x02, connectors_user:AMASS_XT60PW-F, F.Cu at (51.5, -91.9)
- added L1: 5n6, vanalles:0603, F.Cu at (111.8, -88.4)
- added MOD1: teseo-LIV, Module:SON_STM_TESEO-LIV3R, F.Cu at (115.8, -96.7)
- added MOD2: RFM98W-433S2, Module:XCVR_RFM98W-433S2, F.Cu at (139.8, -94.1)
- added PZ1: buzzer, vanalles:PROSIGNAL_ABI-017-RC, F.Cu at (87.6, -53.9)
- added Q1: BSS138, halfgeleiders:sot-23,, F.Cu at (112.1, -59.5)
- added R1: 0, vanalles:0603RL, F.Cu at (89.1, -69.2)
- added R10: NM, vanalles:0603RL, F.Cu at (57.4, -60.8)
- added R11: 1M ohm, vanalles:0603, F.Cu at (36.9, -70.0)
- added R12: 36Kohm, vanalles:0603, F.Cu at (36.9, -67.6)
- added R2: 100m Ohm, vanalles:R_2512_6332Metric_Pad1.40x3.35mm_HandSolder, F.Cu at (180.8, 49.7)
- added R3: 10K, vanalles:0603, F.Cu at (90.8, -43.2)
- added R4: 220, vanalles:0603, F.Cu at (106.3, -51.8)
- added R5: 10K, vanalles:0603, F.Cu at (106.3, -54.1)
- added R6: 10K, vanalles:0603, F.Cu at (94.5, -43.2)
- added R7: 10K, vanalles:0603RL, F.Cu at (134.5, -84.1)
- added R8: 10K, vanalles:0603RL, F.Cu at (61.0, -60.8)
- added R9: 10K, vanalles:0603RL, F.Cu at (64.7, -60.8)
- added U1: INA219BxDCN, halfgeleiders:SOIC127P599X175-8N, F.Cu at (133.1, 1.86)
- added U10: nextion, connectors_user:NS-Tech_Grove_1x04_P2mm_Vertical, F.Cu at (124.8, -64.8)
- added U2: recom_psu, vanalles:recom psu, F.Cu at (45.9, -74.3)
- added U3: recom_psu, vanalles:recom psu, F.Cu at (32.6, -74.3)
- added U4: LIS3DH, halfgeleiders:QFN-16_0.5MM, F.Cu at (163.0, -100.6)
- added U5: G3VM-61HR2(TR05), halfgeleiders:sop4 P=2.54, F.Cu at (99.7, -53.5)
- added U6: DS28CM00R-A00+T, halfgeleiders:SOT-25, F.Cu at (107.2, -59.9)
- added U7: ATECC608B, halfgeleiders:soic p1.27 lengt 5.40, F.Cu at (97.5, -50.1)
- added U8: ESP32-WROOM, Module:ESP32-WROOM-32, F.Cu at (40.7, -40.5)
- added U9: STM32L052K6Tx, halfgeleiders:QFP32P80_900X900X160L60X37N, F.Cu at (85.9, -32.3)
- added Y1: 32khz, vanalles:crystal tht, F.Cu at (82.3, -23.5)
