File: pcb/voedings print voor v1/voedingsprint/voedingsprint.kicad_sch (KiCad schematic)
At the start: 0 parts

Commit message: voedings print voor v1
voedingsprint getekend voor tracker V1
Parts:
- added C?: C, symbol Device:C
- added CON?: XT60 connector, symbol conectors:con_2pin
- added CON?: con_2pin, symbol conectors:con_2pin
- added D?: double_diode, symbol Halfgelijders:double_diode
Connections:
- new net: CON?.2, D?.1
- new net: C?.1, D?.2, D?.4
- new net: CON?.2, D?.3
- new net GNDD: CON?.1, CON?.1
Changed lines of the file:
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@@
 (kicad_sch (version 20210406) (generator eeschema)
   (paper "A4")
-  (symbol_instances)
+  (junction (at 54.61 59.69) (diameter 0.9144) (color 0 0 0 0))
+  (wire (pts (xy 39.37 44.45) (xy 54.61 44.45))
+    (stroke (width 0) (type solid) (color 0 0 0 0))
+  )
+  (wire (pts (xy 39.37 57.15) (xy 63.5 57.15))
+    (stroke (width 0) (type solid) (color 0 0 0 0))
+  )
+  (wire (pts (xy 39.37 59.69) (xy 54.61 59.69))
+    (stroke (width 0) (type solid) (color 0 0 0 0))
+  )
+  (wire (pts (xy 54.61 44.45) (xy 54.61 59.69))
+    (stroke (width 0) (type solid) (color 0 0 0 0))
+  )
+  (wire (pts (xy 54.61 59.69) (xy 54.61 66.04))
+    (stroke (width 0) (type solid) (color 0 0 0 0))
+  )
+  (wire (pts (xy 63.5 41.91) (xy 39.37 41.91))
+    (stroke (width 0) (type solid) (color 0 0 0 0))
+  )
+  (wire (pts (xy 63.5 46.99) (xy 63.5 41.91))
+    (stroke (width 0) (type solid) (color 0 0 0 0))
+  )
+  (wire (pts (xy 63.5 52.07) (xy 78.74 52.07))
+    (stroke (width 0) (type solid) (color 0 0 0 0))
+  )
+  (wire (pts (xy 63.5 57.15) (xy 63.5 52.07))
+    (stroke (width 0) (type solid) (color 0 0 0 0))
+  )
+  (wire (pts (xy 78.74 46.99) (xy 63.5 46.99))
+    (stroke (width 0) (type solid) (color 0 0 0 0))
+  )
+  (wire (pts (xy 99.06 49.53) (xy 87.63 49.53))
+    (stroke (width 0) (type solid) (color 0 0 0 0))
+  )
+  (wire (pts (xy 99.06 59.69) (xy 99.06 49.53))
+    (stroke (width 0) (type solid) (color 0 0 0 0))
+  )
+  (symbol (lib_id "power:GNDD") (at 54.61 66.04 0) (unit 1)
+    (in_bom yes) (on_board yes) (fields_autoplaced)
+    (property "Reference" "#PWR?" (id 0) (at 54.61 72.39 0)
+      (effects (font (size 1.27 1.27)) hide)
+    )
+    (property "Value" "GNDD" (id 1) (at 54.61 71.12 0))
+    (property "Footprint" "" (id 2) (at 54.61 66.04 0)
+      (effects (font (size 1.27 1.27)) hide)
+    )
+    (property "Datasheet" "" (id 3) (at 54.61 66.04 0)
+      (effects (font (size 1.27 1.27)) hide)
+    )
+    (pin "1")
+  )
+  (symbol (lib_id "conectors:con_2pin") (at 35.56 43.18 180) (unit 1)
+    (in_bom yes) (on_board yes) (fields_autoplaced)
+    (property "Reference" "CON?" (id 0) (at 36.3855 36.83 0))
+    (property "Value" "con_2pin" (id 1) (at 36.3855 39.37 0))
+    (property "Footprint" "" (id 2) (at 35.56 43.18 0)
+      (effects (font (size 1.27 1.27)) hide)
+    )
+    (property "Datasheet" "" (id 3) (at 35.56 43.18 0)
+      (effects (font (size 1.27 1.27)) hide)
+    )
+    (pin "1")
+    (pin "2")
+  )
+  (symbol (lib_id "conectors:con_2pin") (at 35.56 58.42 180) (unit 1)
+    (in_bom yes) (on_board yes) (fields_autoplaced)
+    (property "Reference" "CON?" (id 0) (at 36.3855 52.07 0))
+    (property "Value" "XT60 connector" (id 1) (at 36.3855 54.61 0))
+    (property "Footprint" "" (id 2) (at 35.56 58.42 0)
+      (effects (font (size 1.27 1.27)) hide)
+    )
+    (property "Datasheet" "" (id 3) (at 35.56 58.42 0)
+      (effects (font (size 1.27 1.27)) hide)
+    )
+    (pin "1")
+    (pin "2")
+  )
+  (symbol (lib_id "Device:C") (at 99.06 63.5 0) (unit 1)
+    (in_bom yes) (on_board yes) (fields_autoplaced)
+    (property "Reference" "C?" (id 0) (at 102.87 62.8649 0)
+      (effects (font (size 1.27 1.27)) (justify left))
+    )
+    (property "Value" "C" (id 1) (at 102.87 65.4049 0)
+      (effects (font (size 1.27 1.27)) (justify left))
+    )
+    (property "Footprint" "" (id 2) (at 100.0252 67.31 0)
+      (effects (font (size 1.27 1.27)) hide)
+    )
+    (property "Datasheet" "~" (id 3) (at 99.06 63.5 0)
+      (effects (font (size 1.27 1.27)) hide)
+    )
+    (pin "1")
+    (pin "2")
+  )
+  (symbol (lib_id "Halfgelijders:double_diode") (at 85.09 49.53 270) (unit 1)
+    (in_bom yes) (on_board yes) (fields_autoplaced)
+    (property "Reference" "D?" (id 0) (at 83.185 41.91 90))
+    (property "Value" "double_diode" (id 1) (at 83.185 44.45 90))
+    (property "Footprint" "" (id 2) (at 87.63 49.53 0)
+      (effects (font (size 1.27 1.27)) hide)
+    )
+    (property "Datasheet" "" (id 3) (at 87.63 49.53 0)
+      (effects (font (size 1.27 1.27)) hide)
+    )
+    (pin "1")
+    (pin "2")
+    (pin "3")
+    (pin "4")
+  )
+  (sheet_instances
+    (path "/" (page "1"))
+  )
+  (symbol_instances
+    (path "/92df61db-18a2-434c-b2c9-0119a91685bd"
+      (reference "#PWR?") (unit 1) (value "GNDD") (footprint "")
+    )
+    (path "/e82a3e23-7c20-450c-b7b5-4949fb083bd7"
+      (reference "C?") (unit 1) (value "C") (footprint "")
+    )
+    (path "/34e76240-61be-4c70-bc17-8304b959401f"
+      (reference "CON?") (unit 1) (value "XT60 connector") (footprint "")
+    )
+    (path "/a38ecfc5-9501-4a29-ad7e-b2fa0819ba2c"
+      (reference "CON?") (unit 1) (value "con_2pin") (footprint "")
+    )
+    (path "/4a7396a3-f4e9-4765-9587-24fa75a4923c"
+      (reference "D?") (unit 1) (value "double_diode") (footprint "")
+    )
+  )
 )
