File: pcb/asset tracker LoRa/voedings modulle loratracker/voedings_modulle/DCDC.kicad_sch (KiCad schematic)
At the start: 0 parts

Commit message: wef
wef
Parts:
- added C?: C_Polarized_Small_US, symbol Device:C_Polarized_Small_US
- added C? (x2): C_Small, symbol Device:C_Small
- added C?: C, symbol Device:C
- added D?: D_Schottky, symbol Device:D_Schottky
- added J?: Screw_Terminal_01x02, symbol Connector:Screw_Terminal_01x02
- added L?: L, symbol Device:L
- added R? (x2): R_Small_US, symbol Device:R_Small_US
- added U?: MAX5035AUSA, Package_SO:SOIC-8_3.9x4.9mm_P1.27mm, symbol Regulator_Switching:MAX5035AUSA
Connections:
- net VIN: now also C?.1, R?.1, U?.7 (VIN)
- new net: R?.1, R?.2, U?.5 (ON/~{OFF})
- new net: C?.2, D?.1 (K), L?.1, U?.8 (LX)
- new net: C?.1, J?.1 (Pin_1), L?.2, U?.4 (FB)
- new net: C?.1, U?.1 (BST)
- new net: C?.1, U?.2 (VD)
- new net GND: C?.2, C?.2, C?.2, D?.2 (A), J?.2 (Pin_2), R?.2, U?.3 (SGND), U?.6 (GND)

Commit message: voedings PCB
Voedings pcb schema afgetekend
Parts:
- added C?: 0.22uF/100V, symbol Device:C_Small
- C1: renamed from C?; value C_Small -> 68uF/100V
- C2: renamed from C?; value C_Small -> 0.1uF
- C3: renamed from C?; value C -> 0.1uF
- C4: renamed from C?; value C_Polarized_Small_US -> 68uF/10V
- L1: renamed from L?; value L -> 100uH
- R1: renamed from R?; value R_Small_US -> 43.5Kohm/1%
- R2: renamed from R?; value R_Small_US -> 130Kohm/1%
- gave numbers to parts that had none: 3
Connections:
- net GND: now also C?.2
- net VIN: now also C?.1
- net +3V3: now reaches C4.1, J1.1 (Pin_1), L1.2, U1.4 (FB)
