File: pcb/asset tracker LoRa/voedings modulle loratracker/voedings_modulle/microcontroller.kicad_sch (KiCad schematic)
At the start: 19 parts

Commit message: schema voedingswitcher af
voeding switcher voor v1 afgetekend
Connections:
- net SSR0: now reaches U?.21 (PA11)
- net Relay renamed SSR1
- no-connect marks 12 -> 11
Changed lines of the file:
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@@
-(kicad_sch (version 20210621) (generator eeschema)
+(kicad_sch (version 20210406) (generator eeschema)
   (paper "A4")
   (junction (at 75.565 124.46) (diameter 0.9144) (color 0 0 0 0))
@@
   (no_connect (at 89.535 99.06))
   (no_connect (at 89.535 101.6))
-  (no_connect (at 89.535 104.14))
   (no_connect (at 89.535 114.3))
   (no_connect (at 104.775 172.72))
@@
     (stroke (width 0) (type solid) (color 0 0 0 0))
   )
+  (wire (pts (xy 89.535 104.14) (xy 113.665 104.14))
+    (stroke (width 0) (type solid) (color 0 0 0 0))
+  )
   (wire (pts (xy 89.535 106.68) (xy 113.665 106.68))
     (stroke (width 0) (type solid) (color 0 0 0 0))
@@
     (effects (font (size 1.27 1.27)) (justify left))
   )
-  (hierarchical_label "Relay" (shape output) (at 113.665 106.68 0)
+  (hierarchical_label "SSR0" (shape output) (at 113.665 104.14 0)
     (effects (font (size 1.27 1.27)) (justify left))
   )
+  (hierarchical_label "SSR1" (shape output) (at 113.665 106.68 0)
+    (effects (font (size 1.27 1.27)) (justify left))
+  )
