File: pcb/asset tracker LoRa/voedings modulle loratracker/voedings_modulle/_autosave-voedings_modulle.kicad_sch (KiCad schematic)
At the start: 13 parts, among them con1 screw terminal, con2 xt60

Commit message: datasheet
Datasheet toegevoegd
Parts:
- R?: value 100ohm -> 1Kohm
- R?: value 100 ohm -> 1K ohm
Changed lines of the file:
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@@
       (effects (font (size 1.27 1.27)) (justify right))
     )
-    (property "Value" "100 ohm" (id 1) (at 118.11 104.7749 0)
+    (property "Value" "1K ohm " (id 1) (at 118.11 104.7749 0)
       (effects (font (size 1.27 1.27)) (justify right))
     )
@@
       (effects (font (size 1.27 1.27)) (justify right))
     )
-    (property "Value" "100ohm" (id 1) (at 135.89 102.8699 0)
+    (property "Value" "1Kohm" (id 1) (at 135.89 102.8699 0)
       (effects (font (size 1.27 1.27)) (justify right))
     )
@@
     )
     (path "/6fbbb8c8-ff36-4738-b0b6-7937d6f2a83e"
-      (reference "R?") (unit 1) (value "100ohm") (footprint "")
+      (reference "R?") (unit 1) (value "1Kohm") (footprint "")
     )
     (path "/b04b8752-3c3d-40d5-a512-14142a0fd0cf/7968de54-d1e4-4a7a-8fb2-6c341d0be18a"
@@
     )
     (path "/a845edb1-d258-4d61-aea3-3107d32c4a39"
-      (reference "R?") (unit 1) (value "100 ohm") (footprint "")
+      (reference "R?") (unit 1) (value "1K ohm ") (footprint "")
     )
     (path "/d18b4f86-0612-4f9e-a07a-aa57208b1cb1"
