File: pcb/asset tracker LoRa/voedings modulle loratracker/voedings switcher/_autosave-microcontroller.kicad_sch (KiCad schematic)
At the start: 19 parts

Commit message: zdsxvc
zxcv
Parts:
- CON1: renamed from CON?; footprint connectors_user:Tag-Connect_TC2050-IDC-FP_2x05_P1.27mm_Vertical -> connectors_user:Tag-Connect_TC2050-IDC-NL_2x05_P1.27mm_Vertical
- D1, D3, D4, D5, D6, D7: renamed from D?; footprint (none) -> halfgeleiders:led0603
- R10, R11, R12, R13, R14, R9: renamed from R?; footprint (none) -> vanalles:0603
- gave numbers to parts that had none: 6
