File: pcb/asset tracker LoRa/voedings modulle loratracker/voedings switcher/_autosave-voedings switcher.kicad_sch (KiCad schematic)
At the start: 13 parts, among them con1 screw terminal, con2 xt60

Commit message: zdsxvc
zxcv
Parts:
- removed JP?: Jumper_2_Open, symbol Jumper:Jumper_2_Open
- added FID1, FID2, FID3: Fiducial, symbol Mechanical:Fiducial
- added JP?: Jumper_2_Open, symbol Jumper:Jumper_2_Open
- R5: renamed from R?; value R_Small_US -> 900K; footprint (none) -> vanalles:0603
- R6: renamed from R?; value R_Small_US -> 58K; footprint (none) -> vanalles:0603
- R7: renamed from R?; value 100 ohm -> 1K ohm; footprint (none) -> vanalles:0603
- R8: renamed from R?; value 100ohm -> 1Kohm; footprint (none) -> vanalles:0603
- RV1: renamed from RV?; footprint (none) -> vanalles:3314G-1-201E bourns trimmer
- U2, U3: renamed from U?; footprint Package_DIP:DIP-5-6_W7.62mm -> halfgeleiders:TLP3542
- gave numbers to parts that had none: 3
Connections:
- net VM1: now also JP?.2 (B)
- net at R6.1, RV1.2, RV1.3: now also JP?.1 (A)
- net at R5.1, con2.2 (+), con3.2 (+): now also U3.6; no longer U2.6
- net at R3.1, con1.2 (+): now also U2.6; no longer U3.6
