File: pcb/asset tracker LoRa/voedings modulle loratracker/voedings switcher/dc-dc.kicad_sch (KiCad schematic)
At the start: 11 parts, among them J1 Screw_Terminal_01x02, U1 MAX5035AUSA

Commit message: zdsxvc
zxcv
Parts:
- removed D2: D_Schottky, symbol Device:D_Schottky
- added D?: MBRM5100, halfgeleiders:DPAK, symbol Halfgelijders:diode4
Connections:
- net GND: now also D?.1, D?.3
- net at C3.2, L1.1, U1.8 (LX): now also D?.4
Changed lines of the file:
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@@
-(kicad_sch (version 20210406) (generator eeschema)
+(kicad_sch (version 20210621) (generator eeschema)
   (paper "A4")
   (junction (at 35.56 52.07) (diameter 0.9144) (color 0 0 0 0))
@@
   (junction (at 182.88 52.07) (diameter 0.9144) (color 0 0 0 0))
   (junction (at 191.77 52.07) (diameter 0.9144) (color 0 0 0 0))
+  (junction (at 191.77 69.215) (diameter 0.9144) (color 0 0 0 0))
   (junction (at 220.98 52.07) (diameter 0.9144) (color 0 0 0 0))
   (junction (at 231.14 52.07) (diameter 0.9144) (color 0 0 0 0))
@@
     (stroke (width 0) (type solid) (color 0 0 0 0))
   )
+  (wire (pts (xy 190.5 69.215) (xy 190.5 66.04))
+    (stroke (width 0) (type solid) (color 0 0 0 0))
+  )
   (wire (pts (xy 191.77 52.07) (xy 205.74 52.07))
     (stroke (width 0) (type solid) (color 0 0 0 0))
@@
     (stroke (width 0) (type solid) (color 0 0 0 0))
   )
-  (wire (pts (xy 191.77 60.96) (xy 191.77 67.31))
+  (wire (pts (xy 191.77 69.215) (xy 190.5 69.215))
+    (stroke (width 0) (type solid) (color 0 0 0 0))
+  )
+  (wire (pts (xy 191.77 69.215) (xy 193.04 69.215))
+    (stroke (width 0) (type solid) (color 0 0 0 0))
+  )
+  (wire (pts (xy 193.04 69.215) (xy 193.04 66.04))
     (stroke (width 0) (type solid) (color 0 0 0 0))
   )
@@
   (symbol (lib_id "power:+3V3") (at 242.57 46.355 0) (unit 1)
     (in_bom yes) (on_board yes)
-    (property "Reference" "#PWR?" (id 0) (at 242.57 50.165 0)
+    (property "Reference" "#PWR0112" (id 0) (at 242.57 50.165 0)
       (effects (font (size 1.27 1.27)) hide)
     )
@@
   (symbol (lib_id "power:GND") (at 55.88 77.47 0) (unit 1)
     (in_bom yes) (on_board yes) (fields_autoplaced)
-    (property "Reference" "#PWR?" (id 0) (at 55.88 83.82 0)
+    (property "Reference" "#PWR0110" (id 0) (at 55.88 83.82 0)
       (effects (font (size 1.27 1.27)) hide)
     )
@@
   (symbol (lib_id "power:GND") (at 149.86 85.09 0) (unit 1)
     (in_bom yes) (on_board yes) (fields_autoplaced)
-    (property "Reference" "#PWR0103" (id 0) (at 149.86 91.44 0)
+    (property "Reference" "#PWR0111" (id 0) (at 149.86 91.44 0)
       (effects (font (size 1.27 1.27)) hide)
     )
@@
     (pin "1")
   )
-  (symbol (lib_id "power:GND") (at 191.77 67.31 0) (unit 1)
-    (in_bom yes) (on_board yes) (fields_autoplaced)
-    (property "Reference" "#PWR0105" (id 0) (at 191.77 73.66 0)
-      (effects (font (size 1.27 1.27)) hide)
-    )
-    (property "Value" "GND" (id 1) (at 191.77 72.39 0))
-    (property "Footprint" "" (id 2) (at 191.77 67.31 0)
-      (effects (font (size 1.27 1.27)) hide)
-    )
-    (property "Datasheet" "" (id 3) (at 191.77 67.31 0)
+  (symbol (lib_id "power:GND") (at 191.77 69.215 0) (unit 1)
+    (in_bom yes) (on_board yes) (fields_autoplaced)
+    (property "Reference" "#PWR0105" (id 0) (at 191.77 75.565 0)
+      (effects (font (size 1.27 1.27)) hide)
+    )
+    (property "Value" "GND" (id 1) (at 191.77 74.295 0))
+    (property "Footprint" "" (id 2) (at 191.77 69.215 0)
+      (effects (font (size 1.27 1.27)) hide)
+    )
+    (property "Datasheet" "" (id 3) (at 191.77 69.215 0)
       (effects (font (size 1.27 1.27)) hide)
     )
@@
     (pin "2")
   )
-  (symbol (lib_id "Device:D_Schottky") (at 191.77 57.15 270) (unit 1)
-    (in_bom yes) (on_board yes) (fields_autoplaced)
-    (property "Reference" "D2" (id 0) (at 194.31 55.8799 90)
-      (effects (font (size 1.27 1.27)) (justify left))
-    )
-    (property "Value" "D_Schottky" (id 1) (at 194.31 58.4199 90)
-      (effects (font (size 1.27 1.27)) (justify left))
-    )
-    (property "Footprint" "" (id 2) (at 191.77 57.15 0)
-      (effects (font (size 1.27 1.27)) hide)
-    )
-    (property "Datasheet" "~" (id 3) (at 191.77 57.15 0)
-      (effects (font (size 1.27 1.27)) hide)
-    )
-    (pin "1")
-    (pin "2")
-  )
   (symbol (lib_id "Connector:Screw_Terminal_01x02") (at 259.08 52.07 0) (unit 1)
     (in_bom yes) (on_board yes) (fields_autoplaced)
@@
     (pin "2")
   )
+  (symbol (lib_id "Halfgelijders:diode4") (at 191.77 62.23 0) (unit 1)
+    (in_bom yes) (on_board yes) (fields_autoplaced)
+    (property "Reference" "D?" (id 0) (at 194.31 58.4199 0)
+      (effects (font (size 1.27 1.27)) (justify left))
+    )
+    (property "Value" "MBRM5100" (id 1) (at 194.31 60.9599 0)
+      (effects (font (size 1.27 1.27)) (justify left))
+    )
+    (property "Footprint" "halfgeleiders:DPAK" (id 2) (at 191.77 62.23 0)
+      (effects (font (size 1.27 1.27)) hide)
+    )
+    (property "Datasheet" "" (id 3) (at 191.77 62.23 0)
+      (effects (font (size 1.27 1.27)) hide)
+    )
+    (pin "1")
+    (pin "3")
+    (pin "4")
+  )
   (symbol (lib_id "Regulator_Switching:MAX5035AUSA") (at 149.86 57.15 0) (unit 1)

Commit message: fb
dfb
Parts:
- C1, C4: footprint (none) -> vanalles:CAPAE1030X1050D1200L350X90N
- C2, C3, R1, R2: footprint (none) -> vanalles:0603
- C5: renamed from C?; footprint (none) -> vanalles:CAPAE1030X1050D1200L350X90N
- J1: footprint (none) -> connectors_user:2pin_screw_vast
- L1: footprint (none) -> vanalles:DO5022p
- U1: footprint Package_SO:SOIC-8_3.9x4.9mm_P1.27mm -> halfgeleiders:soic HV clearance
- gave numbers to parts that had none: 1
Changed lines of the file:
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@@
     (stroke (width 0) (type solid) (color 0 0 0 0))
   )
-  (wire (pts (xy 149.86 85.09) (xy 149.86 76.2))
+  (wire (pts (xy 149.86 86.36) (xy 149.86 76.2))
     (stroke (width 0) (type solid) (color 0 0 0 0))
   )
@@
     (pin "1")
   )
-  (symbol (lib_id "power:GND") (at 149.86 85.09 0) (unit 1)
-    (in_bom yes) (on_board yes) (fields_autoplaced)
-    (property "Reference" "#PWR0111" (id 0) (at 149.86 91.44 0)
-      (effects (font (size 1.27 1.27)) hide)
-    )
-    (property "Value" "GND" (id 1) (at 149.86 90.17 0))
-    (property "Footprint" "" (id 2) (at 149.86 85.09 0)
-      (effects (font (size 1.27 1.27)) hide)
-    )
-    (property "Datasheet" "" (id 3) (at 149.86 85.09 0)
+  (symbol (lib_id "power:GND") (at 149.86 86.36 0) (unit 1)
+    (in_bom yes) (on_board yes) (fields_autoplaced)
+    (property "Reference" "#PWR0111" (id 0) (at 149.86 92.71 0)
+      (effects (font (size 1.27 1.27)) hide)
+    )
+    (property "Value" "GND" (id 1) (at 149.86 91.44 0))
+    (property "Footprint" "" (id 2) (at 149.86 86.36 0)
+      (effects (font (size 1.27 1.27)) hide)
+    )
+    (property "Datasheet" "" (id 3) (at 149.86 86.36 0)
       (effects (font (size 1.27 1.27)) hide)
     )
@@
     (property "Reference" "L1" (id 0) (at 209.55 45.72 90))
     (property "Value" "100uH" (id 1) (at 209.55 48.26 90))
-    (property "Footprint" "" (id 2) (at 209.55 52.07 0)
+    (property "Footprint" "vanalles:DO5022p" (id 2) (at 209.55 52.07 0)
       (effects (font (size 1.27 1.27)) hide)
     )
@@
       (effects (font (size 1.27 1.27)) (justify left))
     )
-    (property "Footprint" "" (id 2) (at 85.09 59.69 0)
+    (property "Footprint" "vanalles:0603" (id 2) (at 85.09 59.69 0)
       (effects (font (size 1.27 1.27)) hide)
     )
@@
       (effects (font (size 1.27 1.27)) (justify left))
     )
-    (property "Footprint" "" (id 2) (at 85.09 69.85 0)
+    (property "Footprint" "vanalles:0603" (id 2) (at 85.09 69.85 0)
       (effects (font (size 1.27 1.27)) hide)
     )
@@
       (effects (font (size 1.27 1.27)) (justify left))
     )
-    (property "Footprint" "" (id 2) (at 231.14 62.23 0)
+    (property "Footprint" "vanalles:CAPAE1030X1050D1200L350X90N" (id 2) (at 231.14 62.23 0)
       (effects (font (size 1.27 1.27)) hide)
     )
@@
       (effects (font (size 1.27 1.27)) (justify left))
     )
-    (property "Footprint" "" (id 2) (at 35.56 64.77 0)
+    (property "Footprint" "vanalles:CAPAE1030X1050D1200L350X90N" (id 2) (at 35.56 64.77 0)
       (effects (font (size 1.27 1.27)) hide)
     )
@@
   (symbol (lib_id "Device:C_Small") (at 55.88 64.77 0) (unit 1)
     (in_bom yes) (on_board yes) (fields_autoplaced)
-    (property "Reference" "C?" (id 0) (at 58.42 63.4999 0)
+    (property "Reference" "C5" (id 0) (at 58.42 63.4999 0)
       (effects (font (size 1.27 1.27)) (justify left))
     )
@@
       (effects (font (size 1.27 1.27)) (justify left))
     )
-    (property "Footprint" "" (id 2) (at 55.88 64.77 0)
+    (property "Footprint" "vanalles:CAPAE1030X1050D1200L350X90N" (id 2) (at 55.88 64.77 0)
       (effects (font (size 1.27 1.27)) hide)
     )
@@
       (effects (font (size 1.27 1.27)) (justify left))
     )
-    (property "Footprint" "" (id 2) (at 128.27 67.31 0)
+    (property "Footprint" "vanalles:0603" (id 2) (at 128.27 67.31 0)
       (effects (font (size 1.27 1.27)) hide)
     )
@@
       (effects (font (size 1.27 1.27)) (justify left))
     )
-    (property "Footprint" "" (id 2) (at 259.08 52.07 0)
+    (property "Footprint" "connectors_user:2pin_screw_vast" (id 2) (at 259.08 52.07 0)
       (effects (font (size 1.27 1.27)) hide)
     )
@@
     (property "Reference" "C3" (id 0) (at 179.07 44.45 90))
     (property "Value" "0.1uF" (id 1) (at 179.07 46.99 90))
-    (property "Footprint" "" (id 2) (at 182.88 51.1048 0)
+    (property "Footprint" "vanalles:0603" (id 2) (at 182.88 51.1048 0)
       (effects (font (size 1.27 1.27)) hide)
     )
@@
   (symbol (lib_id "Halfgelijders:diode4") (at 191.77 62.23 0) (unit 1)
     (in_bom yes) (on_board yes) (fields_autoplaced)
-    (property "Reference" "D?" (id 0) (at 194.31 58.4199 0)
+    (property "Reference" "D2" (id 0) (at 194.31 58.4199 0)
       (effects (font (size 1.27 1.27)) (justify left))
     )
@@
     (property "Reference" "U1" (id 0) (at 149.86 44.45 0))
     (property "Value" "MAX5035AUSA" (id 1) (at 149.86 46.99 0))
-    (property "Footprint" "Package_SO:SOIC-8_3.9x4.9mm_P1.27mm" (id 2) (at 153.67 66.04 0)
+    (property "Footprint" "halfgeleiders:soic HV clearance" (id 2) (at 153.67 66.04 0)
       (effects (font (size 1.27 1.27) italic) (justify left) hide)
     )
