File: pcb/asset tracker LoRa/voedings modulle loratracker/voedings switcher/microcontroller.kicad_sch (KiCad schematic)
At the start: 19 parts, among them CON1 jtag, U4 STM32L052K6Tx, Y1 32khz

Commit message: fb
dfb
Parts:
- removed D1, D5: LED_GROEN, symbol Device:LED
- removed D3, D6: LED_GEEL, symbol Device:LED
- removed D4, D7: LED_ROOD, symbol Device:LED
- removed R10, R11, R12, R13, R14, R9: 40, symbol Device:R_Small_US
- CON1: footprint connectors_user:Tag-Connect_TC2050-IDC-FP_2x05_P1.27mm_Vertical -> connectors_user:Tag-Connect_TC2050-IDC-NL_2x05_P1.27mm_Vertical
Connections:
- net BAT1_0: no longer names the net of U4.14 (PB0)
- net BAT1_1: no longer names the net of U4.15 (PB1)
- net BAT1_2: no longer names the net of U4.26 (PB3)
- net BAT1_2: no longer U4.29 (PB6)
- net BAT2_0: no longer names the net of U4.27 (PB4)
- net BAT2_1: no longer names the net of U4.28 (PB5)
- no-connect marks 11 -> 17
