File: pcb/asset tracker LoRa/voedings modulle loratracker/voedings switcher/voedings switcher.kicad_pcb (KiCad board)
At the start: 0 parts

Commit message: fb
dfb
Parts:
- added C1: 68uF/100V, vanalles:CAPAE1030X1050D1200L350X90N, F.Cu at (110.8, 83.1)
- added C2: 0.1uF, vanalles:0603, F.Cu at (131.9, 81.2)
- added C3: 0.1uF, vanalles:0603, F.Cu at (137.2, 78.1)
- added C4: 68uF/10V, vanalles:CAPAE1030X1050D1200L350X90N, F.Cu at (153.7, 100.0)
- added C5: 0.22uF/100V, vanalles:CAPAE1030X1050D1200L350X90N, F.Cu at (124.2, 82.4)
- added C6: 100nF, vanalles:0603, F.Cu at (86.9, 169.4)
- added C7: 1uF, vanalles:0603, F.Cu at (88.4, 164.3)
- added C8: 6.8pF, vanalles:0603, F.Cu at (83.3, 169.4)
- added C9: 6.8pF, vanalles:0603, F.Cu at (88.4, 166.7)
- added CON1: jtag, connectors_user:Tag-Connect_TC2050-IDC-NL_2x05_P1.27mm_Vertical, F.Cu at (141.7, 115.3)
- added D2: MBRM5100, halfgeleiders:DPAK, F.Cu at (135.1, 69.5)
- added FID1: Fiducial, vanalles:Fiducial_0.5mm_Mask1.5mm, F.Cu at (166.3, 111.8)
- added FID2: Fiducial, vanalles:Fiducial_0.5mm_Mask1.5mm, F.Cu at (72.9, 68.9)
- added FID3: Fiducial, vanalles:Fiducial_0.5mm_Mask1.5mm, F.Cu at (166.2, 68.9)
- added J1: Screw_Terminal_01x02, connectors_user:2pin_screw_vast, F.Cu at (163.9, 98.4)
- added JP1: Jumper_2_Open, vanalles:SolderJumper-2_P1.3mm_Open_Pad1.0x1.5mm, F.Cu at (69.7, 164.9)
- added L1: 100uH, vanalles:DO5022p, F.Cu at (146.5, 83.3)
- added R1: 43.5Kohm/1%, vanalles:0603, F.Cu at (132.9, 88.8)
- added R2: 130Kohm/1%, vanalles:0603, F.Cu at (139.6, 88.9)
- added R3: 1Mohm, vanalles:0603, F.Cu at (96.2, 74.1)
- added R4: 58Kohm, vanalles:0603, F.Cu at (96.2, 69.3)
- added R5: 900K, vanalles:0603, F.Cu at (69.4, 167.8)
- added R6: 58K, vanalles:0603, F.Cu at (73.8, 164.3)
- added R7: 1K ohm, vanalles:0603, F.Cu at (96.5, 116.0)
- added R8: 1Kohm, vanalles:0603, F.Cu at (110.3, 116.2)
- added RV1: 100K, vanalles:3314G-1-201E bourns trimmer, F.Cu at (62.9, 165.7)
- added U1: MAX5035AUSA, halfgeleiders:soic HV clearance, F.Cu at (134.9, 80.8)
- added U2: TLP3542, halfgeleiders:TLP3542, F.Cu at (99.2, 108.4)
- added U3: TLP3542, halfgeleiders:TLP3542, F.Cu at (113.0, 108.1)
- added U4: STM32L052K6Tx, halfgeleiders:QFP32P80_900X900X160L60X37N, F.Cu at (140.5, 101.4)
- added Y1: 32khz, vanalles:crystal tht, F.Cu at (83.5, 165.7)
- added con1: screw terminal, connectors_user:2pin_screw, F.Cu at (77.9, 80.9)
- added con2: xt60, connectors_user:AMASS_XT60PW-F, F.Cu at (72.4, 97.8)
Routing:
- net /dcdc/VIN: track 0.00 -> 62.3 mm
- net Net-(R3-Pad1): track 0.00 -> 48.5 mm
- net /microcontroller/SSR1: track 0.00 -> 47.5 mm
- net /microcontroller/SSR0: track 0.00 -> 41.2 mm, vias 0 -> 2
- net Net-(R5-Pad1): track 0.00 -> 33.5 mm
- net GND: track 0.00 -> 28.6 mm, vias 0 -> 8
- net Net-(C3-Pad2): track 0.00 -> 19.0 mm
- net Net-(R1-Pad2): track 0.00 -> 12.1 mm
- net Net-(R8-Pad2): track 0.00 -> 3.72 mm
- net /VM0: track 0.00 -> 3.52 mm
- net Net-(C3-Pad1): track 0.00 -> 3.37 mm
- net Net-(C2-Pad1): track 0.00 -> 3.15 mm
- net Net-(R7-Pad2): track 0.00 -> 3.13 mm
- added copper zone on F.Cu, net +3V3
- added copper zone on B.Cu, net GND
Other:
- board outline added: 96.5 x 59 mm
- copper layers 0 -> 2
