File: pcb/asset tracker LoRa/voedings modulle loratracker/voedings switcher/voedings switcher.kicad_sch (KiCad schematic)
At the start: 13 parts, among them con1 screw terminal, con2 xt60

Commit message: zdsxvc
zxcv
Parts:
- removed JP?: Jumper_2_Open, symbol Jumper:Jumper_2_Open
- added FID1, FID2, FID3: Fiducial, symbol Mechanical:Fiducial
- added JP?: Jumper_2_Open, symbol Jumper:Jumper_2_Open
- R5: renamed from R?; value R_Small_US -> 900K
- R6: renamed from R?; value R_Small_US -> 58K
- RV1: renamed from RV?; footprint (none) -> vanalles:3314G-1-201E bourns trimmer
- gave numbers to parts that had none: 7
Connections:
- net VM1: now also JP?.2 (B)
- net at R6.1, RV1.2, RV1.3: now also JP?.1 (A)
- net at R5.1, con2.2 (+), con3.2 (+): now also U3.6; no longer U2.6
- net at R3.1, con1.2 (+): now also U2.6; no longer U3.6

Commit message: fb
dfb
Parts:
- removed con3: xt90, symbol conectors:battery_con
- FID1, FID2, FID3: footprint (none) -> vanalles:Fiducial_0.5mm_Mask1.5mm
- JP1: renamed from JP?; footprint (none) -> vanalles:SolderJumper-2_P1.3mm_Open_Pad1.0x1.5mm
- R3, R4, R5, R6, R7, R8: footprint (none) -> vanalles:0603
- U2, U3: footprint Package_DIP:DIP-5-6_W7.62mm -> halfgeleiders:TLP3542
- con1: footprint (none) -> connectors_user:2pin_screw
- con2: footprint (none) -> connectors_user:AMASS_XT60PW-F
