File: pcb/asset tracker LoRa/lora tracker V3/Lora_tracker_V3/DC_DC.kicad_sch (KiCad schematic)
At the start: 11 parts, among them J1 Screw_Terminal_01x02, U1 MAX5035AUSA

Commit message: eadf
sdfv
Parts:
- removed C1: 68uF/100V, vanalles:CAPAE1030X1050D1200L350X90N, symbol Device:C_Small
- removed C2: 0.1uF, vanalles:0603, symbol Device:C_Small
- removed C3: 0.1uF, vanalles:0603, symbol Device:C
- removed C4: 68uF/10V, vanalles:CAPAE1030X1050D1200L350X90N, symbol Device:C_Polarized_Small_US
- removed C5: 0.22uF/100V, vanalles:CAPAE1030X1050D1200L350X90N, symbol Device:C_Small
- removed D2: MBRM5100, halfgeleiders:DPAK, symbol Halfgelijders:diode4
- removed J1: Screw_Terminal_01x02, connectors_user:2pin_screw_vast, symbol Connector:Screw_Terminal_01x02
- removed L1: 100uH, vanalles:DO5022p, symbol Device:L
- removed R1: 43.5Kohm/1%, vanalles:0603, symbol Device:R_Small_US
- removed R2: 130Kohm/1%, vanalles:0603, symbol Device:R_Small_US
- removed U1: MAX5035AUSA, halfgeleiders:soic HV clearance, symbol Regulator_Switching:MAX5035AUSA
- added C?: 68uF/10V, vanalles:CAPAE1030X1050D1200L350X90N, symbol Device:C_Polarized_Small_US
- added C?: 0.22uF/100V, vanalles:CAPAE1030X1050D1200L350X90N, symbol Device:C_Small
- added C?: 0.1uF, vanalles:0603, symbol Device:C
- added C?: 68uF/100V, vanalles:CAPAE1030X1050D1200L350X90N, symbol Device:C_Small
- added C?: 0.1uF, vanalles:0603, symbol Device:C_Small
- added D?: MBRM5100, halfgeleiders:DPAK, symbol Halfgelijders:diode4
- added L?: 100uH, vanalles:DO5022p, symbol Device:L
- added R?: 130Kohm/1%, vanalles:0603, symbol Device:R_Small_US
- added R?: 43.5Kohm/1%, vanalles:0603, symbol Device:R_Small_US
- added TP?: 3V3, symbol Connector:Test_Point_Probe
- added U?: MAX5035AUSA, halfgeleiders:soic HV clearance, symbol Regulator_Switching:MAX5035AUSA
Connections:
- net +3V3: now also C?.1, L?.2, TP?.1, U?.4 (FB)
- net GND: now also C?.2, C?.2, C?.2, C?.2, D?.1, D?.3, R?.2, U?.3 (SGND), U?.6 (GND)
- net VIN: now also C?.1, C?.1, R?.1, U?.7 (VIN)
- new net: C?.1, U?.1 (BST)
- new net: C?.2, D?.4, L?.1, U?.8 (LX)
- new net: R?.1, R?.2, U?.5 (ON/~{OFF})
- new net: C?.1, U?.2 (VD)

Commit message: sdf
fsgv
Connections:
- net VIN renamed VIN DC_DC
Changed lines of the file:
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@@
     (stroke (width 0) (type solid) (color 0 0 0 0))
   )
-  (hierarchical_label "VIN" (shape input) (at 30.48 57.785 180)
+  (hierarchical_label "VIN DC_DC" (shape input) (at 30.48 57.785 180)
     (effects (font (size 1.27 1.27)) (justify right))
   )

Commit message: versie 3
verscie 3 afgetekend
Parts:
- removed TP?: 3V3, symbol Connector:Test_Point_Probe
- gave numbers to parts that had none: 10
Changed lines of the file:
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@@
   (junction (at 231.14 57.785) (diameter 0.9144) (color 0 0 0 0))
   (junction (at 241.3 57.785) (diameter 0.9144) (color 0 0 0 0))
-  (junction (at 252.73 57.785) (diameter 0.9144) (color 0 0 0 0))
   (wire (pts (xy 30.48 57.785) (xy 45.72 57.785))
     (stroke (width 0) (type solid) (color 0 0 0 0))
@@
   )
   (wire (pts (xy 252.73 52.07) (xy 252.73 57.785))
-    (stroke (width 0) (type solid) (color 0 0 0 0))
-  )
-  (wire (pts (xy 252.73 57.785) (xy 260.985 57.785))
     (stroke (width 0) (type solid) (color 0 0 0 0))
   )
@@
   (symbol (lib_id "power:+3V3") (at 252.73 52.07 0) (unit 1)
     (in_bom yes) (on_board yes)
-    (property "Reference" "#PWR?" (id 0) (at 252.73 55.88 0)
+    (property "Reference" "#PWR0113" (id 0) (at 252.73 55.88 0)
       (effects (font (size 1.27 1.27)) hide)
     )
@@
   (symbol (lib_id "power:GND") (at 45.72 83.185 0) (unit 1)
     (in_bom yes) (on_board yes) (fields_autoplaced)
-    (property "Reference" "#PWR?" (id 0) (at 45.72 89.535 0)
+    (property "Reference" "#PWR0109" (id 0) (at 45.72 89.535 0)
       (effects (font (size 1.27 1.27)) hide)
     )
@@
   (symbol (lib_id "power:GND") (at 66.04 83.185 0) (unit 1)
     (in_bom yes) (on_board yes) (fields_autoplaced)
-    (property "Reference" "#PWR?" (id 0) (at 66.04 89.535 0)
+    (property "Reference" "#PWR0110" (id 0) (at 66.04 89.535 0)
       (effects (font (size 1.27 1.27)) hide)
     )
@@
   (symbol (lib_id "power:GND") (at 95.25 84.455 0) (unit 1)
     (in_bom yes) (on_board yes) (fields_autoplaced)
-    (property "Reference" "#PWR?" (id 0) (at 95.25 90.805 0)
+    (property "Reference" "#PWR0111" (id 0) (at 95.25 90.805 0)
       (effects (font (size 1.27 1.27)) hide)
     )
@@
   (symbol (lib_id "power:GND") (at 160.02 92.075 0) (unit 1)
     (in_bom yes) (on_board yes) (fields_autoplaced)
-    (property "Reference" "#PWR?" (id 0) (at 160.02 98.425 0)
+    (property "Reference" "#PWR0108" (id 0) (at 160.02 98.425 0)
       (effects (font (size 1.27 1.27)) hide)
     )
@@
   (symbol (lib_id "power:GND") (at 201.93 74.93 0) (unit 1)
     (in_bom yes) (on_board yes) (fields_autoplaced)
-    (property "Reference" "#PWR?" (id 0) (at 201.93 81.28 0)
+    (property "Reference" "#PWR0112" (id 0) (at 201.93 81.28 0)
       (effects (font (size 1.27 1.27)) hide)
     )
@@
   (symbol (lib_id "power:GND") (at 241.3 76.835 0) (unit 1)
     (in_bom yes) (on_board yes) (fields_autoplaced)
-    (property "Reference" "#PWR?" (id 0) (at 241.3 83.185 0)
+    (property "Reference" "#PWR0114" (id 0) (at 241.3 83.185 0)
       (effects (font (size 1.27 1.27)) hide)
     )
@@
   (symbol (lib_id "Device:L") (at 219.71 57.785 90) (unit 1)
     (in_bom yes) (on_board yes) (fields_autoplaced)
-    (property "Reference" "L?" (id 0) (at 219.71 51.435 90))
+    (property "Reference" "L1" (id 0) (at 219.71 51.435 90))
     (property "Value" "100uH" (id 1) (at 219.71 53.975 90))
     (property "Footprint" "vanalles:DO5022p" (id 2) (at 219.71 57.785 0)
@@
   (symbol (lib_id "Device:R_Small_US") (at 95.25 65.405 0) (unit 1)
     (in_bom yes) (on_board yes) (fields_autoplaced)
-    (property "Reference" "R?" (id 0) (at 97.79 64.1349 0)
+    (property "Reference" "R8" (id 0) (at 97.79 64.1349 0)
       (effects (font (size 1.27 1.27)) (justify left))
     )
@@
   (symbol (lib_id "Device:R_Small_US") (at 95.25 75.565 0) (unit 1)
     (in_bom yes) (on_board yes) (fields_autoplaced)
-    (property "Reference" "R?" (id 0) (at 97.79 74.2949 0)
+    (property "Reference" "R9" (id 0) (at 97.79 74.2949 0)
       (effects (font (size 1.27 1.27)) (justify left))
     )
@@
     (pin "2")
   )
-  (symbol (lib_id "Connector:Test_Point_Probe") (at 260.985 57.785 0) (unit 1)
-    (in_bom yes) (on_board yes) (fields_autoplaced)
-    (property "Reference" "TP?" (id 0) (at 265.43 55.1179 0)
-      (effects (font (size 1.27 1.27)) (justify left))
-    )
-    (property "Value" "3V3" (id 1) (at 265.43 57.6579 0)
-      (effects (font (size 1.27 1.27)) (justify left))
-    )
-    (property "Footprint" "" (id 2) (at 266.065 57.785 0)
-      (effects (font (size 1.27 1.27)) hide)
-    )
-    (property "Datasheet" "" (id 3) (at 266.065 57.785 0)
-      (effects (font (size 1.27 1.27)) hide)
-    )
-    (pin "1")
-  )
   (symbol (lib_id "Device:C_Polarized_Small_US") (at 241.3 67.945 0) (unit 1)
     (in_bom yes) (on_board yes) (fields_autoplaced)
-    (property "Reference" "C?" (id 0) (at 243.84 66.6749 0)
+    (property "Reference" "C7" (id 0) (at 243.84 66.6749 0)
       (effects (font (size 1.27 1.27)) (justify left))
     )
@@
   (symbol (lib_id "Device:C_Small") (at 45.72 70.485 0) (unit 1)
     (in_bom yes) (on_board yes) (fields_autoplaced)
-    (property "Reference" "C?" (id 0) (at 48.26 69.2149 0)
+    (property "Reference" "C3" (id 0) (at 48.26 69.2149 0)
       (effects (font (size 1.27 1.27)) (justify left))
     )
@@
   (symbol (lib_id "Device:C_Small") (at 66.04 70.485 0) (unit 1)
     (in_bom yes) (on_board yes) (fields_autoplaced)
-    (property "Reference" "C?" (id 0) (at 68.58 69.2149 0)
+    (property "Reference" "C4" (id 0) (at 68.58 69.2149 0)
       (effects (font (size 1.27 1.27)) (justify left))
     )
@@
   (symbol (lib_id "Device:C_Small") (at 143.51 74.295 0) (unit 1)
     (in_bom yes) (on_board yes) (fields_autoplaced)
-    (property "Reference" "C?" (id 0) (at 146.05 73.0249 0)
+    (property "Reference" "C5" (id 0) (at 146.05 73.0249 0)
       (effects (font (size 1.27 1.27)) (justify left))
     )
@@
   (symbol (lib_id "Device:C") (at 189.23 57.785 90) (unit 1)
     (in_bom yes) (on_board yes) (fields_autoplaced)
-    (property "Reference" "C?" (id 0) (at 189.23 50.165 90))
+    (property "Reference" "C6" (id 0) (at 189.23 50.165 90))
     (property "Value" "0.1uF" (id 1) (at 189.23 52.705 90))
     (property "Footprint" "vanalles:0603" (id 2) (at 193.04 56.8198 0)
@@
   (symbol (lib_id "Halfgelijders:diode4") (at 201.93 67.945 0) (unit 1)
     (in_bom yes) (on_board yes) (fields_autoplaced)
-    (property "Reference" "D?" (id 0) (at 204.47 64.1349 0)
+    (property "Reference" "D1" (id 0) (at 204.47 64.1349 0)
       (effects (font (size 1.27 1.27)) (justify left))
     )
@@
   (symbol (lib_id "Regulator_Switching:MAX5035AUSA") (at 160.02 62.865 0) (unit 1)
     (in_bom yes) (on_board yes) (fields_autoplaced)
-    (property "Reference" "U?" (id 0) (at 160.02 50.165 0))
+    (property "Reference" "U3" (id 0) (at 160.02 50.165 0))
     (property "Value" "MAX5035AUSA" (id 1) (at 160.02 52.705 0))
     (property "Footprint" "halfgeleiders:soic HV clearance" (id 2) (at 163.83 71.755 0)
