File: pcb/asset tracker LoRa/lora tracker V3/Lora_tracker_V3/GPS.kicad_sch (KiCad schematic)
At the start: 7 parts

Commit message: versie 3
verscie 3 afgetekend
Parts:
- gave numbers to parts that had none: 7
Changed lines of the file:
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@@
   (symbol (lib_id "power:+3V3") (at 109.22 45.085 0) (unit 1)
     (in_bom yes) (on_board yes) (fields_autoplaced)
-    (property "Reference" "#PWR?" (id 0) (at 109.22 48.895 0)
+    (property "Reference" "#PWR0150" (id 0) (at 109.22 48.895 0)
       (effects (font (size 1.27 1.27)) hide)
     )
@@
   (symbol (lib_id "Device:L_Small") (at 167.64 93.345 90) (unit 1)
     (in_bom yes) (on_board yes) (fields_autoplaced)
-    (property "Reference" "L?" (id 0) (at 167.64 89.535 90))
+    (property "Reference" "L2" (id 0) (at 167.64 89.535 90))
     (property "Value" "5n6" (id 1) (at 167.64 92.075 90))
     (property "Footprint" "vanalles:0603" (id 2) (at 167.64 93.345 0)
@@
   (symbol (lib_id "power:GND") (at 85.09 95.885 270) (unit 1)
     (in_bom yes) (on_board yes) (fields_autoplaced)
-    (property "Reference" "#PWR?" (id 0) (at 78.74 95.885 0)
+    (property "Reference" "#PWR0148" (id 0) (at 78.74 95.885 0)
       (effects (font (size 1.27 1.27)) hide)
     )
@@
   (symbol (lib_id "power:GND") (at 116.84 130.175 0) (unit 1)
     (in_bom yes) (on_board yes) (fields_autoplaced)
-    (property "Reference" "#PWR?" (id 0) (at 116.84 136.525 0)
+    (property "Reference" "#PWR0152" (id 0) (at 116.84 136.525 0)
       (effects (font (size 1.27 1.27)) hide)
     )
@@
   (symbol (lib_id "power:GND") (at 132.08 66.675 0) (unit 1)
     (in_bom yes) (on_board yes) (fields_autoplaced)
-    (property "Reference" "#PWR?" (id 0) (at 132.08 73.025 0)
+    (property "Reference" "#PWR0149" (id 0) (at 132.08 73.025 0)
       (effects (font (size 1.27 1.27)) hide)
     )
@@
   (symbol (lib_id "power:GND") (at 168.91 108.585 0) (unit 1)
     (in_bom yes) (on_board yes) (fields_autoplaced)
-    (property "Reference" "#PWR?" (id 0) (at 168.91 114.935 0)
+    (property "Reference" "#PWR0151" (id 0) (at 168.91 114.935 0)
       (effects (font (size 1.27 1.27)) hide)
     )
@@
   (symbol (lib_id "Device:C_Small") (at 128.27 59.055 0) (unit 1)
     (in_bom yes) (on_board yes)
-    (property "Reference" "C?" (id 0) (at 128.27 57.1499 0)
+    (property "Reference" "C17" (id 0) (at 128.27 57.1499 0)
       (effects (font (size 1.27 1.27)) (justify left))
     )
@@
   (symbol (lib_id "Device:C_Small") (at 137.16 60.325 0) (unit 1)
     (in_bom yes) (on_board yes)
-    (property "Reference" "C?" (id 0) (at 137.16 58.4199 0)
+    (property "Reference" "C18" (id 0) (at 137.16 58.4199 0)
       (effects (font (size 1.27 1.27)) (justify left))
     )
@@
   (symbol (lib_id "Device:C_Small") (at 176.53 93.345 90) (unit 1)
     (in_bom yes) (on_board yes) (fields_autoplaced)
-    (property "Reference" "C?" (id 0) (at 176.53 88.265 90))
+    (property "Reference" "C19" (id 0) (at 176.53 88.265 90))
     (property "Value" "120nF" (id 1) (at 176.53 90.805 90))
     (property "Footprint" "vanalles:0603" (id 2) (at 176.53 93.345 0)
@@
   (symbol (lib_id "Device:Battery_Cell") (at 92.71 95.885 270) (unit 1)
     (in_bom yes) (on_board yes)
-    (property "Reference" "BT?" (id 0) (at 93.98 89.535 90))
+    (property "Reference" "BT1" (id 0) (at 93.98 89.535 90))
     (property "Value" "Battery_Cell" (id 1) (at 93.98 92.075 90))
     (property "Footprint" "vanalles:3012TR" (id 2) (at 94.234 95.885 90)
@@
   (symbol (lib_id "Device:Antenna_Shield") (at 194.31 93.345 270) (unit 1)
     (in_bom yes) (on_board yes) (fields_autoplaced)
-    (property "Reference" "AE?" (id 0) (at 200.66 93.4719 90)
+    (property "Reference" "AE2" (id 0) (at 200.66 93.4719 90)
       (effects (font (size 1.27 1.27)) (justify left))
     )
@@
   (symbol (lib_id "modulles:teseo-LIV") (at 127 90.805 0) (unit 1)
     (in_bom yes) (on_board yes) (fields_autoplaced)
-    (property "Reference" "MOD?" (id 0) (at 140.335 85.725 0))
+    (property "Reference" "MOD2" (id 0) (at 140.335 85.725 0))
     (property "Value" "teseo-LIV" (id 1) (at 140.335 88.265 0))
     (property "Footprint" "Module:SON_STM_TESEO-LIV3R" (id 2) (at 127 90.805 0)
