File: pcb/asset tracker LoRa/lora tracker V3/Lora_tracker_V3/Lora_RFM.kicad_sch (KiCad schematic)
At the start: 5 parts

Commit message: versie 3
verscie 3 afgetekend
Parts:
- gave numbers to parts that had none: 5
Changed lines of the file:
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@@
   (symbol (lib_id "power:+3V3") (at 66.04 69.215 0) (unit 1)
     (in_bom yes) (on_board yes) (fields_autoplaced)
-    (property "Reference" "#PWR?" (id 0) (at 66.04 73.025 0)
+    (property "Reference" "#PWR0137" (id 0) (at 66.04 73.025 0)
       (effects (font (size 1.27 1.27)) hide)
     )
@@
   (symbol (lib_id "power:+3V3") (at 156.21 43.815 0) (unit 1)
     (in_bom yes) (on_board yes) (fields_autoplaced)
-    (property "Reference" "#PWR?" (id 0) (at 156.21 47.625 0)
+    (property "Reference" "#PWR0136" (id 0) (at 156.21 47.625 0)
       (effects (font (size 1.27 1.27)) hide)
     )
@@
   (symbol (lib_id "power:GND") (at 134.62 107.315 0) (unit 1)
     (in_bom yes) (on_board yes)
-    (property "Reference" "#PWR?" (id 0) (at 134.62 113.665 0)
+    (property "Reference" "#PWR0138" (id 0) (at 134.62 113.665 0)
       (effects (font (size 1.27 1.27)) hide)
     )
@@
   (symbol (lib_id "power:GND") (at 184.15 69.215 0) (unit 1)
     (in_bom yes) (on_board yes)
-    (property "Reference" "#PWR?" (id 0) (at 184.15 75.565 0)
+    (property "Reference" "#PWR0135" (id 0) (at 184.15 75.565 0)
       (effects (font (size 1.27 1.27)) hide)
     )
@@
   (symbol (lib_id "Device:R_Small_US") (at 66.04 71.755 0) (unit 1)
     (in_bom yes) (on_board yes) (fields_autoplaced)
-    (property "Reference" "R?" (id 0) (at 68.58 71.1199 0)
+    (property "Reference" "R14" (id 0) (at 68.58 71.1199 0)
       (effects (font (size 1.27 1.27)) (justify left))
     )
@@
   (symbol (lib_id "Device:C_Small") (at 173.99 57.785 0) (unit 1)
     (in_bom yes) (on_board yes) (fields_autoplaced)
-    (property "Reference" "C?" (id 0) (at 176.53 57.1499 0)
+    (property "Reference" "C14" (id 0) (at 176.53 57.1499 0)
       (effects (font (size 1.27 1.27)) (justify left))
     )
@@
   (symbol (lib_id "Device:C_Small") (at 184.15 57.785 0) (unit 1)
     (in_bom yes) (on_board yes) (fields_autoplaced)
-    (property "Reference" "C?" (id 0) (at 186.69 57.1499 0)
+    (property "Reference" "C15" (id 0) (at 186.69 57.1499 0)
       (effects (font (size 1.27 1.27)) (justify left))
     )
@@
   (symbol (lib_id "Device:C_Small") (at 194.31 57.785 0) (unit 1)
     (in_bom yes) (on_board yes) (fields_autoplaced)
-    (property "Reference" "C?" (id 0) (at 196.85 57.1499 0)
+    (property "Reference" "C16" (id 0) (at 196.85 57.1499 0)
       (effects (font (size 1.27 1.27)) (justify left))
     )
@@
   (symbol (lib_id "RFM98W-433S2:RFM98W-433S2") (at 107.95 92.075 0) (unit 1)
     (in_bom yes) (on_board yes) (fields_autoplaced)
-    (property "Reference" "MOD?" (id 0) (at 107.95 70.485 0))
+    (property "Reference" "MOD1" (id 0) (at 107.95 70.485 0))
     (property "Value" "RFM98W-433S2" (id 1) (at 107.95 73.025 0))
     (property "Footprint" "Module:XCVR_RFM98W-433S2" (id 2) (at 107.95 92.075 0)
