File: pcb/asset tracker LoRa/lora tracker V3/Lora_tracker_V3/Lora_tracker_V3.kicad_pcb (KiCad board)
At the start: 0 parts

Commit message: versie 3
verscie 3 afgetekend
Parts:
- added AE1: Antenna_Shield, connectors_user:ufl connector, F.Cu at (95.2, 140.3)
- added AE2: sma, connectors_user:ufl connector, F.Cu at (133.9, 139.9)
- added BT1: Battery_Cell, vanalles:3012TR, F.Cu at (147.4, 128.3)
- added C1: NM, vanalles:0603, F.Cu at (96.2, 131.5)
- added C10: 100nF, vanalles:0603, F.Cu at (151.9, 101.0)
- added C11: 10uF, vanalles:0603, F.Cu at (122.2, 139.5)
- added C12: 100nF, vanalles:0603, F.Cu at (122.1, 137.7)
- added C13: 10uF, vanalles:0603, F.Cu at (151.9, 98.3)
- added C14: 10uF, vanalles:0603, F.Cu at (104.0, 132.0)
- added C15: 1uF, vanalles:0603, F.Cu at (104.0, 134.8)
- added C16: 0.1uF, vanalles:0603, F.Cu at (103.9, 138.2)
- added C17: 10uF, vanalles:0603, F.Cu at (122.4, 123.8)
- added C18: 100nF, vanalles:0603, F.Cu at (125.1, 123.8)
- added C19: 120nF, vanalles:0603, F.Cu at (128.3, 137.3)
- added C2: NM, vanalles:0603, F.Cu at (92.4, 134.9)
- added C20: 10uF, vanalles:0603, F.Cu at (116.8, 45.2)
- added C21: 10nF, vanalles:0603, F.Cu at (116.8, 42.8)
- added C3: 68uF/100V, vanalles:CAPAE1030X1050D1200L350X90N, F.Cu at (98.5, 42.1)
- added C4: 0.22uF/100V, vanalles:CAPAE1030X1050D1200L350X90N, F.Cu at (85.9, 42.5)
- added C5: 0.1uF, vanalles:0603, F.Cu at (91.9, 64.2)
- added C6: 0.1uF, vanalles:0603, F.Cu at (87.6, 64.5)
- added C7: 68uF/10V, vanalles:CAPAE1030X1050D1200L350X90N, F.Cu at (69.5, 43.0)
- added C8: 10uF, vanalles:0603, F.Cu at (152.1, 111.3)
- added C9: 100nF, vanalles:0603, F.Cu at (152.0, 109.0)
- added CON1: TAGconnect_ESP, connectors_user:Tag-Connect_TC2030-IDC-NL_2x03_P1.27mm_Vertical, F.Cu at (69.2, 121.2)
- added D1: MBRM5100, halfgeleiders:DPAK, F.Cu at (84.7, 73.7)
- added J1: Screw_Terminal_01x02, connectors_user:2pin_screw, F.Cu at (165.2, 82.9)
- added JP1: Jumper_2_Open, vanalles:SolderJumper-2_P1.3mm_Open_Pad1.0x1.5mm, F.Cu at (151.0, 55.5)
- added L1: 100uH, vanalles:DO5022p, F.Cu at (79.6, 57.3)
- added L2: 5n6, vanalles:0603, F.Cu at (128.4, 133.5)
- added MOD1: RFM98W-433S2, Module:XCVR_RFM98W-433S2, F.Cu at (102.3, 119.8)
- added MOD2: teseo-LIV, Module:SON_STM_TESEO-LIV3R, F.Cu at (131.7, 124.4)
- added PZ1: buzzer, vanalles:PROSIGNAL_ABI-017-RC, F.Cu at (162.7, 105.1)
- added Q1: BSS84, halfgeleiders:sot-23,, F.Cu at (161.7, 118.7)
- added R1: 0, vanalles:0603RL, F.Cu at (95.4, 134.2)
- added R10: 10K, vanalles:0603, F.Cu at (162.8, 124.8)
- added R11: 220, vanalles:0603, F.Cu at (148.3, 77.7)
- added R12: 10K, vanalles:0603, F.Cu at (115.2, 136.6)
- added R13: 10K, vanalles:0603, F.Cu at (115.4, 133.1)
- added R14: 10K, vanalles:0603RL, F.Cu at (101.4, 105.1)
- added R15: 10K, vanalles:0603RL, F.Cu at (72.3, 116.3)
- added R16: 10K, vanalles:0603RL, F.Cu at (81.3, 90.3)
- added R17: NM, vanalles:0603RL, F.Cu at (85.0, 90.3)
- added R2: 1Mohm, vanalles:0603, F.Cu at (159.9, 62.7)
- added R3: 58Kohm, vanalles:0603, F.Cu at (159.8, 58.1)
- added R4: 900K, vanalles:0603, F.Cu at (145.1, 45.6)
- added R5: 58K, vanalles:0603, F.Cu at (156.7, 45.6)
- added R6: 1K ohm, vanalles:0603, F.Cu at (124.1, 43.7)
- added R7: 1Kohm, vanalles:0603, F.Cu at (137.4, 44.0)
- added R8: 43.5Kohm/1%, vanalles:0603, F.Cu at (92.2, 50.5)
- added R9: 130Kohm/1%, vanalles:0603, F.Cu at (95.3, 51.7)
- added RV1: 100K, vanalles:3314G-1-201E bourns trimmer, F.Cu at (149.8, 45.7)
- added U1: TLP3542, halfgeleiders:TLP3542, F.Cu at (126.1, 37.1)
- added U2: TLP3542, halfgeleiders:TLP3542, F.Cu at (139.4, 37.5)
- added U3: MAX5035AUSA, halfgeleiders:soic HV clearance, F.Cu at (86.9, 61.1)
- added U4: LIS3DH, halfgeleiders:QFN-16_0.5MM, F.Cu at (149.6, 105.4)
- added U5: G3VM-61HR2(TR05), halfgeleiders:sop4 P=2.54, F.Cu at (155.4, 83.6)
- added U6: DS28CM00R-A00+T, halfgeleiders:SOT-25, F.Cu at (120.0, 134.1)
- added U7: ATECC608B, halfgeleiders:soic p1.27 lengt 5.40, F.Cu at (156.7, 94.9)
- added U8: ESP32-WROOM, Module:ESP32-WROOM-32, F.Cu at (74.8, 103.0)
- added U9: MLX91221, halfgeleiders:SOIC-8, F.Cu at (111.5, 40.6)
- added con1: screw terminal, connectors_user:2pin_screw, F.Cu at (164.5, 65.9)
- added con2: xt60, connectors_user:AMASS_XT60PW-F, F.Cu at (167.9, 44.1)
- added kibuzzard-6130D8CD: G***, kibuzzard-6130D8CD, F.Cu at (164.7, 57.0)
- added kibuzzard-6130D8CD: G***, kibuzzard-6130D8CD, F.Cu at (162.3, 34.1)
Routing:
- net GND: track 0.00 -> 150.4 mm, vias 0 -> 39
- net VDC: track 0.00 -> 120.5 mm
- net Net-(R2-Pad1): track 0.00 -> 65.1 mm, vias 0 -> 1
- net /voeding/DC_DC/VIN DC_DC: track 0.00 -> 49.2 mm, vias 0 -> 1
- net /esp32/GPIO0: track 0.00 -> 45.9 mm, vias 0 -> 2
- net Net-(BT1-Pad1): track 0.00 -> 42.6 mm
- net Net-(R4-Pad1): track 0.00 -> 36.5 mm, vias 0 -> 1
- net /esp32/RX: track 0.00 -> 31.9 mm, vias 0 -> 2
- net /esp32/TX: track 0.00 -> 27.0 mm, vias 0 -> 2
- net Net-(C6-Pad2): track 0.00 -> 26.3 mm
- net Net-(J1-Pad2): track 0.00 -> 21.0 mm
- net Net-(JP1-Pad1): track 0.00 -> 13.6 mm
- net Net-(R8-Pad2): track 0.00 -> 12.9 mm
- net /esp32/RESET: track 0.00 -> 11.5 mm
- net Net-(PZ1-Pad1): track 0.00 -> 7.65 mm
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- added copper zone on F.Cu, net +3V3
- added copper zone on B.Cu, net GND
Other:
- board outline added: 116.3 x 114.5 mm
- copper layers 0 -> 2
