File: pcb/asset tracker LoRa/lora tracker V3/Lora_tracker_V3/Lora_tracker_V3.kicad_pcb (KiCad board)
At the start: 2 copper layers, 116.3 x 114.5 mm, 65 parts, among them CON1 TAGconnect_ESP, J1 Screw_Terminal_01x02, Q1 BSS84, U1 TLP3542, U2 TLP3542, U3 MAX5035AUSA, U4 LIS3DH, U5 G3VM-61HR2(TR05), U6 DS28CM00R-A00+T, U7 ATECC608B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

Commit message: v3
v3 bijna af
Parts:
- removed R7: 1Kohm, vanalles:0603
- removed U1, U2: TLP3542, halfgeleiders:TLP3542
- removed kibuzzard-6130D8CD (x2): G***, kibuzzard-6130D8CD
- added Q2: BSS138, halfgeleiders:sot-23,, F.Cu at (155.6, 52.4)
- added RL1: Relais, vanalles:G5V-1, F.Cu at (161.6, 53.3)
- added kibuzzard-61389C09: G***, kibuzzard-61389C09, F.Cu at (189.6, 34.2)
- added kibuzzard-61389C09: G***, kibuzzard-61389C09, F.Cu at (186.1, 58.7)
- added kibuzzard-61389CC5: G***, kibuzzard-61389CC5, F.Cu at (174.3, 62.8)
- Q1: value BSS84 -> BSS138
- R6: value 1K ohm -> 10K
- moved C3 68.4 mm to (166.4, 34.1), turned to 0 degrees
- moved AE2 65.0 mm to (80.8, 102.4), turned to 90 degrees
- moved C4 62.0 mm to (147.5, 34.8), turned to 0 degrees
- moved D1 61.5 mm to (134.6, 37.7), turned to 180 degrees
- moved C19 55.4 mm to (85.4, 102.4), turned to 180 degrees
- moved C2 52.3 mm to (144.7, 134.1)
- moved C16 51.4 mm to (154.6, 129.3)
- moved C15 50.7 mm to (154.6, 131.2)
- moved C14 50.7 mm to (154.6, 133.3)
- moved U7 50.5 mm to (111.9, 118.1), turned to 0 degrees
- moved MOD1 50.2 mm to (152.4, 117.1)
- moved L2 50.2 mm to (89.0, 102.4), turned to 180 degrees
- moved R1 50.2 mm to (145.5, 131.2)
- moved C1 50.1 mm to (146.2, 128.4)
- moved R14 49.9 mm to (151.3, 103.6)
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Connections:
- R6 pad 1: /voeding/SSR1_IN -> GND
- R6 pad 2: Net-(R6-Pad2) -> /voeding/Relay control
Routing:
- net GND: track 150.4 -> 186.9 mm, vias 39 -> 32
- net Net-(R2-Pad1): track 65.1 -> 32.6 mm, vias 1 -> 0
- net Net-(BT1-Pad1): track 42.6 -> 62.2 mm
- net Net-(Q2-Pad3): track 0.00 -> 10.5 mm
- net Net-(J1-Pad2): track 21.0 -> 12.7 mm
- net Net-(R8-Pad2): track 12.9 -> 6.61 mm
- net /esp32/RX: track 31.9 -> 36.4 mm
- net Net-(C6-Pad2): track 26.3 -> 22.4 mm
- net /esp32/RESET: track 11.5 -> 15.4 mm
- net /voeding/DC_DC/VIN DC_DC: track 49.2 -> 52.8 mm, vias 1 -> 0
- net Net-(AE2-Pad1): track 5.96 -> 2.46 mm
- net /esp32/TX: track 27.0 -> 30.3 mm
- net Net-(R6-Pad2): track 2.81 -> 0.00 mm
- net /voeding/Relay control: track 0.00 -> 2.71 mm
- net Net-(R7-Pad2): track 2.64 -> 0.00 mm
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
Commit message: firmware
aan de firmware beginnen  schrijven
Parts:
- added C22: 10uF, vanalles:0603, F.Cu at (168.9, 110.2)
- added C23: 100nF, vanalles:0603, F.Cu at (171.3, 110.2)
- added DISP1: ConnectEVE, connectors_user:10pin header, F.Cu at (170.9, 128.0)
- added U1: STM32F407ZGTx, halfgeleiders:STM32F407ZGT6, F.Cu at (132.4, 80.5)
- added kibuzzard-613B3452: G***, kibuzzard-613B3452, F.Cu at (106.4, 69.6)
- added kibuzzard-613B3465: G***, kibuzzard-613B3465, F.Cu at (97.0, 98.8)
- added kibuzzard-613B6735: G***, kibuzzard-613B6735, F.Cu at (142.6, 116.6)
- added kibuzzard-613B6746: G***, kibuzzard-613B6746, F.Cu at (167.1, 136.0)
- added kibuzzard-613B6752: G***, kibuzzard-613B6752, F.Cu at (181.2, 121.1)
- added kibuzzard-613F18F5: G***, kibuzzard-613F18F5, F.Cu at (184.3, 45.5)
- added kibuzzard-613F1907: G***, kibuzzard-613F1907, F.Cu at (182.2, 65.1)
- moved C8 49.1 mm to (129.0, 132.8), turned to 90 degrees
- moved C9 46.5 mm to (131.9, 132.8), turned to 90 degrees
- moved U4 44.8 mm to (127.8, 136.7)
Connections:
- net /GPS/GPS_PPS renamed /PPS
- net /GPS/GPS_RESET renamed /RESET_GPS
- net /GPS/GPS_RX renamed /RX
- net /GPS/GPS_TX renamed /TX
- net /GPS/GPS_WAKE renamed /WAKE
- net /IO/BUZZER renamed /BUZZER
- net /IO/IN_SSR renamed /SSR
- net /Lora_RFM/CLK renamed /CLK
- net /Lora_RFM/CS renamed /CS
- net /Lora_RFM/MISO renamed /MISO
- net /Lora_RFM/MOSI renamed /MOSI
- net /Lora_RFM/RESET renamed /RESET_LORA
- net /beweging/LIS_INT1 renamed /LIS_INT1
- net /beweging/LIS_INT2 renamed /LIS_INT2
- net /voeding/CURRENT_OUT1 renamed /Current
- net /voeding/Relay control renamed /RELAY
- net /voeding/VM0 renamed /Voltage1
- net /voeding/VM1 renamed /voltage2
- R12 pad 2: /IO/SDA_SERIAL_NR -> /SDA
- R13 pad 2: /IO/SCL_SERIAL_NR -> /SCL
- U4 pad 4: /beweging/LIS_SCL -> /SCL
- U4 pad 6: /beweging/LIS_SDA -> /SDA
- U6 pad 1: /IO/SCL_SERIAL_NR -> /SCL
- U6 pad 3: /IO/SDA_SERIAL_NR -> /SDA
- U7 pad 5: /IO/SDA_CRYPTO -> /SDA
- U7 pad 6: /IO/SCL_CRYPTO -> /SCL
- U8 pad 33: /esp32/ESP_SDA -> /SDA
- U8 pad 36: /esp32/ESP_SCL -> /SCL
Routing:
- net /SDA: track 0.00 -> 113.1 mm, vias 0 -> 7
- net /SCL: track 0.00 -> 112.7 mm, vias 0 -> 2
- net /CLK: track 0.00 -> 28.0 mm
- net /MISO: track 0.00 -> 25.7 mm
- net /MOSI: track 0.00 -> 23.5 mm, vias 0 -> 1
- net GND: track 186.9 -> 202.2 mm, vias 32 -> 44
- net /IO/SDA_SERIAL_NR: track 2.47 -> 0.00 mm
- net /IO/SCL_SERIAL_NR: track 2.32 -> 0.00 mm
- net /LIS_INT2: track 0.00 -> 1.95 mm
