File: pcb/asset tracker LoRa/lora tracker V3/Lora_tracker_V3/beweging.kicad_sch (KiCad schematic)
At the start: 3 parts

Commit message: sdf
fsgv
Changed lines of the file:
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@@
     (property "Reference" "U?" (id 0) (at 131.445 91.44 0))
     (property "Value" "LIS3DH" (id 1) (at 131.445 93.98 0))
-    (property "Footprint" "halfgeleiders:QFN-16_0.5MM" (id 2) (at 127.635 109.22 0))
+    (property "Footprint" "halfgeleiders:QFN-16_0.5MM" (id 2) (at 127.635 109.22 0)
+      (effects (font (size 1.27 1.27)) hide)
+    )
     (property "Datasheet" "https://www.st.com/resource/en/datasheet/cd00274221.pdf" (id 3) (at 120.015 85.09 0)
       (effects (font (size 1.27 1.27)) hide)

Commit message: versie 3
verscie 3 afgetekend
Parts:
- gave numbers to parts that had none: 3
Changed lines of the file:
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@@
   (symbol (lib_id "power:+3V3") (at 98.425 82.55 90) (unit 1)
     (in_bom yes) (on_board yes) (fields_autoplaced)
-    (property "Reference" "#PWR?" (id 0) (at 102.235 82.55 0)
+    (property "Reference" "#PWR0118" (id 0) (at 102.235 82.55 0)
       (effects (font (size 1.27 1.27)) hide)
     )
@@
   (symbol (lib_id "power:+3V3") (at 98.425 90.17 90) (unit 1)
     (in_bom yes) (on_board yes) (fields_autoplaced)
-    (property "Reference" "#PWR?" (id 0) (at 102.235 90.17 0)
+    (property "Reference" "#PWR0119" (id 0) (at 102.235 90.17 0)
       (effects (font (size 1.27 1.27)) hide)
     )
@@
   (symbol (lib_id "power:+3V3") (at 125.095 48.26 0) (unit 1)
     (in_bom yes) (on_board yes) (fields_autoplaced)
-    (property "Reference" "#PWR?" (id 0) (at 125.095 52.07 0)
+    (property "Reference" "#PWR0117" (id 0) (at 125.095 52.07 0)
       (effects (font (size 1.27 1.27)) hide)
     )
@@
   (symbol (lib_id "power:GND") (at 99.695 68.58 0) (unit 1)
     (in_bom yes) (on_board yes) (fields_autoplaced)
-    (property "Reference" "#PWR?" (id 0) (at 99.695 74.93 0)
+    (property "Reference" "#PWR0115" (id 0) (at 99.695 74.93 0)
       (effects (font (size 1.27 1.27)) hide)
     )
@@
   (symbol (lib_id "power:GND") (at 125.095 102.87 0) (unit 1)
     (in_bom yes) (on_board yes) (fields_autoplaced)
-    (property "Reference" "#PWR?" (id 0) (at 125.095 109.22 0)
+    (property "Reference" "#PWR0116" (id 0) (at 125.095 109.22 0)
       (effects (font (size 1.27 1.27)) hide)
     )
@@
   (symbol (lib_id "Device:C_Small") (at 95.885 60.96 0) (unit 1)
     (in_bom yes) (on_board yes)
-    (property "Reference" "C?" (id 0) (at 95.885 59.0549 0)
+    (property "Reference" "C8" (id 0) (at 95.885 59.0549 0)
       (effects (font (size 1.27 1.27)) (justify left))
     )
@@
   (symbol (lib_id "Device:C_Small") (at 104.775 62.23 0) (unit 1)
     (in_bom yes) (on_board yes)
-    (property "Reference" "C?" (id 0) (at 104.775 60.3249 0)
+    (property "Reference" "C9" (id 0) (at 104.775 60.3249 0)
       (effects (font (size 1.27 1.27)) (justify left))
     )
@@
   (symbol (lib_id "Sensor_Motion:LIS3DH") (at 125.095 82.55 0) (unit 1)
     (in_bom yes) (on_board yes)
-    (property "Reference" "U?" (id 0) (at 131.445 91.44 0))
+    (property "Reference" "U4" (id 0) (at 131.445 91.44 0))
     (property "Value" "LIS3DH" (id 1) (at 131.445 93.98 0))
     (property "Footprint" "halfgeleiders:QFN-16_0.5MM" (id 2) (at 127.635 109.22 0)
