File: pcb/asset tracker LoRa/lora tracker V3/Lora_tracker_V3/curent meseurment .kicad_sch (KiCad schematic)
At the start: 0 parts

Commit message: sdf
fsgv
Parts:
- added C?: 10nF, symbol Device:C_Small
- added C?: 10uF, symbol Device:C_Small
- added JP? (x2): Jumper_2_Open, symbol Jumper:Jumper_2_Open
- added R? (x4): R_Small_US, symbol Device:R_Small_US
- added U?: MCP6021, symbol Halfgelijders:MCP6021
- added U?: MLX91221, symbol Halfgelijders:MLX91221
Connections:
- new net: R?.1, R?.2, U?.4 (-)
- new net: R?.1, R?.2, U?.3 (+)
- new net: JP?.1 (A), JP?.2 (B), U?.7 (VOUT)
- new net: JP?.2 (B), R?.1
- new net +3V3: C?.1, C?.1, R?.2, U?.6 (VREF), U?.8 (VDD)
- new net CURRENT_OUT: JP?.1 (A), R?.2, U?.1 (OUT)
- new net GND: C?.2, C?.2, R?.1, U?.5 (GND)
- new net VIN_1: U?.1 (IP+), U?.2 (IP+)
- new net VOUT: U?.3 (IP-), U?.4 (IP-)

Commit message: versie 3
verscie 3 afgetekend
Parts:
- removed JP? (x2): Jumper_2_Open, symbol Jumper:Jumper_2_Open
- removed R? (x4): R_Small_US, symbol Device:R_Small_US
- removed U?: MCP6021, symbol Halfgelijders:MCP6021
- C20, C21: renamed from C?; footprint (none) -> vanalles:0603
- U9: renamed from U?; footprint (none) -> halfgeleiders:SOIC-8
Connections:
- net CURRENT_OUT: now also U9.7 (VOUT)
