File: pcb/asset tracker LoRa/lora tracker V3/Lora_tracker_V3/esp32.kicad_sch (KiCad schematic)
At the start: 5 parts

Commit message: versie 3
verscie 3 afgetekend
Parts:
- gave numbers to parts that had none: 5
Changed lines of the file:
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@@
   (symbol (lib_id "power:+3V3") (at 88.265 31.115 0) (unit 1)
     (in_bom yes) (on_board yes) (fields_autoplaced)
-    (property "Reference" "#PWR?" (id 0) (at 88.265 34.925 0)
+    (property "Reference" "#PWR0140" (id 0) (at 88.265 34.925 0)
       (effects (font (size 1.27 1.27)) hide)
     )
@@
   (symbol (lib_id "power:+3V3") (at 104.775 29.845 0) (unit 1)
     (in_bom yes) (on_board yes) (fields_autoplaced)
-    (property "Reference" "#PWR?" (id 0) (at 104.775 33.655 0)
+    (property "Reference" "#PWR0141" (id 0) (at 104.775 33.655 0)
       (effects (font (size 1.27 1.27)) hide)
     )
@@
   (symbol (lib_id "power:+3V3") (at 132.715 135.89 0) (unit 1)
     (in_bom yes) (on_board yes) (fields_autoplaced)
-    (property "Reference" "#PWR?" (id 0) (at 132.715 139.7 0)
+    (property "Reference" "#PWR0143" (id 0) (at 132.715 139.7 0)
       (effects (font (size 1.27 1.27)) hide)
     )
@@
   (symbol (lib_id "power:+3V3") (at 187.325 34.925 0) (unit 1)
     (in_bom yes) (on_board yes) (fields_autoplaced)
-    (property "Reference" "#PWR?" (id 0) (at 187.325 38.735 0)
+    (property "Reference" "#PWR0139" (id 0) (at 187.325 38.735 0)
       (effects (font (size 1.27 1.27)) hide)
     )
@@
   (symbol (lib_id "power:GND") (at 108.585 81.915 0) (unit 1)
     (in_bom yes) (on_board yes) (fields_autoplaced)
-    (property "Reference" "#PWR?" (id 0) (at 108.585 88.265 0)
+    (property "Reference" "#PWR0142" (id 0) (at 108.585 88.265 0)
       (effects (font (size 1.27 1.27)) hide)
     )
@@
   (symbol (lib_id "power:GND") (at 121.285 90.805 0) (unit 1)
     (in_bom yes) (on_board yes) (fields_autoplaced)
-    (property "Reference" "#PWR?" (id 0) (at 121.285 97.155 0)
+    (property "Reference" "#PWR0144" (id 0) (at 121.285 97.155 0)
       (effects (font (size 1.27 1.27)) hide)
     )
@@
   (symbol (lib_id "power:GND") (at 132.715 158.75 0) (unit 1)
     (in_bom yes) (on_board yes) (fields_autoplaced)
-    (property "Reference" "#PWR?" (id 0) (at 132.715 165.1 0)
+    (property "Reference" "#PWR0147" (id 0) (at 132.715 165.1 0)
       (effects (font (size 1.27 1.27)) hide)
     )
@@
   (symbol (lib_id "power:GND") (at 164.465 83.185 0) (unit 1)
     (in_bom yes) (on_board yes) (fields_autoplaced)
-    (property "Reference" "#PWR?" (id 0) (at 164.465 89.535 0)
+    (property "Reference" "#PWR0145" (id 0) (at 164.465 89.535 0)
       (effects (font (size 1.27 1.27)) hide)
     )
@@
   (symbol (lib_id "power:GND") (at 187.325 84.455 0) (unit 1)
     (in_bom yes) (on_board yes) (fields_autoplaced)
-    (property "Reference" "#PWR?" (id 0) (at 187.325 90.805 0)
+    (property "Reference" "#PWR0146" (id 0) (at 187.325 90.805 0)
       (effects (font (size 1.27 1.27)) hide)
     )
@@
   (symbol (lib_id "Device:R_Small_US") (at 88.265 37.465 0) (unit 1)
     (in_bom yes) (on_board yes) (fields_autoplaced)
-    (property "Reference" "R?" (id 0) (at 90.805 36.8299 0)
+    (property "Reference" "R15" (id 0) (at 90.805 36.8299 0)
       (effects (font (size 1.27 1.27)) (justify left))
     )
@@
   (symbol (lib_id "Device:R_Small_US") (at 187.325 41.275 0) (unit 1)
     (in_bom yes) (on_board yes) (fields_autoplaced)
-    (property "Reference" "R?" (id 0) (at 189.865 40.6399 0)
+    (property "Reference" "R16" (id 0) (at 189.865 40.6399 0)
       (effects (font (size 1.27 1.27)) (justify left))
     )
@@
   (symbol (lib_id "Device:R_Small_US") (at 187.325 79.375 0) (unit 1)
     (in_bom yes) (on_board yes) (fields_autoplaced)
-    (property "Reference" "R?" (id 0) (at 189.865 78.7399 0)
+    (property "Reference" "R17" (id 0) (at 189.865 78.7399 0)
       (effects (font (size 1.27 1.27)) (justify left))
     )
@@
   (symbol (lib_id "conectors:TAGconnect_ESP") (at 137.795 139.7 0) (unit 1)
     (in_bom yes) (on_board yes) (fields_autoplaced)
-    (property "Reference" "CON?" (id 0) (at 146.685 146.0499 0)
+    (property "Reference" "CON1" (id 0) (at 146.685 146.0499 0)
       (effects (font (size 1.27 1.27)) (justify left))
     )
@@
   (symbol (lib_id "ESP32:ESP32-WROOM") (at 132.715 60.325 0) (unit 1)
     (in_bom yes) (on_board yes) (fields_autoplaced)
-    (property "Reference" "U?" (id 0) (at 132.08 24.765 0)
+    (property "Reference" "U8" (id 0) (at 132.08 24.765 0)
       (effects (font (size 1.524 1.524)))
     )
