File: pcb/asset tracker LoRa/lora tracker V3/Lora_tracker_V3/Lora_tracker_V3.kicad_sch (KiCad schematic)
At the start: 4 parts

Commit message: dc
dsc
Other:
- sheet voeding ports: added VM0, VM1; removed none
Changed lines of the file:
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@@
   (junction (at 210.185 114.935) (diameter 0.9144) (color 0 0 0 0))
   (junction (at 229.235 114.935) (diameter 0.9144) (color 0 0 0 0))
+  (bus_entry (at 69.85 49.53) (size 2.54 2.54)
+    (stroke (width 0) (type solid) (color 0 0 0 0))
+  )
+  (bus_entry (at 69.85 52.705) (size 2.54 2.54)
+    (stroke (width 0) (type solid) (color 0 0 0 0))
+  )
+  (bus_entry (at 69.85 55.88) (size 2.54 2.54)
+    (stroke (width 0) (type solid) (color 0 0 0 0))
+  )
+  (bus_entry (at 69.85 59.055) (size 2.54 2.54)
+    (stroke (width 0) (type solid) (color 0 0 0 0))
+  )
+  (bus_entry (at 69.85 61.595) (size 2.54 2.54)
+    (stroke (width 0) (type solid) (color 0 0 0 0))
+  )
+  (bus_entry (at 69.85 78.74) (size 2.54 2.54)
+    (stroke (width 0) (type solid) (color 0 0 0 0))
+  )
+  (bus_entry (at 69.85 82.55) (size 2.54 2.54)
+    (stroke (width 0) (type solid) (color 0 0 0 0))
+  )
+  (bus_entry (at 69.85 85.09) (size 2.54 2.54)
+    (stroke (width 0) (type solid) (color 0 0 0 0))
+  )
+  (bus_entry (at 69.85 88.265) (size 2.54 2.54)
+    (stroke (width 0) (type solid) (color 0 0 0 0))
+  )
+  (bus_entry (at 69.85 103.505) (size 2.54 2.54)
+    (stroke (width 0) (type solid) (color 0 0 0 0))
+  )
+  (bus_entry (at 69.85 107.315) (size 2.54 2.54)
+    (stroke (width 0) (type solid) (color 0 0 0 0))
+  )
+  (bus_entry (at 69.85 111.125) (size 2.54 2.54)
+    (stroke (width 0) (type solid) (color 0 0 0 0))
+  )
+  (bus_entry (at 69.85 113.665) (size 2.54 2.54)
+    (stroke (width 0) (type solid) (color 0 0 0 0))
+  )
+  (bus_entry (at 69.85 116.84) (size 2.54 2.54)
+    (stroke (width 0) (type solid) (color 0 0 0 0))
+  )
+  (bus_entry (at 69.85 119.38) (size 2.54 2.54)
+    (stroke (width 0) (type solid) (color 0 0 0 0))
+  )
+  (bus_entry (at 156.845 60.96) (size 2.54 -2.54)
+    (stroke (width 0) (type solid) (color 0 0 0 0))
+  )
+  (bus_entry (at 156.845 63.5) (size 2.54 -2.54)
+    (stroke (width 0) (type solid) (color 0 0 0 0))
+  )
+  (bus_entry (at 156.845 85.725) (size 2.54 -2.54)
+    (stroke (width 0) (type solid) (color 0 0 0 0))
+  )
+  (bus_entry (at 156.845 88.265) (size 2.54 -2.54)
+    (stroke (width 0) (type solid) (color 0 0 0 0))
+  )
+  (bus_entry (at 156.845 90.805) (size 2.54 -2.54)
+    (stroke (width 0) (type solid) (color 0 0 0 0))
+  )
+  (bus_entry (at 156.845 93.345) (size 2.54 -2.54)
+    (stroke (width 0) (type solid) (color 0 0 0 0))
+  )
+  (bus_entry (at 156.845 95.885) (size 2.54 -2.54)
+    (stroke (width 0) (type solid) (color 0 0 0 0))
+  )
+  (bus_entry (at 156.845 110.49) (size 2.54 -2.54)
+    (stroke (width 0) (type solid) (color 0 0 0 0))
+  )
+  (bus_entry (at 156.845 113.665) (size 2.54 -2.54)
+    (stroke (width 0) (type solid) (color 0 0 0 0))
+  )
+  (bus_entry (at 156.845 116.84) (size 2.54 -2.54)
+    (stroke (width 0) (type solid) (color 0 0 0 0))
+  )
+  (bus_entry (at 156.845 119.38) (size 2.54 -2.54)
+    (stroke (width 0) (type solid) (color 0 0 0 0))
+  )
+  (bus_entry (at 156.845 121.92) (size 2.54 -2.54)
+    (stroke (width 0) (type solid) (color 0 0 0 0))
+  )
+  (wire (pts (xy 43.18 78.74) (xy 69.85 78.74))
+    (stroke (width 0) (type solid) (color 0 0 0 0))
+  )
+  (wire (pts (xy 43.18 82.55) (xy 69.85 82.55))
+    (stroke (width 0) (type solid) (color 0 0 0 0))
+  )
+  (wire (pts (xy 43.18 85.09) (xy 69.85 85.09))
+    (stroke (width 0) (type solid) (color 0 0 0 0))
+  )
+  (wire (pts (xy 43.18 88.265) (xy 69.85 88.265))
+    (stroke (width 0) (type solid) (color 0 0 0 0))
+  )
+  (wire (pts (xy 44.45 49.53) (xy 69.85 49.53))
+    (stroke (width 0) (type solid) (color 0 0 0 0))
+  )
+  (wire (pts (xy 44.45 52.705) (xy 69.85 52.705))
+    (stroke (width 0) (type solid) (color 0 0 0 0))
+  )
+  (wire (pts (xy 44.45 55.88) (xy 69.85 55.88))
+    (stroke (width 0) (type solid) (color 0 0 0 0))
+  )
+  (wire (pts (xy 44.45 59.055) (xy 69.85 59.055))
+    (stroke (width 0) (type solid) (color 0 0 0 0))
+  )
+  (wire (pts (xy 44.45 61.595) (xy 69.85 61.595))
+    (stroke (width 0) (type solid) (color 0 0 0 0))
+  )
+  (wire (pts (xy 48.26 103.505) (xy 69.85 103.505))
+    (stroke (width 0) (type solid) (color 0 0 0 0))
+  )
+  (wire (pts (xy 48.26 107.315) (xy 69.85 107.315))
+    (stroke (width 0) (type solid) (color 0 0 0 0))
+  )
+  (wire (pts (xy 48.26 111.125) (xy 69.85 111.125))
+    (stroke (width 0) (type solid) (color 0 0 0 0))
+  )
+  (wire (pts (xy 48.26 113.665) (xy 69.85 113.665))
+    (stroke (width 0) (type solid) (color 0 0 0 0))
+  )
+  (wire (pts (xy 48.26 116.84) (xy 69.85 116.84))
+    (stroke (width 0) (type solid) (color 0 0 0 0))
+  )
+  (wire (pts (xy 48.26 119.38) (xy 69.85 119.38))
+    (stroke (width 0) (type solid) (color 0 0 0 0))
+  )
+  (wire (pts (xy 159.385 58.42) (xy 173.355 58.42))
+    (stroke (width 0) (type solid) (color 0 0 0 0))
+  )
+  (wire (pts (xy 159.385 60.96) (xy 173.355 60.96))
+    (stroke (width 0) (type solid) (color 0 0 0 0))
+  )
+  (wire (pts (xy 159.385 83.185) (xy 173.355 83.185))
+    (stroke (width 0) (type solid) (color 0 0 0 0))
+  )
+  (wire (pts (xy 159.385 85.725) (xy 173.355 85.725))
+    (stroke (width 0) (type solid) (color 0 0 0 0))
+  )
+  (wire (pts (xy 159.385 88.265) (xy 173.355 88.265))
+    (stroke (width 0) (type solid) (color 0 0 0 0))
+  )
+  (wire (pts (xy 159.385 90.805) (xy 173.355 90.805))
+    (stroke (width 0) (type solid) (color 0 0 0 0))
+  )
+  (wire (pts (xy 159.385 93.345) (xy 173.355 93.345))
+    (stroke (width 0) (type solid) (color 0 0 0 0))
+  )
+  (wire (pts (xy 159.385 107.95) (xy 173.355 107.95))
+    (stroke (width 0) (type solid) (color 0 0 0 0))
+  )
+  (wire (pts (xy 159.385 111.125) (xy 173.355 111.125))
+    (stroke (width 0) (type solid) (color 0 0 0 0))
+  )
+  (wire (pts (xy 159.385 114.3) (xy 173.355 114.3))
+    (stroke (width 0) (type solid) (color 0 0 0 0))
+  )
+  (wire (pts (xy 159.385 116.84) (xy 173.355 116.84))
+    (stroke (width 0) (type solid) (color 0 0 0 0))
+  )
+  (wire (pts (xy 159.385 119.38) (xy 173.355 119.38))
+    (stroke (width 0) (type solid) (color 0 0 0 0))
+  )
   (wire (pts (xy 191.135 114.935) (xy 210.185 114.935))
     (stroke (width 0) (type solid) (color 0 0 0 0))
@@
   )
   (wire (pts (xy 238.125 117.475) (xy 238.125 120.015))
+    (stroke (width 0) (type solid) (color 0 0 0 0))
+  )
+  (bus (pts (xy 72.39 26.67) (xy 72.39 158.75))
+    (stroke (width 0) (type solid) (color 0 0 0 0))
+  )
+  (bus (pts (xy 72.39 158.75) (xy 156.845 158.75))
+    (stroke (width 0) (type solid) (color 0 0 0 0))
+  )
+  (bus (pts (xy 155.575 25.4) (xy 156.845 25.4))
+    (stroke (width 0) (type solid) (color 0 0 0 0))
+  )
+  (bus (pts (xy 156.845 25.4) (xy 156.845 158.75))
     (stroke (width 0) (type solid) (color 0 0 0 0))
   )
@@
     )
   )
-  (sheet (at 88.265 55.88) (size 45.085 89.535) (fields_autoplaced)
-    (stroke (width 0.0006) (type solid) (color 0 0 0 0))
-    (fill (color 0 0 0 0.0000))
-    (property "Sheet name" "MCU" (id 0) (at 88.265 55.2443 0)
+  (sheet (at 88.265 30.48) (size 56.515 114.935) (fields_autoplaced)
+    (stroke (width 0.0006) (type solid) (color 0 0 0 0))
+    (fill (color 0 0 0 0.0000))
+    (property "Sheet name" "MCU" (id 0) (at 88.265 29.8443 0)
       (effects (font (size 1.27 1.27)) (justify left bottom))
     )
@@
     )
   )
-  (sheet (at 27.94 52.07) (size 16.51 16.51) (fields_autoplaced)
-    (stroke (width 0.0006) (type solid) (color 0 0 0 0))
-    (fill (color 0 0 0 0.0000))
-    (property "Sheet name" "voeding" (id 0) (at 27.94 51.4343 0)
-      (effects (font (size 1.27 1.27)) (justify left bottom))
-    )
-    (property "Sheet file" "voeding.kicad_sch" (id 1) (at 27.94 69.0887 0)
-      (effects (font (size 1.27 1.27)) (justify left top))
-    )
-    (pin "SSR0_IN" input (at 44.45 55.88 0)
-      (effects (font (size 1.27 1.27)) (justify right))
-    )
-    (pin "SSR1_IN" input (at 44.45 58.42 0)
-      (effects (font (size 1.27 1.27)) (justify right))
-    )
-    (pin "CURRENT_OUT1" output (at 44.45 64.135 0)
-      (effects (font (size 1.27 1.27)) (justify right))
-    )
+  (sheet (at 27.94 45.72) (size 16.51 19.05) (fields_autoplaced)
+    (stroke (width 0.0006) (type solid) (color 0 0 0 0))
+    (fill (color 0 0 0 0.0000))
+    (property "Sheet name" "voeding" (id 0) (at 27.94 45.0843 0)
+      (effects (font (size 1.27 1.27)) (justify left bottom))
+    )
+    (property "Sheet file" "voeding.kicad_sch" (id 1) (at 27.94 65.2787 0)
+      (effects (font (size 1.27 1.27)) (justify left top))
+    )
+    (pin "SSR0_IN" input (at 44.45 49.53 0)
+      (effects (font (size 1.27 1.27)) (justify right))
+    )
+    (pin "SSR1_IN" input (at 44.45 52.705 0)
+      (effects (font (size 1.27 1.27)) (justify right))
+    )
+    (pin "CURRENT_OUT1" output (at 44.45 55.88 0)
+      (effects (font (size 1.27 1.27)) (justify right))
+    )
+    (pin "VM0" output (at 44.45 59.055 0)
+      (effects (font (size 1.27 1.27)) (justify right))
+    )
+    (pin "VM1" output (at 44.45 61.595 0)
+      (effects (font (size 1.27 1.27)) (justify right))
+    )

Commit message: versie 3
verscie 3 afgetekend
Parts:
- gave numbers to parts that had none: 4

Commit message: firmware
aan de firmware beginnen  schrijven
Other:
- added sheet connectEVE (connectEVE.kicad_sch)
- sheet voeding ports: added Relay control; removed SSR0_IN, SSR1_IN
