File: pcb/asset tracker LoRa/lora tracker V3/Lora_tracker_V3/_autosave-MCU.kicad_sch (KiCad schematic)
At the start: 2 parts

Commit message: firmware
aan de firmware beginnen  schrijven
Parts:
- gave numbers to parts that had none: 2
Changed lines of the file:
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@@
   (symbol (lib_id "power:+3V3") (at 156.845 29.845 0) (unit 1)
     (in_bom yes) (on_board yes)
-    (property "Reference" "#PWR?" (id 0) (at 156.845 33.655 0)
+    (property "Reference" "#PWR0161" (id 0) (at 156.845 33.655 0)
       (effects (font (size 1.27 1.27)) hide)
     )
@@
   (symbol (lib_id "power:GND") (at 101.6 240.665 0) (unit 1)
     (in_bom yes) (on_board yes) (fields_autoplaced)
-    (property "Reference" "#PWR?" (id 0) (at 101.6 247.015 0)
+    (property "Reference" "#PWR0160" (id 0) (at 101.6 247.015 0)
       (effects (font (size 1.27 1.27)) hide)
     )
@@
   (symbol (lib_id "power:GND") (at 145.415 54.61 0) (unit 1)
     (in_bom yes) (on_board yes) (fields_autoplaced)
-    (property "Reference" "#PWR?" (id 0) (at 145.415 60.96 0)
+    (property "Reference" "#PWR0162" (id 0) (at 145.415 60.96 0)
       (effects (font (size 1.27 1.27)) hide)
     )
@@
   (symbol (lib_id "Device:C_Polarized_Small_US") (at 145.415 45.72 0) (unit 1)
     (in_bom yes) (on_board yes) (fields_autoplaced)
-    (property "Reference" "C?" (id 0) (at 147.955 44.4499 0)
+    (property "Reference" "C24" (id 0) (at 147.955 44.4499 0)
       (effects (font (size 1.27 1.27)) (justify left))
     )
@@
   (symbol (lib_id "MCU_ST_STM32F4:STM32F407ZGTx") (at 101.6 139.065 0) (unit 1)
     (in_bom yes) (on_board yes)
-    (property "Reference" "U?" (id 0) (at 102.87 210.185 0))
+    (property "Reference" "U1" (id 0) (at 102.87 210.185 0))
     (property "Value" "STM32F407ZGTx" (id 1) (at 102.87 212.725 0))
     (property "Footprint" "halfgeleiders:STM32F407ZGT6" (id 2) (at 76.2 225.425 0)
